Commit message: Added robot state node.  Currently it just republishes joint positions.

File: trunk/industrial/motoman/cfg/sia10d_mesh.xacro (robot description, xacro)
@@ -2,4 +2,4 @@
 <robot name="sia10d_mesh" xmlns:xacro="http://ros.org/wiki/xacro">
 	<include filename="$(find motoman)/cfg/sia10d_mesh_macro.xacro" />
-	<xacro:sia20d_mesh/>
+	<xacro:sia20d_mesh prefix=""/>
 </robot>

File: trunk/industrial/motoman/cfg/sia10d_mesh_macro.xacro (robot description, xacro)
@@ -1,6 +1,6 @@
 <robot xmlns:xacro="http://ros.org/wiki/xacro">
-	<xacro:macro name="sia20d_mesh">
+	<xacro:macro name="sia20d_mesh" params="prefix">
 		<!-- link list -->
-		<link name="base_link">
+		<link name="${prefix}base_link">
 			<visual>
 				<geometry>
@@ -20,5 +20,5 @@
 			</collision>
 		</link>
-		<link name="link_s">
+		<link name="${prefix}link_s">
 			<visual>
 				<geometry>
@@ -36,5 +36,5 @@
 			</collision>
 		</link>
-		<link name="link_l">
+		<link name="${prefix}link_l">
 			<visual>
 				<geometry>
@@ -50,5 +50,5 @@
 			</collision>
 		</link>
-		<link name="link_e">
+		<link name="${prefix}link_e">
 			<visual>
 				<geometry>
@@ -64,5 +64,5 @@
 			</collision>
 		</link>
-		<link name="link_u">
+		<link name="${prefix}link_u">
 			<visual>
 				<geometry>
@@ -78,5 +78,5 @@
 			</collision>
 		</link>
-		<link name="link_r">
+		<link name="${prefix}link_r">
 			<visual>
 				<geometry>
@@ -92,5 +92,5 @@
 			</collision>
 		</link>
-		<link name="link_b">
+		<link name="${prefix}link_b">
 			<visual>
 				<geometry>
@@ -106,5 +106,5 @@
 			</collision>
 		</link>
-		<link name="link_t">
+		<link name="${prefix}link_t">
 			<visual>
 				<geometry>
@@ -122,5 +122,5 @@
 		<!-- end of link list -->
 		<!-- joint list -->
-		<joint name="joint_s" type="revolute">
+		<joint name="${prefix}joint_s" type="revolute">
 			<parent link="base_link"/>
 			<child link="link_s"/>
@@ -129,5 +129,5 @@
 			<limit lower="-3.1416" upper="3.1416" effort="100" velocity="2.96" />
 		</joint>
-		<joint name="joint_l" type="revolute">
+		<joint name="${prefix}joint_l" type="revolute">
 			<parent link="link_s"/>
 			<child link="link_l"/>
@@ -136,5 +136,5 @@
 			<limit lower="-1.91" upper="1.91" effort="100" velocity="2.96" />
 		</joint>
-		<joint name="joint_e" type="revolute">
+		<joint name="${prefix}joint_e" type="revolute">
 			<parent link="link_l"/>
 			<child link="link_e"/>
@@ -143,5 +143,5 @@
 			<limit lower="-2.96" upper="2.96" effort="100" velocity="2.96" />
 		</joint>
-		<joint name="joint_u" type="revolute">
+		<joint name="${prefix}joint_u" type="revolute">
 			<parent link="link_e"/>
 			<child link="link_u"/>
@@ -150,5 +150,5 @@
 			<limit lower="-2.35" upper="2.35" effort="100" velocity="2.96" />
 		</joint>
-		<joint name="joint_r" type="revolute">
+		<joint name="${prefix}joint_r" type="revolute">
 			<parent link="link_u"/>
 			<child link="link_r"/>
@@ -157,5 +157,5 @@
 			<limit lower="-3.1416" upper="3.1416" effort="100" velocity="3.48" />
 		</joint>
-		<joint name="joint_b" type="revolute">
+		<joint name="${prefix}joint_b" type="revolute">
 			<parent link="link_r"/>
 			<child link="link_b"/>
@@ -164,5 +164,5 @@
 			<limit lower="-1.91" upper="1.91" effort="100" velocity="3.48" />
 		</joint>
-		<joint name="joint_t" type="revolute">
+		<joint name="${prefix}joint_t" type="revolute">
 			<parent link="link_b"/>
 			<child link="link_t"/>
