Commit message: Fixed file location of link_t visual mesh.  Regenerated urdf.

File: trunk/industrial/motoman/cfg/sia10d_mesh_macro.xacro (robot description, xacro)
@@ -109,5 +109,5 @@
 			<visual>
 				<geometry>
-					<mesh filename="package://motoman/meshes/sia10d/collision/MOTOMAN_AXIS_T.stl" />
+					<mesh filename="package://motoman/meshes/sia10d/visual/MOTOMAN_AXIS_T.stl" />
 				</geometry>
 				<material name="silver"/>
