Commit message: Reworked sia20d files to match sia20d.  Prefix now required for generating robot from the xacro.  Joint frames are now oriented such that in the zero position the z axis points up and the x axis points forward (this is required for calibration under fuerte).  Join axis direction has not been verified.

File: trunk/industrial/motoman/cfg/sia20d_mesh_macro.xacro (robot description, xacro)
@@ -1,6 +1,7 @@
+<?xml version="1.0" ?>
 <robot xmlns:xacro="http://ros.org/wiki/xacro">
-	<xacro:macro name="sia20d_mesh">
+	<xacro:macro name="sia20d_mesh" params="prefix">
 		<!-- link list -->
-		<link name="base_link">
+		<link name="${prefix}base_link">
 			<visual>
 				<geometry>
@@ -20,5 +21,5 @@
 			</collision>
 		</link>
-		<link name="link_s">
+		<link name="${prefix}link_s">
 			<visual>
 				<geometry>
@@ -36,6 +37,7 @@
 			</collision>
 		</link>
-		<link name="link_l">
+		<link name="${prefix}link_l">
 			<visual>
+				<origin rpy="1.57 3.1416 0" xyz="0 0 0"/>
 				<geometry>
 					<mesh filename="package://motoman/meshes/sia20d/visual/MOTOMAN_AXIS_L.stl"/>
@@ -44,4 +46,5 @@
 			</visual>
 			<collision>
+				<origin rpy="1.57 3.1416 0" xyz="0 0 0"/>
 				<geometry>
 					<mesh filename="package://motoman/meshes/sia20d/collision/MOTOMAN_AXIS_L.stl"/>
@@ -50,6 +53,7 @@
 			</collision>
 		</link>
-		<link name="link_e">
+		<link name="${prefix}link_e">
 			<visual>
+				<origin rpy="0 0 0" xyz="0 0 0"/>
 				<geometry>
 					<mesh filename="package://motoman/meshes/sia20d/visual/MOTOMAN_AXIS_E.stl"/>
@@ -58,4 +62,5 @@
 			</visual>
 			<collision>
+				<origin rpy="0 0 0" xyz="0 0 0"/>
 				<geometry>
 					<mesh filename="package://motoman/meshes/sia20d/collision/MOTOMAN_AXIS_E.stl"/>
@@ -64,6 +69,7 @@
 			</collision>
 		</link>
-		<link name="link_u">
+		<link name="${prefix}link_u">
 			<visual>
+				<origin rpy="1.57 -3.1415 0" xyz="0 0 0"/>
 				<geometry>
 					<mesh filename="package://motoman/meshes/sia20d/visual/MOTOMAN_AXIS_U.stl"/>
@@ -72,4 +78,5 @@
 			</visual>
 			<collision>
+				<origin rpy="1.57 -3.1415 0" xyz="0 0 0"/>
 				<geometry>
 					<mesh filename="package://motoman/meshes/sia20d/collision/MOTOMAN_AXIS_U.stl"/>
@@ -78,6 +85,7 @@
 			</collision>
 		</link>
-		<link name="link_r">
+		<link name="${prefix}link_r">
 			<visual>
+				<origin rpy="0 0 3.1416" xyz="0 0 0"/>
 				<geometry>
 					<mesh filename="package://motoman/meshes/sia20d/visual/MOTOMAN_AXIS_R.stl"/>
@@ -86,4 +94,5 @@
 			</visual>
 			<collision>
+				<origin rpy="0 0 3.1416" xyz="0 0 0"/>
 				<geometry>
 					<mesh filename="package://motoman/meshes/sia20d/collision/MOTOMAN_AXIS_R.stl"/>
@@ -92,6 +101,7 @@
 			</collision>
 		</link>
-		<link name="link_b">
+		<link name="${prefix}link_b">
 			<visual>
+				<origin rpy="-1.57 0 3.1416" xyz="0 0 0"/>
 				<geometry>
 					<mesh filename="package://motoman/meshes/sia20d/visual/MOTOMAN_AXIS_B.stl"/>
@@ -100,4 +110,5 @@
 			</visual>
 			<collision>
+				<origin rpy="-1.57 0 3.1416" xyz="0 0 0"/>
 				<geometry>
 					<mesh filename="package://motoman/meshes/sia20d/collision/MOTOMAN_AXIS_B.stl"/>
@@ -106,5 +117,5 @@
 			</collision>
 		</link>
-		<link name="link_t">
+		<link name="${prefix}link_t">
 			<visual>
 				<geometry>
@@ -122,16 +133,16 @@
 		<!-- end of link list -->
 		<!-- joint list -->
-		<joint name="joint_s" type="revolute">
+		<joint name="${prefix}joint_s" type="revolute">
 			<parent link="base_link"/>
 			<child link="link_s"/>
-			<origin xyz="0 0 0.41" rpy="0 0 3.1415"/>
+			<origin xyz="0 0 0.41" rpy="0 0 0"/>
 			<axis xyz="0 0 1" />
 			<limit lower="-3.1416" upper="3.1416" effort="100" velocity="2.66" />
 		</joint>
-		<joint name="joint_l" type="revolute">
+		<joint name="${prefix}joint_l" type="revolute">
 			<parent link="link_s"/>
 			<child link="link_l"/>
-			<origin xyz="0 0 0" rpy="1.570 3.1416 0"/>
-			<axis xyz="0 0 1" />
+			<origin xyz="0 0 0" rpy="0 0 0"/>
+			<axis xyz="0 1 0" />
 			<limit lower="-1.91" upper="1.91" effort="100" velocity="2.66" />
 		</joint>
@@ -139,13 +150,13 @@
 			<parent link="link_l"/>
 			<child link="link_e"/>
-			<origin xyz="0 -0.49 0" rpy="1.570 0 0"/>
+			<origin xyz="0 0 0.49" rpy="0 0 0"/>
 			<axis xyz="0 0 1" />
 			<limit lower="-2.96" upper="2.96" effort="100" velocity="2.96" />
 		</joint>
-		<joint name="joint_u" type="revolute">
+		<joint name="${prefix}joint_u" type="revolute">
 			<parent link="link_e"/>
 			<child link="link_u"/>
-			<origin xyz="0 0 0" rpy="-1.570 0 0"/>
-			<axis xyz="0 0 -1" />
+			<origin xyz="0 0 0" rpy="0 0 0"/>
+			<axis xyz="0 -1 0" />
 			<limit lower="-3.1416" upper="3.1416" effort="100" velocity="2.96" />
 		</joint>
@@ -153,19 +164,19 @@
 			<parent link="link_u"/>
 			<child link="link_r"/>
-			<origin xyz="0 -0.420 0" rpy="1.570 0 0"/>
+			<origin xyz="0 0 0.420" rpy="0 0 0"/>
 			<axis xyz="0 0 -1" />
 			<limit lower="-3.1416" upper="3.1416" effort="100" velocity="3.48" />
 		</joint>
-		<joint name="joint_b" type="revolute">
+		<joint name="${prefix}joint_b" type="revolute">
 			<parent link="link_r"/>
 			<child link="link_b"/>
-			<origin xyz="0 0 0" rpy="-1.570 0 0"/>
-			<axis xyz="0 0 -1" />
+			<origin xyz="0 0 0" rpy="0 0 0"/>
+			<axis xyz="0 -1 0" />
 			<limit lower="-1.91" upper="1.91" effort="100" velocity="3.48" />
 		</joint>
-		<joint name="joint_t" type="revolute">
+		<joint name="${prefix}joint_t" type="revolute">
 			<parent link="link_b"/>
 			<child link="link_t"/>
-			<origin xyz="0 -0.18 0" rpy="1.570 0 0"/>
+			<origin xyz="0 0 0.18" rpy="0 0 0"/>
 			<axis xyz="0 0 -1" />
 			<limit lower="-3.1416" upper="3.1416" effort="100" velocity="6.97" />

Commit message: Updated URDF and macro to reflect joint orientation.  Changes only affected joint orientation, robot geometry(for full joint motion range) remains unchanged.  Any arm packages auto generated do not need to be recreated.

File: trunk/industrial/motoman/cfg/sia20d_mesh_macro.xacro (robot description, xacro)
@@ -1,3 +1,2 @@
-<?xml version="1.0" ?>
 <robot xmlns:xacro="http://ros.org/wiki/xacro">
 	<xacro:macro name="sia20d_mesh" params="prefix">
@@ -23,4 +22,5 @@
 		<link name="${prefix}link_s">
 			<visual>
+				<origin rpy="0 0 3.1416" xyz="0 0 0"/>
 				<geometry>
 					<mesh filename="package://motoman/meshes/sia20d/visual/MOTOMAN_AXIS_S.stl"/>
@@ -31,4 +31,5 @@
 			</visual>
 			<collision>
+				<origin rpy="0 0 3.1416" xyz="0 0 0"/>
 				<geometry>
 					<mesh filename="package://motoman/meshes/sia20d/collision/MOTOMAN_AXIS_S.stl" />
@@ -39,5 +40,5 @@
 		<link name="${prefix}link_l">
 			<visual>
-				<origin rpy="1.57 3.1416 0" xyz="0 0 0"/>
+				<origin rpy="1.57 3.1416 3.1416" xyz="0 0 0"/>
 				<geometry>
 					<mesh filename="package://motoman/meshes/sia20d/visual/MOTOMAN_AXIS_L.stl"/>
@@ -46,5 +47,5 @@
 			</visual>
 			<collision>
-				<origin rpy="1.57 3.1416 0" xyz="0 0 0"/>
+				<origin rpy="1.57 3.1416 3.1416" xyz="0 0 0"/>
 				<geometry>
 					<mesh filename="package://motoman/meshes/sia20d/collision/MOTOMAN_AXIS_L.stl"/>
@@ -71,5 +72,5 @@
 		<link name="${prefix}link_u">
 			<visual>
-				<origin rpy="1.57 -3.1415 0" xyz="0 0 0"/>
+				<origin rpy="1.57 -3.1415 3.1416" xyz="0 0 0"/>
 				<geometry>
 					<mesh filename="package://motoman/meshes/sia20d/visual/MOTOMAN_AXIS_U.stl"/>
@@ -78,5 +79,5 @@
 			</visual>
 			<collision>
-				<origin rpy="1.57 -3.1415 0" xyz="0 0 0"/>
+				<origin rpy="1.57 -3.1415 3.1416" xyz="0 0 0"/>
 				<geometry>
 					<mesh filename="package://motoman/meshes/sia20d/collision/MOTOMAN_AXIS_U.stl"/>
@@ -87,5 +88,5 @@
 		<link name="${prefix}link_r">
 			<visual>
-				<origin rpy="0 0 3.1416" xyz="0 0 0"/>
+				<origin rpy="0 0 0" xyz="0 0 0"/>
 				<geometry>
 					<mesh filename="package://motoman/meshes/sia20d/visual/MOTOMAN_AXIS_R.stl"/>
@@ -94,5 +95,5 @@
 			</visual>
 			<collision>
-				<origin rpy="0 0 3.1416" xyz="0 0 0"/>
+				<origin rpy="0 0 0" xyz="0 0 0"/>
 				<geometry>
 					<mesh filename="package://motoman/meshes/sia20d/collision/MOTOMAN_AXIS_R.stl"/>
@@ -103,5 +104,5 @@
 		<link name="${prefix}link_b">
 			<visual>
-				<origin rpy="-1.57 0 3.1416" xyz="0 0 0"/>
+				<origin rpy="-1.57 0 0" xyz="0 0 0"/>
 				<geometry>
 					<mesh filename="package://motoman/meshes/sia20d/visual/MOTOMAN_AXIS_B.stl"/>
@@ -110,5 +111,5 @@
 			</visual>
 			<collision>
-				<origin rpy="-1.57 0 3.1416" xyz="0 0 0"/>
+				<origin rpy="-1.57 0 0" xyz="0 0 0"/>
 				<geometry>
 					<mesh filename="package://motoman/meshes/sia20d/collision/MOTOMAN_AXIS_B.stl"/>
@@ -154,5 +155,5 @@
 			<limit lower="-2.96" upper="2.96" effort="100" velocity="2.96" />
 		</joint>
-		<joint name="${prefix}joint_u" type="revolute">
+		<joint name="joint_u" type="revolute">
 			<parent link="link_e"/>
 			<child link="link_u"/>
@@ -168,5 +169,5 @@
 			<limit lower="-3.1416" upper="3.1416" effort="100" velocity="3.48" />
 		</joint>
-		<joint name="${prefix}joint_b" type="revolute">
+		<joint name="joint_b" type="revolute">
 			<parent link="link_r"/>
 			<child link="link_b"/>
@@ -175,5 +176,5 @@
 			<limit lower="-1.91" upper="1.91" effort="100" velocity="3.48" />
 		</joint>
-		<joint name="${prefix}joint_t" type="revolute">
+		<joint name="joint_t" type="revolute">
 			<parent link="link_b"/>
 			<child link="link_t"/>

Commit message: Updated sia20d urdf to reflex actual joint limits (from official motoman drawing).  Previous limits were incorrect.  Any generated arm_navigation packages should be updated.

File: trunk/industrial/motoman/cfg/sia20d_mesh_macro.xacro (robot description, xacro)
@@ -139,5 +139,5 @@
 			<origin xyz="0 0 0.41" rpy="0 0 0"/>
 			<axis xyz="0 0 1" />
-			<limit lower="-3.1416" upper="3.1416" effort="100" velocity="2.66" />
+			<limit lower="-3.1416" upper="3.1416" effort="100" velocity="2.26" />
 		</joint>
 		<joint name="${prefix}joint_l" type="revolute">
@@ -146,7 +146,7 @@
 			<origin xyz="0 0 0" rpy="0 0 0"/>
 			<axis xyz="0 1 0" />
-			<limit lower="-1.91" upper="1.91" effort="100" velocity="2.66" />
+			<limit lower="-1.91" upper="1.91" effort="100" velocity="2.26" />
 		</joint>
-		<joint name="joint_e" type="revolute">
+		<joint name="{prefix}joint_e" type="revolute">
 			<parent link="link_l"/>
 			<child link="link_e"/>
@@ -155,12 +155,12 @@
 			<limit lower="-2.96" upper="2.96" effort="100" velocity="2.96" />
 		</joint>
-		<joint name="joint_u" type="revolute">
+		<joint name="{prefix}joint_u" type="revolute">
 			<parent link="link_e"/>
 			<child link="link_u"/>
 			<origin xyz="0 0 0" rpy="0 0 0"/>
 			<axis xyz="0 -1 0" />
-			<limit lower="-3.1416" upper="3.1416" effort="100" velocity="2.96" />
+			<limit lower="-2.26" upper="2.26" effort="100" velocity="2.96" />
 		</joint>
-		<joint name="joint_r" type="revolute">
+		<joint name="{prefix}joint_r" type="revolute">
 			<parent link="link_u"/>
 			<child link="link_r"/>
@@ -169,5 +169,5 @@
 			<limit lower="-3.1416" upper="3.1416" effort="100" velocity="3.48" />
 		</joint>
-		<joint name="joint_b" type="revolute">
+		<joint name="{prefix}joint_b" type="revolute">
 			<parent link="link_r"/>
 			<child link="link_b"/>
@@ -176,5 +176,5 @@
 			<limit lower="-1.91" upper="1.91" effort="100" velocity="3.48" />
 		</joint>
-		<joint name="joint_t" type="revolute">
+		<joint name="{prefix}joint_t" type="revolute">
 			<parent link="link_b"/>
 			<child link="link_t"/>

Commit message: Fixed xacro parameter ${prefix}

File: trunk/industrial/motoman/cfg/sia20d_mesh_macro.xacro (robot description, xacro)
@@ -148,5 +148,5 @@
 			<limit lower="-1.91" upper="1.91" effort="100" velocity="2.26" />
 		</joint>
-		<joint name="{prefix}joint_e" type="revolute">
+		<joint name="${prefix}joint_e" type="revolute">
 			<parent link="link_l"/>
 			<child link="link_e"/>
@@ -155,5 +155,5 @@
 			<limit lower="-2.96" upper="2.96" effort="100" velocity="2.96" />
 		</joint>
-		<joint name="{prefix}joint_u" type="revolute">
+		<joint name="${prefix}joint_u" type="revolute">
 			<parent link="link_e"/>
 			<child link="link_u"/>
@@ -162,5 +162,5 @@
 			<limit lower="-2.26" upper="2.26" effort="100" velocity="2.96" />
 		</joint>
-		<joint name="{prefix}joint_r" type="revolute">
+		<joint name="${prefix}joint_r" type="revolute">
 			<parent link="link_u"/>
 			<child link="link_r"/>
@@ -169,5 +169,5 @@
 			<limit lower="-3.1416" upper="3.1416" effort="100" velocity="3.48" />
 		</joint>
-		<joint name="{prefix}joint_b" type="revolute">
+		<joint name="${prefix}joint_b" type="revolute">
 			<parent link="link_r"/>
 			<child link="link_b"/>
@@ -176,5 +176,5 @@
 			<limit lower="-1.91" upper="1.91" effort="100" velocity="3.48" />
 		</joint>
-		<joint name="{prefix}joint_t" type="revolute">
+		<joint name="${prefix}joint_t" type="revolute">
 			<parent link="link_b"/>
 			<child link="link_t"/>
