Commit message: 

File: trunk/industrial/adept/adept_common/urdf/Adept_Viper_s650.urdf (robot description, URDF)
Before this commit: robot ADEPT_VIPER_S650, 6 links, 5 joints
Links:
- added link Adept_Viper_650_Interface_Plate; collision mesh filename=package://adept_common/meshes/collision/STL/binary/Adept_Vi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; visual mesh filename=package://adept_common/meshes/visual/STL/binary/Adept_Viper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
Joints:
- added joint joint_6: type revolute, parent Adept_Viper_s650_Link6, child Adept_Viper_650_Interface_Plate, origin xyz=0.08 0 0, axis 1 0 0, limit lower=-3.1416 upper=3.1416 effort=100 velocity=1.0
