Commit message: Finished longhorn urdf.  Not yet verified.

File: trunk/industrial/longhorn/cfg/longhorn.xacro (robot description, xacro)
@@ -1,4 +1,4 @@
 <?xml version="1.0" ?>
-<robot name="armadillo" xmlns:xacro="http://ros.org/wiki/xacro">
+<robot name="longhorn" xmlns:xacro="http://ros.org/wiki/xacro">
 	<include filename="$(find motoman)/cfg/sia10d_mesh_macro.xacro" />
 	<include filename="$(find robotiq)/cfg/s-model_mesh_macro.xacro" />
@@ -41,5 +41,5 @@
 			<visual>
 				<geometry>
-					<box size="2 2 0.75"/>
+					<box size="1.83 2.44 0.25"/>
 				</geometry>
 				<material name="">
@@ -47,74 +47,77 @@
 				</material>
 			</visual>
+      <collision>
+				<geometry>
+					<box size="1.83 2.44 0.25"/>
+				</geometry>
+				<material name="">
+					<color rgba="1 0 1 1"/>
+				</material>
+			</collision>
 		</link>
 		<link name="table_keepout_1">
-			<visual>
+			<collision>
 				<geometry>
-					<box size="2 0.25 2"/>
+					<box size="2.08 0.25 2"/>
 				</geometry>
 				<material name="">
-					<color rgba="1 0.2 1 0.25"/>
+					<color rgba="1 0.2 1 0.1"/>
 				</material>
-			</visual>
+			</collision>
 		</link>
 		<link name="table_keepout_2">
-			<visual>
+			<collision>
 				<geometry>
-					<box size="0.25 2 2"/>
+					<box size="0.25 2.69 2"/>
 				</geometry>
 				<material name="">
-					<color rgba="1 0.2 1 0.25"/>
+					<color rgba="1 0.2 1 0.1"/>
 				</material>
-			</visual>
+			</collision>
 		</link>
 		<link name="kinect_keepout">
-			<visual>
+			<collision>
 				<geometry>
-					<box size="0.25 2 2"/>
+					<box size="0.25 2.69 2"/>
 				</geometry>
 				<material name="">
-					<color rgba="1 0.2 1 0.25"/>
+					<color rgba="1 0.2 1 0.1"/>
 				</material>
-			</visual>
+			</collision>
 		</link>
     <link name="kinect">
-			<visual>
+			<collision>
 				<geometry>
 					<box size="0.36 0.28 0.22"/>
 				</geometry>
 				<material name="">
-					<color rgba="1 0.8 1 1"/>
+					<color rgba="1 0.8 1 0.1"/>
 				</material>
-			</visual>
+			</collision>
 		</link>
 		<joint name="base-table" type="fixed">
 			<parent link="base_link"/>
 			<child link="table"/>
-			<origin xyz="-0.52 -0.34 -0.11" rpy="0 0 0"/>
+			<origin xyz="1.19 0.22 -0.125" rpy="0 0 -0.785"/>
 		</joint>
-		<joint name="base-controller" type="fixed">
+		<joint name="base-kinect" type="fixed">
 			<parent link="base_link"/>
-			<child link="controller"/>
-			<origin xyz="-0.75 -0.50 0.50" rpy="0 0 0"/>
+			<child link="kinect"/>
+			<origin xyz="1.26 -0.72 0.75" rpy="0 0 2.356"/>
 		</joint>
-		<joint name="base-filter" type="fixed">
-			<parent link="base_link"/>
-			<child link="filter"/>
-			<origin xyz="-0.17 -0.50 0.63" rpy="0 0 0"/>
+		<joint name="table-keepout_1" type="fixed">
+			<parent link="table"/>
+			<child link="table_keepout_1"/>
+			<origin xyz="0 -1.34 1" rpy="0 0 0"/>
 		</joint>
-		<joint name="pallet-floor" type="fixed">
-			<parent link="pallet"/>
-			<child link="floor"/>
-			<origin xyz="0 0 -0.11" rpy="0 0 0"/>
+		<joint name="table-keepout_2" type="fixed">
+			<parent link="table"/>
+			<child link="table_keepout_2"/>
+			<origin xyz="-1.025 0 1" rpy="0 0 0"/>
 		</joint>
-		<joint name="filter-kinect" type="fixed">
-			<parent link="filter"/>
-			<child link="kinect"/>
-			<origin xyz="0.18 0 0.29" rpy="0 0 0"/>
-		</joint>
-		<joint name="base-tables" type="fixed">
-			<parent link="base_link"/>
-			<child link="tables"/>
-			<origin xyz="0.84 0 0" rpy="0 0 0"/>
+		<joint name="table-kinect" type="fixed">
+			<parent link="table"/>
+			<child link="kinect_keepout"/>
+			<origin xyz=".5 0 1" rpy="0 0 0"/>
 		</joint>
   <!-- end environment list -->
@@ -123,5 +126,5 @@
 			<parent link="kinect"/>
 			<child link="kinect_frame"/>
-			<origin rpy="0.075 0.351422870712 0.396594014755" xyz="-0.12481258247 0.064659133914 -0.022541275619"/>
+			<origin rpy="0 0 0" xyz="0 0 0"/>
 		</joint>
 		<link name="kinect_frame">

Commit message: Updated longhorn xacro and urdf to reflect physical construction.

File: trunk/industrial/longhorn/cfg/longhorn.xacro (robot description, xacro)
@@ -34,5 +34,5 @@
 			<parent link="coupler"/>
 			<child link="palm"/>
-			<origin xyz="0 0.240 0" rpy="-1.570 -0.478 0"/>
+			<origin xyz="0 0.240 0" rpy="-1.570 -2.356 0"/>
 		</joint>
   <!-- end of joint list -->

Commit message: Updated URDF and macro.  Significant changes were made to geometry (sia10 models were replaced with sia20).  Auto generated arm packages must be regenerated.

File: trunk/industrial/longhorn/cfg/longhorn.xacro (robot description, xacro)
@@ -1,7 +1,7 @@
 <?xml version="1.0" ?>
 <robot name="longhorn" xmlns:xacro="http://ros.org/wiki/xacro">
-	<include filename="$(find motoman)/cfg/sia10d_mesh_macro.xacro" />
+	<include filename="$(find motoman)/cfg/sia20d_mesh_macro.xacro" />
 	<include filename="$(find robotiq)/cfg/s-model_mesh_macro.xacro" />
-	<xacro:sia10d_mesh prefix=""/>
+	<xacro:sia20d_mesh prefix=""/>
 	<xacro:s-model_mesh prefix=""/>
   <!-- link list -->
@@ -9,5 +9,5 @@
 			<visual>
 				<geometry>
-					<mesh filename="package://armadillo/meshes/coupler/visual/COUPLER.stl" />
+					<mesh filename="package://longhorn/meshes/coupler/visual/COUPLER.stl" />
 				</geometry>
 				<material name="orange">
@@ -17,5 +17,5 @@
 			<collision>
 				<geometry>
-					<mesh filename="package://armadillo/meshes/coupler/collision/COUPLER.stl" />
+					<mesh filename="package://longhorn/meshes/coupler/collision/COUPLER.stl" />
 				</geometry>
 				<material name="yellow">

Commit message: Fixed longhorn arm navigation package.  Regenerated with wizard.  (sia10d arm was used in previous attempt).

File: trunk/industrial/longhorn/cfg/longhorn.xacro (robot description, xacro)
@@ -76,4 +76,14 @@
 			</collision>
 		</link>
+		<link name="abb_keepout">
+			<collision>
+				<geometry>
+					<box size="0.915 1.524 2"/>
+				</geometry>
+				<material name="">
+					<color rgba="1 0.2 1 0.1"/>
+				</material>
+			</collision>
+		</link>
 		<link name="kinect_keepout">
 			<collision>
@@ -115,4 +125,9 @@
 			<child link="table_keepout_2"/>
 			<origin xyz="-1.025 0 1" rpy="0 0 0"/>
+		</joint>
+		<joint name="abb-keepout" type="fixed">
+			<parent link="table"/>
+			<child link="abb_keepout"/>
+			<origin xyz="0.475 0.458 1.125" rpy="0 0 0"/>
 		</joint>
 		<joint name="table-kinect" type="fixed">

Commit message: Updated URDF (should have been included with previous check-in).

File: trunk/industrial/longhorn/cfg/longhorn.xacro (robot description, xacro)
@@ -86,4 +86,14 @@
 			</collision>
 		</link>
+		<link name="power_supply">
+			<visual>
+				<geometry>
+					<box size="0.400 0.250 0.115"/>
+				</geometry>
+				<material name="">
+					<color rgba="1 0.2 1 0.1"/>
+				</material>
+			</visual>
+		</link>
 		<link name="kinect_keepout">
 			<collision>
@@ -130,4 +140,9 @@
 			<child link="abb_keepout"/>
 			<origin xyz="0.475 0.458 1.125" rpy="0 0 0"/>
+		</joint>
+		<joint name="base-power_supply" type="fixed">
+			<parent link="base_link"/>
+			<child link="power_supply"/>
+			<origin xyz="0 -0.260 0.050" rpy="0 0 0"/>
 		</joint>
 		<joint name="table-kinect" type="fixed">
