Commit message: Added comments to urdf xacros.  Collsion STLs changed to convex hulls.  Removed limits from fixed links.

File: trunk/industrial/robotiq/cfg/s-model_articulated.urdf (robot description, URDF)
Before this commit: robot s-model_articulated, 13 links, 12 joints
Joints:
- joint joint_finger_1: limit lower=0 upper=3.1416 effort=100 velocity=100 -> (none)
- joint joint_finger_2: limit lower=0 upper=3.1416 effort=100 velocity=100 -> (none)
- joint joint_finger_middle: limit lower=0 upper=3.1416 effort=100 velocity=100 -> (none)

File: trunk/industrial/robotiq/cfg/s-model_articulated_macro.xacro (robot description, xacro)
@@ -1,2 +1,9 @@
+<!--
+s-model_articulated_macro(prefix)
+Creates an articulated s-model hand with the passed in prefix.  If there
+is only one hand in the urdf then an empty prefix can be used "".  If
+there are multiple hands then a prefix followed by an "_" is needed.
+NOTE: This urdf does not include the "scissor" degree of freedom.
+-->
 <robot xmlns:xacro="http://ros.org/wiki/xacro">
 	<include filename="$(find robotiq)/cfg/s-model_finger_articulated_macro.xacro" />
@@ -26,5 +33,4 @@
 		<!-- end of link list -->
 		<!-- joint list -->
-		<!-- WARNING: LIMITS NOT CORRECT -->
 		<joint name="${prefix}joint_finger_1" type="fixed">
 			<parent link="${prefix}palm"/>
@@ -32,7 +38,5 @@
 			<axis xyz="0 0 1"/>
 			<origin xyz="0 0 0" rpy="0 0 0"/>
-			<limit lower="0" upper="3.1416" effort="100" velocity="100" />
 		</joint>
-		<!-- WARNING: LIMITS NOT CORRECT -->
 		<joint name="${prefix}joint_finger_2" type="fixed">
 			<parent link="${prefix}palm"/>
@@ -40,7 +44,5 @@
 			<axis xyz="0 0 1"/>
 			<origin xyz="0 0 0" rpy="0 0 0"/>
-			<limit lower="0" upper="3.1416" effort="100" velocity="100" />
 		</joint>
-		<!-- WARNING: LIMITS NOT CORRECT -->
 		<joint name="${prefix}joint_finger_middle" type="fixed">
 			<parent link="${prefix}palm"/>
@@ -48,5 +50,4 @@
 			<axis xyz="0 0 1"/>
 			<origin xyz="0 0 0" rpy="0 0 0"/>
-			<limit lower="0" upper="3.1416" effort="100" velocity="100" />
 		</joint>
 		<!-- end of joint list -->

File: trunk/industrial/robotiq/cfg/s-model_finger_articulated_macro.xacro (robot description, xacro)
@@ -1,2 +1,11 @@
+<!--
+s-model_finder_articulated_macro(prefix, origin_xyz, origin_rpy)
+Creates an articulated s-model finder with the passed in prefix.  The
+prefix typcially includes the hand prefix and an identifier for the
+finger(i.e. finger_1, etc...).
+The origin of the first link (link_0) must is also required.  It is
+passed as two parameters, one for xyz and one for rpy.
+NOTE: This urdf does not include the "scissor" degree of freedom.
+-->
 <robot xmlns:xacro="http://ros.org/wiki/xacro">
 	<xacro:macro name="s-model_finger_articulated" params="prefix origin_xyz origin_rpy">

Commit message: Added scissor degree of freedom to s-model gripper.

File: trunk/industrial/robotiq/cfg/s-model_articulated.urdf (robot description, URDF)
Before this commit: robot s-model_articulated, 13 links, 12 joints
Joints:
- removed joint joint_finger_1
- removed joint joint_finger_2
- removed joint joint_finger_middle
- added joint palm_finger_1_joint: type revolute, parent palm, child finger_1_link_0, origin xyz=-0.0455 0.0214 0.036 rpy=0 3.1416 -1.57, axis 0 1 0, limit lower=-0.16 upper=0.25 effort=100 velocity=100
- added joint palm_finger_2_joint: type revolute, parent palm, child finger_2_link_0, origin xyz=-0.0455 0.0214 -0.036 rpy=0 3.1416 -1.57, axis 0 1 0, limit lower=-0.25 upper=0.16 effort=100 velocity=100
- added joint palm_finger_middle_joint: type fixed, parent palm, child finger_middle_link_0, origin xyz=0.0455 0.0214 0 rpy=0 0 1.57, axis 0 0 1
- joint finger_1_joint_1: origin xyz=-0.0455 0.0414 0.036 rpy=0 3.1416 -1.57 -> xyz=0.020 0 0 rpy=0 0 0
- joint finger_2_joint_1: origin xyz=-0.0455 0.0414 -0.036 rpy=0 3.1416 -1.57 -> xyz=0.020 0 0 rpy=0 0 0
- joint finger_middle_joint_1: origin xyz=0.0455 0.0414 0 rpy=0 0 1.57 -> xyz=0.020 0 0 rpy=0 0 0

File: trunk/industrial/robotiq/cfg/s-model_articulated_macro.xacro (robot description, xacro)
@@ -4,12 +4,11 @@
 is only one hand in the urdf then an empty prefix can be used "".  If
 there are multiple hands then a prefix followed by an "_" is needed.
-NOTE: This urdf does not include the "scissor" degree of freedom.
 -->
 <robot xmlns:xacro="http://ros.org/wiki/xacro">
 	<include filename="$(find robotiq)/cfg/s-model_finger_articulated_macro.xacro" />
 	<xacro:macro name="s-model_articulated" params="prefix">
-	<xacro:s-model_finger_articulated prefix="${prefix}finger_1_" origin_xyz="-0.0455 0.0414 0.036" origin_rpy="0 3.1416 -1.57"/>
-	<xacro:s-model_finger_articulated prefix="${prefix}finger_2_" origin_xyz="-0.0455 0.0414 -0.036" origin_rpy="0 3.1416 -1.57"/>
-	<xacro:s-model_finger_articulated prefix="${prefix}finger_middle_" origin_xyz="0.0455 0.0414 0" origin_rpy="0 0 1.57"/>
+	<xacro:s-model_finger_articulated prefix="${prefix}finger_1_"/>
+	<xacro:s-model_finger_articulated prefix="${prefix}finger_2_"/>
+	<xacro:s-model_finger_articulated prefix="${prefix}finger_middle_"/>
 		<!-- link list -->
 		<link name="${prefix}palm">
@@ -33,21 +32,25 @@
 		<!-- end of link list -->
 		<!-- joint list -->
-		<joint name="${prefix}joint_finger_1" type="fixed">
+		<!-- WARNING: LIMITS NOT CORRECT -->
+		<joint name="${prefix}palm_finger_1_joint" type="revolute">
 			<parent link="${prefix}palm"/>
 			<child link="${prefix}finger_1_link_0"/>
-			<axis xyz="0 0 1"/>
-			<origin xyz="0 0 0" rpy="0 0 0"/>
+			<axis xyz="0 1 0"/>
+			<origin xyz="-0.0455 0.0214 0.036" rpy="0 3.1416 -1.57"/>
+			<limit lower="-0.16" upper="0.25" effort="100" velocity="100"/>
 		</joint>
-		<joint name="${prefix}joint_finger_2" type="fixed">
+		<!-- WARNING: LIMITS NOT CORRECT -->
+		<joint name="${prefix}palm_finger_2_joint" type="revolute">
 			<parent link="${prefix}palm"/>
 			<child link="${prefix}finger_2_link_0"/>
-			<axis xyz="0 0 1"/>
-			<origin xyz="0 0 0" rpy="0 0 0"/>
+			<axis xyz="0 1 0"/>
+			<origin xyz="-0.0455 0.0214 -0.036" rpy="0 3.1416 -1.57"/>
+			<limit lower="-0.25" upper="0.16" effort="100" velocity="100"/>
 		</joint>
-		<joint name="${prefix}joint_finger_middle" type="fixed">
+		<joint name="${prefix}palm_finger_middle_joint" type="fixed">
 			<parent link="${prefix}palm"/>
 			<child link="${prefix}finger_middle_link_0"/>
 			<axis xyz="0 0 1"/>
-			<origin xyz="0 0 0" rpy="0 0 0"/>
+			<origin xyz="0.0455 0.0214 0" rpy="0 0 1.57"/>
 		</joint>
 		<!-- end of joint list -->

File: trunk/industrial/robotiq/cfg/s-model_finger_articulated_macro.xacro (robot description, xacro)
@@ -1,17 +1,14 @@
 <!--
-s-model_finder_articulated_macro(prefix, origin_xyz, origin_rpy)
+s-model_finder_articulated_macro(prefix)
 Creates an articulated s-model finder with the passed in prefix.  The
 prefix typcially includes the hand prefix and an identifier for the
 finger(i.e. finger_1, etc...).
-The origin of the first link (link_0) must is also required.  It is
-passed as two parameters, one for xyz and one for rpy.
-NOTE: This urdf does not include the "scissor" degree of freedom.
 -->
 <robot xmlns:xacro="http://ros.org/wiki/xacro">
-	<xacro:macro name="s-model_finger_articulated" params="prefix origin_xyz origin_rpy">
+	<xacro:macro name="s-model_finger_articulated" params="prefix">
 		<!-- link list -->
 		<link name="${prefix}link_0">
 			<visual>
-				<origin xyz="${origin_xyz}" rpy="${origin_rpy}"/>
+				<origin xyz="0.020 0 0" rpy="0 0 0"/>
 				<geometry>
 					<mesh filename="package://robotiq/meshes/s-model_articulated/visual/link_0.STL" />
@@ -91,5 +88,5 @@
 			<child link="${prefix}link_1"/>
 			<axis xyz="0 0 1"/>
-			<origin xyz="${origin_xyz}" rpy="${origin_rpy}"/>
+			<origin xyz="0.020 0 0" rpy="0 0 0"/>
 			<limit lower="0" upper="3.1416" effort="100" velocity="100"/>
 		</joint>
