Commit message: Making everything work with manipulation with articulated hand

File: branches/moveit_industrial/armadillo/cfg/armadillo.urdf (robot description, URDF)
Before this commit: robot armadillo, 24 links, 23 joints
Links:
- removed link finger_1
- removed link finger_2
- removed link finger_3
- added link finger_0_link_0; collision mesh filename=package://robotiq/meshes/s-model_articulated/collision/link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; visual mesh filename=package://robotiq/meshes/s-model_articulated/visual/link_0.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
- added link finger_0_link_1; collision mesh filename=package://robotiq/meshes/s-model_articulated/collision/link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; visual mesh filename=package://robotiq/meshes/s-model_articulated/visual/link_1.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
- added link finger_0_link_2; collision mesh filename=package://robotiq/meshes/s-model_articulated/collision/link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; visual mesh filename=package://robotiq/meshes/s-model_articulated/visual/link_2.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
- added link finger_0_link_3; collision mesh filename=package://robotiq/meshes/s-model_articulated/collision/link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; visual mesh filename=package://robotiq/meshes/s-model_articulated/visual/link_3.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
- added link finger_1_link_0; collision mesh filename=package://robotiq/meshes/s-model_articulated/collision/link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; visual mesh filename=package://robotiq/meshes/s-model_articulated/visual/link_0.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
- added link finger_1_link_1; collision mesh filename=package://robotiq/meshes/s-model_articulated/collision/link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; visual mesh filename=package://robotiq/meshes/s-model_articulated/visual/link_1.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
- added link finger_1_link_2; collision mesh filename=package://robotiq/meshes/s-model_articulated/collision/link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; visual mesh filename=package://robotiq/meshes/s-model_articulated/visual/link_2.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
- added link finger_1_link_3; collision mesh filename=package://robotiq/meshes/s-model_articulated/collision/link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; visual mesh filename=package://robotiq/meshes/s-model_articulated/visual/link_3.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
- added link finger_2_link_0; collision mesh filename=package://robotiq/meshes/s-model_articulated/collision/link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; visual mesh filename=package://robotiq/meshes/s-model_articulated/visual/link_0.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
- added link finger_2_link_1; collision mesh filename=package://robotiq/meshes/s-model_articulated/collision/link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; visual mesh filename=package://robotiq/meshes/s-model_articulated/visual/link_1.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
- added link finger_2_link_2; collision mesh filename=package://robotiq/meshes/s-model_articulated/collision/link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; visual mesh filename=package://robotiq/meshes/s-model_articulated/visual/link_2.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
- added link finger_2_link_3; collision mesh filename=package://robotiq/meshes/s-model_articulated/collision/link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; visual mesh filename=package://robotiq/meshes/s-model_articulated/visual/link_3.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
- link palm: geometry collision mesh filename=package://robotiq/meshes/s-model_articulated/collision/palm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; visual mesh filename=package://robotiq/meshes/s-model_articulated/visual/palm.STL
Joints:
- removed joint joint_1
- removed joint joint_2
- removed joint joint_3
- added joint finger_0_joint_1: type revolute, parent finger_0_link_0, child finger_0_link_1, origin xyz=0.020 0 0 rpy=0 0 0, axis 0 0 1, limit lower=0 upper=3.1416 effort=100 velocity=100
- added joint finger_0_joint_2: type revolute, parent finger_0_link_1, child finger_0_link_2, origin xyz=0.050 -.028 0 rpy=0 0 -0.52, axis 0 0 1, limit lower=0 upper=3.1416 effort=100 velocity=100
- added joint finger_0_joint_3: type revolute, parent finger_0_link_2, child finger_0_link_3, origin xyz=0.039 0 0 rpy=0 0 0, axis 0 0 1, limit lower=0 upper=3.1416 effort=100 velocity=100
- added joint finger_1_joint_1: type revolute, parent finger_1_link_0, child finger_1_link_1, origin xyz=0.020 0 0 rpy=0 0 0, axis 0 0 1, limit lower=0 upper=3.1416 effort=100 velocity=100
- added joint finger_1_joint_2: type revolute, parent finger_1_link_1, child finger_1_link_2, origin xyz=0.050 -.028 0 rpy=0 0 -0.52, axis 0 0 1, limit lower=0 upper=3.1416 effort=100 velocity=100
- added joint finger_1_joint_3: type revolute, parent finger_1_link_2, child finger_1_link_3, origin xyz=0.039 0 0 rpy=0 0 0, axis 0 0 1, limit lower=0 upper=3.1416 effort=100 velocity=100
- added joint finger_2_joint_1: type revolute, parent finger_2_link_0, child finger_2_link_1, origin xyz=0.020 0 0 rpy=0 0 0, axis 0 0 1, limit lower=0 upper=3.1416 effort=100 velocity=100
- added joint finger_2_joint_2: type revolute, parent finger_2_link_1, child finger_2_link_2, origin xyz=0.050 -.028 0 rpy=0 0 -0.52, axis 0 0 1, limit lower=0 upper=3.1416 effort=100 velocity=100
- added joint finger_2_joint_3: type revolute, parent finger_2_link_2, child finger_2_link_3, origin xyz=0.039 0 0 rpy=0 0 0, axis 0 0 1, limit lower=0 upper=3.1416 effort=100 velocity=100
- added joint palm_finger_0_joint: type fixed, parent palm, child finger_0_link_0, origin xyz=0.0455 0.0214 0 rpy=0 0 1.57, axis 0 0 1
- added joint palm_finger_1_joint: type revolute, parent palm, child finger_1_link_0, origin xyz=-0.0455 0.0214 0.036 rpy=0 3.1416 -1.57, axis 0 1 0, limit lower=-0.16 upper=0.25 effort=100 velocity=100
- added joint palm_finger_2_joint: type revolute, parent palm, child finger_2_link_0, origin xyz=-0.0455 0.0214 -0.036 rpy=0 3.1416 -1.57, axis 0 1 0, limit lower=-0.25 upper=0.16 effort=100 velocity=100
- joint coupler-hand: origin xyz=0 0.240 0 rpy=-1.570 -0.478 0 -> xyz=0 0.120 0 rpy=0 0 0

File: branches/moveit_industrial/armadillo/cfg/armadillo.xacro (robot description, xacro)
@@ -1,191 +1,191 @@
 <?xml version="1.0" ?>
 <robot name="armadillo" xmlns:xacro="http://ros.org/wiki/xacro">
-	<include filename="$(find motoman)/cfg/sia10d_mesh_macro.xacro" />
-	<include filename="$(find robotiq)/cfg/s-model_mesh_macro.xacro" />
-	<xacro:sia10d_mesh prefix=""/>
-	<xacro:s-model_mesh prefix=""/>
+  <include filename="$(find motoman)/cfg/sia10d_mesh_macro.xacro" />
+  <include filename="$(find robotiq)/cfg/s-model_articulated_macro.xacro" />
+  <xacro:sia10d_mesh prefix=""/>
+  <xacro:s-model_articulated prefix=""/>
   <!-- link list -->
-		<link name="coupler">
-			<visual>
-				<geometry>
-					<mesh filename="package://armadillo/meshes/coupler/visual/COUPLER.stl" />
-				</geometry>
-				<material name="orange">
-					<color rgba="1 0.5 0 1"/>
-				</material>
-			</visual>
-			<collision>
-				<geometry>
-					<mesh filename="package://armadillo/meshes/coupler/collision/COUPLER.stl" />
-				</geometry>
-				<material name="yellow">
-					<color rgba="0 1 1 1"/>
-				</material>
-			</collision>
-		</link>
+  <link name="coupler">
+    <visual>
+      <geometry>
+	<mesh filename="package://armadillo/meshes/coupler/visual/COUPLER.stl" />
+      </geometry>
+      <material name="orange">
+	<color rgba="1 0.5 0 1"/>
+      </material>
+    </visual>
+    <collision>
+      <geometry>
+	<mesh filename="package://armadillo/meshes/coupler/collision/COUPLER.stl" />
+      </geometry>
+      <material name="yellow">
+	<color rgba="0 1 1 1"/>
+      </material>
+    </collision>
+  </link>
   <!-- end link list -->
   <!-- joint list -->
-		<joint name="tool-coupler" type="fixed">
-			<parent link="link_t"/>
-			<child link="coupler"/>
-			<origin xyz="0 0 0" rpy="1.570 0 0"/>
-		</joint>
-		<joint name="coupler-hand" type="fixed">
-			<parent link="coupler"/>
-			<child link="palm"/>
-			<origin xyz="0 0.240 0" rpy="-1.570 -0.478 0"/>
-		</joint>
+  <joint name="tool-coupler" type="fixed">
+    <parent link="link_t"/>
+    <child link="coupler"/>
+    <origin xyz="0 0 0" rpy="1.570 0 0"/>
+  </joint>
+  <joint name="coupler-hand" type="fixed">
+    <parent link="coupler"/>
+    <child link="palm"/>
+    <origin xyz="0 0.120 0" rpy="0 0 0"/>
+  </joint>
   <!-- end of joint list -->
   <!-- environment list -->
-		<link name="pallet">
-			<visual>
-				<geometry>
-					<box size="1.61 1.16 0.213"/>
-				</geometry>
-				<material name="">
-					<color rgba="1 0 1 1"/>
-				</material>
-			</visual>
-		</link>
-		<link name="controller">
-			<visual>
-				<geometry>
-					<box size="0.80 0.65 1.00"/>
-				</geometry>
-				<material name="">
-					<color rgba="1 0.2 1 1"/>
-				</material>
-			</visual>
-		</link>
-    <link name="filter">
-			<visual>
-				<geometry>
-					<box size="0.36 0.36 0.36"/>
-				</geometry>
-				<material name="">
-					<color rgba="1 0.4 1 1"/>
-				</material>
-			</visual>
-		</link>
-    <link name="floor">
-			<visual>
-				<geometry>
-					<box size="6 6 0.010"/>
-				</geometry>
-				<material name="">
-					<color rgba="1 0.6 1 0.5"/>
-				</material>
-			</visual>
-		</link>
-    <link name="kinect">
-			<visual>
-				<geometry>
-					<box size="0.36 0.28 0.22"/>
-				</geometry>
-				<material name="">
-					<color rgba="1 0.8 1 1"/>
-				</material>
-			</visual>
-		</link>
-    <link name="tables">
-			<visual>
-				<geometry>
-					<box size="1.10 1.65 0.45"/>
-				</geometry>
-				<material name="">
-					<color rgba="1 0.7 1 1"/>
-				</material>
-			</visual>
-		</link>
-		<joint name="base-pallet" type="fixed">
-			<parent link="base_link"/>
-			<child link="pallet"/>
-			<origin xyz="-0.52 -0.34 -0.11" rpy="0 0 0"/>
-		</joint>
-		<joint name="base-controller" type="fixed">
-			<parent link="base_link"/>
-			<child link="controller"/>
-			<origin xyz="-0.75 -0.50 0.50" rpy="0 0 0"/>
-		</joint>
-		<joint name="base-filter" type="fixed">
-			<parent link="base_link"/>
-			<child link="filter"/>
-			<origin xyz="-0.17 -0.50 0.63" rpy="0 0 0"/>
-		</joint>
-		<joint name="pallet-floor" type="fixed">
-			<parent link="pallet"/>
-			<child link="floor"/>
-			<origin xyz="0 0 -0.11" rpy="0 0 0"/>
-		</joint>
-		<joint name="filter-kinect" type="fixed">
-			<parent link="filter"/>
-			<child link="kinect"/>
-			<origin xyz="0.18 0 0.29" rpy="0 0 0"/>
-		</joint>
-		<joint name="base-tables" type="fixed">
-			<parent link="base_link"/>
-			<child link="tables"/>
-			<origin xyz="0.84 0 0" rpy="0 0 0"/>
-		</joint>
+  <link name="pallet">
+    <visual>
+      <geometry>
+	<box size="1.61 1.16 0.213"/>
+      </geometry>
+      <material name="">
+	<color rgba="1 0 1 1"/>
+      </material>
+    </visual>
+  </link>
+  <link name="controller">
+    <visual>
+      <geometry>
+	<box size="0.80 0.65 1.00"/>
+      </geometry>
+      <material name="">
+	<color rgba="1 0.2 1 1"/>
+      </material>
+    </visual>
+  </link>
+  <link name="filter">
+    <visual>
+      <geometry>
+	<box size="0.36 0.36 0.36"/>
+      </geometry>
+      <material name="">
+	<color rgba="1 0.4 1 1"/>
+      </material>
+    </visual>
+  </link>
+  <link name="floor">
+    <visual>
+      <geometry>
+	<box size="6 6 0.010"/>
+      </geometry>
+      <material name="">
+	<color rgba="1 0.6 1 0.5"/>
+      </material>
+    </visual>
+  </link>
+  <link name="kinect">
+    <visual>
+      <geometry>
+	<box size="0.36 0.28 0.22"/>
+      </geometry>
+      <material name="">
+	<color rgba="1 0.8 1 1"/>
+      </material>
+    </visual>
+  </link>
+  <link name="tables">
+    <visual>
+      <geometry>
+	<box size="1.10 1.65 0.45"/>
+      </geometry>
+      <material name="">
+	<color rgba="1 0.7 1 1"/>
+      </material>
+    </visual>
+  </link>
+  <joint name="base-pallet" type="fixed">
+    <parent link="base_link"/>
+    <child link="pallet"/>
+    <origin xyz="-0.52 -0.34 -0.11" rpy="0 0 0"/>
+  </joint>
+  <joint name="base-controller" type="fixed">
+    <parent link="base_link"/>
+    <child link="controller"/>
+    <origin xyz="-0.75 -0.50 0.50" rpy="0 0 0"/>
+  </joint>
+  <joint name="base-filter" type="fixed">
+    <parent link="base_link"/>
+    <child link="filter"/>
+    <origin xyz="-0.17 -0.50 0.63" rpy="0 0 0"/>
+  </joint>
+  <joint name="pallet-floor" type="fixed">
+    <parent link="pallet"/>
+    <child link="floor"/>
+    <origin xyz="0 0 -0.11" rpy="0 0 0"/>
+  </joint>
+  <joint name="filter-kinect" type="fixed">
+    <parent link="filter"/>
+    <child link="kinect"/>
+    <origin xyz="0.18 0 0.29" rpy="0 0 0"/>
+  </joint>
+  <joint name="base-tables" type="fixed">
+    <parent link="base_link"/>
+    <child link="tables"/>
+    <origin xyz="0.84 0 0" rpy="0 0 0"/>
+  </joint>
   <!-- end environment list -->
   <!-- kinect -->
-		<joint name="kinect_frame_joint" type="fixed">
-			<parent link="kinect"/>
-			<child link="kinect_frame"/>
-			<origin rpy="0.075 0.351422870712 0.396594014755" xyz="-0.12481258247 0.064659133914 -0.022541275619"/>
-		</joint>
-		<link name="kinect_frame">
-			<visual>
-				<origin rpy="0 0 0" xyz="0 0 0"/>
-				<geometry>
-					<box size="0.064 0.28 0.04"/>
-				</geometry>
-				<material name="silver"/>
-			</visual>
-			<collision>
-				<origin rpy="0 0 0" xyz="0 0 0"/>
-				<geometry>
-					<box size="0.064 0.28 0.04"/>
-				</geometry>
-			</collision>
-		</link>
-		<joint name="kinect_ir_joint" type="fixed">
-			<parent link="kinect_frame"/>
-			<child link="kinect_ir_link"/>
-			<origin rpy="0 0 0" xyz="0 0 0"/>
-		</joint>
-		<link name="kinect_ir_link">
-			<visual>
-				<origin rpy="0 0 0" xyz="0 0 0"/>
-				<geometry>
-					<sphere radius="0.0005"/>
-				</geometry>
-			</visual>
-		</link>
-		<joint name="kinect_ir_optical_frame_joint" type="fixed">
-			<parent link="kinect_ir_link"/>
-			<child link="kinect_ir_optical_frame"/>
-			<origin rpy="-1.57 0 -1.57" xyz="0 0 0"/>
-		</joint>
-		<link name="kinect_ir_optical_frame"/>
-		<joint name="kinect_rgb_joint" type="fixed">
-			<parent link="kinect_ir_link"/>
-			<child link="kinect_rgb_link"/>
-			<origin rpy="0 0 0" xyz="0 -0.03 0"/>
-		</joint>
-		<link name="kinect_rgb_link">
-			<visual>
-				<origin rpy="0 0 0" xyz="0 0 0"/>
-				<geometry>
-					<sphere radius="0.0005"/>
-				</geometry>
-			</visual>
-		</link>
-		<joint name="kinect_rgb_optical_frame_joint" type="fixed">
-			<parent link="kinect_rgb_link"/>
-			<child link="kinect_rgb_optical_frame"/>
-			<origin rpy="-1.57 0 -1.57" xyz="0 0 0"/>
-		</joint>
-		<link name="kinect_rgb_optical_frame"/>
+  <joint name="kinect_frame_joint" type="fixed">
+    <parent link="kinect"/>
+    <child link="kinect_frame"/>
+    <origin rpy="0.075 0.351422870712 0.396594014755" xyz="-0.12481258247 0.064659133914 -0.022541275619"/>
+  </joint>
+  <link name="kinect_frame">
+    <visual>
+      <origin rpy="0 0 0" xyz="0 0 0"/>
+      <geometry>
+	<box size="0.064 0.28 0.04"/>
+      </geometry>
+      <material name="silver"/>
+    </visual>
+    <collision>
+      <origin rpy="0 0 0" xyz="0 0 0"/>
+      <geometry>
+	<box size="0.064 0.28 0.04"/>
+      </geometry>
+    </collision>
+  </link>
+  <joint name="kinect_ir_joint" type="fixed">
+    <parent link="kinect_frame"/>
+    <child link="kinect_ir_link"/>
+    <origin rpy="0 0 0" xyz="0 0 0"/>
+  </joint>
+  <link name="kinect_ir_link">
+    <visual>
+      <origin rpy="0 0 0" xyz="0 0 0"/>
+      <geometry>
+	<sphere radius="0.0005"/>
+      </geometry>
+    </visual>
+  </link>
+  <joint name="kinect_ir_optical_frame_joint" type="fixed">
+    <parent link="kinect_ir_link"/>
+    <child link="kinect_ir_optical_frame"/>
+    <origin rpy="-1.57 0 -1.57" xyz="0 0 0"/>
+  </joint>
+  <link name="kinect_ir_optical_frame"/>
+  <joint name="kinect_rgb_joint" type="fixed">
+    <parent link="kinect_ir_link"/>
+    <child link="kinect_rgb_link"/>
+    <origin rpy="0 0 0" xyz="0 -0.03 0"/>
+  </joint>
+  <link name="kinect_rgb_link">
+    <visual>
+      <origin rpy="0 0 0" xyz="0 0 0"/>
+      <geometry>
+	<sphere radius="0.0005"/>
+      </geometry>
+    </visual>
+  </link>
+  <joint name="kinect_rgb_optical_frame_joint" type="fixed">
+    <parent link="kinect_rgb_link"/>
+    <child link="kinect_rgb_optical_frame"/>
+    <origin rpy="-1.57 0 -1.57" xyz="0 0 0"/>
+  </joint>
+  <link name="kinect_rgb_optical_frame"/>
   <!-- end kinect -->
 </robot>

File: branches/moveit_industrial/robotiq/cfg/s-model_articulated_macro.xacro (robot description, xacro)
@@ -6,53 +6,53 @@
 -->
 <robot xmlns:xacro="http://ros.org/wiki/xacro">
-	<include filename="$(find robotiq)/cfg/s-model_finger_articulated_macro.xacro" />
-	<xacro:macro name="s-model_articulated" params="prefix">
-	<xacro:s-model_finger_articulated prefix="${prefix}finger_1_"/>
-	<xacro:s-model_finger_articulated prefix="${prefix}finger_2_"/>
-	<xacro:s-model_finger_articulated prefix="${prefix}finger_middle_"/>
-		<!-- link list -->
-		<link name="${prefix}palm">
-			<visual>
-				<geometry>
-					<mesh filename="package://robotiq/meshes/s-model_articulated/visual/palm.STL" />
-				</geometry>
-				<material name="green">
-					<color rgba="0 1 0 1"/>
-				</material>
-			</visual>
-			<collision>
-				<geometry>
-					<mesh filename="package://robotiq/meshes/s-model_articulated/collision/palm.STL" />
-				</geometry>
-				<material name="yellow">
-					<color rgba="0 1 1 1"/>
-				</material>
-			</collision>
-		</link>
-		<!-- end of link list -->
-		<!-- joint list -->
-		<!-- WARNING: LIMITS NOT CORRECT -->
-		<joint name="${prefix}palm_finger_1_joint" type="revolute">
-			<parent link="${prefix}palm"/>
-			<child link="${prefix}finger_1_link_0"/>
-			<axis xyz="0 1 0"/>
-			<origin xyz="-0.0455 0.0214 0.036" rpy="0 3.1416 -1.57"/>
-			<limit lower="-0.16" upper="0.25" effort="100" velocity="100"/>
-		</joint>
-		<!-- WARNING: LIMITS NOT CORRECT -->
-		<joint name="${prefix}palm_finger_2_joint" type="revolute">
-			<parent link="${prefix}palm"/>
-			<child link="${prefix}finger_2_link_0"/>
-			<axis xyz="0 1 0"/>
-			<origin xyz="-0.0455 0.0214 -0.036" rpy="0 3.1416 -1.57"/>
-			<limit lower="-0.25" upper="0.16" effort="100" velocity="100"/>
-		</joint>
-		<joint name="${prefix}palm_finger_middle_joint" type="fixed">
-			<parent link="${prefix}palm"/>
-			<child link="${prefix}finger_middle_link_0"/>
-			<axis xyz="0 0 1"/>
-			<origin xyz="0.0455 0.0214 0" rpy="0 0 1.57"/>
-		</joint>
-		<!-- end of joint list -->
-	</xacro:macro>
+  <include filename="$(find robotiq)/cfg/s-model_finger_articulated_macro.xacro" />
+  <xacro:macro name="s-model_articulated" params="prefix">
+    <xacro:s-model_finger_articulated prefix="${prefix}finger_0_"/>
+    <xacro:s-model_finger_articulated prefix="${prefix}finger_1_"/>
+    <xacro:s-model_finger_articulated prefix="${prefix}finger_2_"/>
+    <!-- link list -->
+    <link name="${prefix}palm">
+      <visual>
+	<geometry>
+	  <mesh filename="package://robotiq/meshes/s-model_articulated/visual/palm.STL" />
+	</geometry>
+	<material name="green">
+	  <color rgba="0 1 0 1"/>
+	</material>
+      </visual>
+      <collision>
+	<geometry>
+	  <mesh filename="package://robotiq/meshes/s-model_articulated/collision/palm.STL" />
+	</geometry>
+	<material name="yellow">
+	  <color rgba="0 1 1 1"/>
+	</material>
+      </collision>
+    </link>
+    <!-- end of link list -->
+    <!-- joint list -->
+    <!-- WARNING: LIMITS NOT CORRECT -->
+    <joint name="${prefix}palm_finger_1_joint" type="revolute">
+      <parent link="${prefix}palm"/>
+      <child link="${prefix}finger_1_link_0"/>
+      <axis xyz="0 1 0"/>
+      <origin xyz="-0.0455 0.0214 0.036" rpy="0 3.1416 -1.57"/>
+      <limit lower="-0.16" upper="0.25" effort="100" velocity="100"/>
+    </joint>
+    <!-- WARNING: LIMITS NOT CORRECT -->
+    <joint name="${prefix}palm_finger_2_joint" type="revolute">
+      <parent link="${prefix}palm"/>
+      <child link="${prefix}finger_2_link_0"/>
+      <axis xyz="0 1 0"/>
+      <origin xyz="-0.0455 0.0214 -0.036" rpy="0 3.1416 -1.57"/>
+      <limit lower="-0.25" upper="0.16" effort="100" velocity="100"/>
+    </joint>
+    <joint name="${prefix}palm_finger_0_joint" type="fixed">
+      <parent link="${prefix}palm"/>
+      <child link="${prefix}finger_0_link_0"/>
+      <axis xyz="0 0 1"/>
+      <origin xyz="0.0455 0.0214 0" rpy="0 0 1.57"/>
+    </joint>
+    <!-- end of joint list -->
+  </xacro:macro>
 </robot>
