Commit message: More configurations for sia10d mounts with and without the RobotIQ hand

File: branches/moveit_industrial/armadillo/cfg/armadillo.urdf (robot description, URDF)
Before this commit: robot armadillo, 33 links, 32 joints
Links:
- removed link controller
- removed link filter
- removed link tables

File: branches/moveit_industrial/armadillo/cfg/armadillo.xacro (robot description, xacro)
@@ -2,39 +2,5 @@
 <robot name="armadillo" xmlns:xacro="http://ros.org/wiki/xacro">
   <include filename="$(find motoman)/cfg/sia10d_mesh_macro.xacro" />
-  <include filename="$(find robotiq)/cfg/s-model_articulated_macro.xacro" />
   <xacro:sia10d_mesh prefix=""/>
-  <xacro:s-model_articulated prefix=""/>
-  <!-- link list -->
-  <link name="coupler">
-    <visual>
-      <geometry>
-	<mesh filename="package://armadillo/meshes/coupler/visual/COUPLER.stl" />
-      </geometry>
-      <material name="orange">
-	<color rgba="1 0.5 0 1"/>
-      </material>
-    </visual>
-    <collision>
-      <geometry>
-	<mesh filename="package://armadillo/meshes/coupler/collision/COUPLER.stl" />
-      </geometry>
-      <material name="yellow">
-	<color rgba="0 1 1 1"/>
-      </material>
-    </collision>
-  </link>
-  <!-- end link list -->
-  <!-- joint list -->
-  <joint name="tool-coupler" type="fixed">
-    <parent link="link_t"/>
-    <child link="coupler"/>
-    <origin xyz="0 0 0" rpy="1.570 0 0"/>
-  </joint>
-  <joint name="coupler-hand" type="fixed">
-    <parent link="coupler"/>
-    <child link="palm"/>
-    <origin xyz="0 0.120 0" rpy="0 0 0"/>
-  </joint>
-  <!-- end of joint list -->
   <!-- environment list -->
   <link name="pallet">
@@ -45,24 +11,4 @@
       <material name="">
 	<color rgba="1 0 1 1"/>
-      </material>
-    </visual>
-  </link>
-  <link name="controller">
-    <visual>
-      <geometry>
-	<box size="0.80 0.65 1.00"/>
-      </geometry>
-      <material name="">
-	<color rgba="1 0.2 1 1"/>
-      </material>
-    </visual>
-  </link>
-  <link name="filter">
-    <visual>
-      <geometry>
-	<box size="0.36 0.36 0.36"/>
-      </geometry>
-      <material name="">
-	<color rgba="1 0.4 1 1"/>
       </material>
     </visual>
@@ -78,38 +24,8 @@
     </visual>
   </link>
-  <link name="kinect">
-    <visual>
-      <geometry>
-	<box size="0.36 0.28 0.22"/>
-      </geometry>
-      <material name="">
-	<color rgba="1 0.8 1 1"/>
-      </material>
-    </visual>
-  </link>
-  <link name="tables">
-    <visual>
-      <geometry>
-	<box size="1.10 1.65 0.45"/>
-      </geometry>
-      <material name="">
-	<color rgba="1 0.7 1 1"/>
-      </material>
-    </visual>
-  </link>
   <joint name="base-pallet" type="fixed">
     <parent link="base_link"/>
     <child link="pallet"/>
     <origin xyz="-0.52 -0.34 -0.11" rpy="0 0 0"/>
-  </joint>
-  <joint name="base-controller" type="fixed">
-    <parent link="base_link"/>
-    <child link="controller"/>
-    <origin xyz="-0.75 -0.50 0.50" rpy="0 0 0"/>
-  </joint>
-  <joint name="base-filter" type="fixed">
-    <parent link="base_link"/>
-    <child link="filter"/>
-    <origin xyz="-0.17 -0.50 0.63" rpy="0 0 0"/>
   </joint>
   <joint name="pallet-floor" type="fixed">
@@ -118,74 +34,3 @@
     <origin xyz="0 0 -0.11" rpy="0 0 0"/>
   </joint>
-  <joint name="filter-kinect" type="fixed">
-    <parent link="filter"/>
-    <child link="kinect"/>
-    <origin xyz="0.18 0 0.29" rpy="0 0 0"/>
-  </joint>
-  <joint name="base-tables" type="fixed">
-    <parent link="base_link"/>
-    <child link="tables"/>
-    <origin xyz="0.84 0 0" rpy="0 0 0"/>
-  </joint>
-  <!-- end environment list -->
-  <!-- kinect -->
-  <joint name="kinect_frame_joint" type="fixed">
-    <parent link="kinect"/>
-    <child link="kinect_frame"/>
-    <origin rpy="0.075 0.351422870712 0.396594014755" xyz="-0.12481258247 0.064659133914 -0.022541275619"/>
-  </joint>
-  <link name="kinect_frame">
-    <visual>
-      <origin rpy="0 0 0" xyz="0 0 0"/>
-      <geometry>
-	<box size="0.064 0.28 0.04"/>
-      </geometry>
-      <material name="silver"/>
-    </visual>
-    <collision>
-      <origin rpy="0 0 0" xyz="0 0 0"/>
-      <geometry>
-	<box size="0.064 0.28 0.04"/>
-      </geometry>
-    </collision>
-  </link>
-  <joint name="kinect_ir_joint" type="fixed">
-    <parent link="kinect_frame"/>
-    <child link="kinect_ir_link"/>
-    <origin rpy="0 0 0" xyz="0 0 0"/>
-  </joint>
-  <link name="kinect_ir_link">
-    <visual>
-      <origin rpy="0 0 0" xyz="0 0 0"/>
-      <geometry>
-	<sphere radius="0.0005"/>
-      </geometry>
-    </visual>
-  </link>
-  <joint name="kinect_ir_optical_frame_joint" type="fixed">
-    <parent link="kinect_ir_link"/>
-    <child link="kinect_ir_optical_frame"/>
-    <origin rpy="-1.57 0 -1.57" xyz="0 0 0"/>
-  </joint>
-  <link name="kinect_ir_optical_frame"/>
-  <joint name="kinect_rgb_joint" type="fixed">
-    <parent link="kinect_ir_link"/>
-    <child link="kinect_rgb_link"/>
-    <origin rpy="0 0 0" xyz="0 -0.03 0"/>
-  </joint>
-  <link name="kinect_rgb_link">
-    <visual>
-      <origin rpy="0 0 0" xyz="0 0 0"/>
-      <geometry>
-	<sphere radius="0.0005"/>
-      </geometry>
-    </visual>
-  </link>
-  <joint name="kinect_rgb_optical_frame_joint" type="fixed">
-    <parent link="kinect_rgb_link"/>
-    <child link="kinect_rgb_optical_frame"/>
-    <origin rpy="-1.57 0 -1.57" xyz="0 0 0"/>
-  </joint>
-  <link name="kinect_rgb_optical_frame"/>
-  <!-- end kinect -->
 </robot>
