Commit message: Changed kinect frame to adjust point cloud data to table top, specifically the urdf file and teh "base-kinect" joint orientation

File: trunk/freetail/freetail_config/urdf/freetail.urdf (robot description, URDF)
Before this commit: robot freetail, 25 links, 24 joints
Joints:
- joint base-kinect: origin xyz=1.26 -0.72 0.75 rpy=0 0 2.356 -> xyz=1.08 -0.72 0.82 rpy=0 0.5235 2.356

Commit message: test_recognition node is functional, made changes to freetail.urdf, xacro to use new robotiq model package path

File: trunk/freetail/freetail_config/urdf/freetail.urdf (robot description, URDF)
Before this commit: robot freetail, 25 links, 24 joints
Links:
- link finger_1: geometry collision mesh filename=package://robotiq_s_model_visualization/meshes/s-model/coll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; visual mesh filename=package://robotiq_s_model_visualization/meshes/s-model/visu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
- link finger_2: geometry collision mesh filename=package://robotiq_s_model_visualization/meshes/s-model/coll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; visual mesh filename=package://robotiq_s_model_visualization/meshes/s-model/visu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
- link finger_3: geometry collision mesh filename=package://robotiq_s_model_visualization/meshes/s-model/coll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; visual mesh filename=package://robotiq_s_model_visualization/meshes/s-model/visu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
- link palm: geometry collision mesh filename=package://robotiq_s_model_visualization/meshes/s-model/coll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; visual mesh filename=package://robotiq_s_model_visualization/meshes/s-model/visu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
Joints:
- joint base-kinect: origin xyz=1.08 -0.72 0.82 rpy=0 0.5235 2.356 -> xyz=1.26 -0.72 0.75 rpy=0 0 2.356

File: trunk/freetail/freetail_config/urdf/freetail.xacro (robot description, xacro)
@@ -2,5 +2,5 @@
 <robot name="freetail" xmlns:xacro="http://ros.org/wiki/xacro">
 	<include filename="$(find motoman_config)/cfg/sia20d_mesh_macro.xacro" />
-	<include filename="$(find robotiq)/cfg/s-model_mesh_macro.xacro" />
+	<include filename="$(find robotiq_s_model_visualization)/cfg/s-model_mesh_macro.xacro" />
 	<xacro:sia20d_mesh prefix=""/>
 	<xacro:s-model_mesh prefix=""/>

Commit message: Modified freetail.xacro to fix issue with the misaligned point cloud, object recognition fails to return object refence

File: trunk/freetail/freetail_config/urdf/freetail.urdf (robot description, URDF)
Before this commit: robot freetail, 25 links, 24 joints
Joints:
- joint base-kinect: origin xyz=1.26 -0.72 0.75 rpy=0 0 2.356 -> xyz=1.08 -0.72 0.82 rpy=0 0.5235 2.356

File: trunk/freetail/freetail_config/urdf/freetail.xacro (robot description, xacro)
@@ -132,5 +132,5 @@
 			<parent link="base_link"/>
 			<child link="kinect"/>
-			<origin xyz="1.26 -0.72 0.75" rpy="0 0 2.356"/>
+			<origin rpy="0 0.5235 2.356" xyz="1.08 -0.72 0.82"/>
 		</joint>
 		<joint name="table-keepout_1" type="fixed">
