Commit message: vacuum gripper simulation demo is functional, needs to put a urdf for the vacuum gripper, using a bounding box for now instead

File: trunk/freetail/freetail_config/urdf/freetail_vacuum_gripper_conf.urdf (robot description, URDF)
Before this commit: robot freetail, 22 links, 21 joints
Links:
- link palm: geometry collision box size=0.040 0.080 0.1086; visual box size=0.040 0.080 0.1086
Joints:
- joint coupler-hand: origin xyz=0 0.019 0.196 rpy=0 0 0 -> xyz=0 0.196 0.019 rpy=-1.570 0 0

File: trunk/freetail/freetail_config/urdf/freetail_vacuum_gripper_conf.xacro (robot description, xacro)
@@ -34,5 +34,5 @@
 		<parent link="coupler"/>
 		<child link="palm"/>
-		<origin xyz="0 0.019 0.196" rpy="0 0 0"/>
+		<origin xyz="0 0.196 0.019" rpy="-1.570 0 0"/>
 	</joint>
   <!-- environment list -->

File: trunk/freetail/freetail_config/urdf/vacuum_gripper.xacro (robot description, xacro)
@@ -4,18 +4,18 @@
 		<link name="${prefix}palm">
 			<visual>
-				<origin xyz="0 0 -0.0543" rpy="0 0 0"/>
+				<origin xyz="0 0.019 -0.0543" rpy="0 0 0"/>
 				<geometry>
-					<box size="0.020 0.040 0.1086"/>
+					<box size="0.040 0.080 0.1086"/>
 				</geometry>
-				<material name="blue">
-					<color rgba="0 0 1 1"/>
+				<material name="another_blue1">
+					<color rgba="0.40 0.40 0.80 1"/>
 				</material>
 			</visual>
 			<collision>
-				<origin xyz="0 0 -0.0543" rpy="0 0 0"/>
+				<origin xyz="0 0.019 -0.0543" rpy="0 0 0"/>
 				<geometry>
-					<box size="0.020 0.040 0.1086"/>
+					<box size="0.040 0.080 0.1086"/>
 				</geometry>
-				<material name="blue">
+				<material name="another_blue2">
 					<color rgba="0.38 0.54 0.83 1"/>
 				</material>
