Commit message: modified mantis__ur5_planning_environment groups in order to ommit gripper links during grasp collsion cchecks

File: trunk/mantis/mantis_config/urdf/mantis_ur5.urdf (robot description, URDF)
Before this commit: robot mantis_ur5, 27 links, 26 joints
Links:
- link ur5_arm_kinect_keepout: geometry collision box size=0.2 0.32 0.7
- link ur5_stand: geometry collision cylinder length=0.2 radius=0.0735; visual cylinder length=0.2 radius=0.0735
Joints:
- joint ur5_arm_ur5_arm_base_link_to_kinect: origin xyz=1.08 -0.72 0.82 rpy=0 0.5235 2.536 -> xyz=1.08 -0.72 0.62 rpy=0 0.5235 2.536
- joint ur5_arm_ur5_arm_base_link_to_kinect_keepout: origin xyz=1.08 -0.72 0.45 rpy=0 0 2.536 -> xyz=1.08 -0.72 0.35 rpy=0 0 2.536
