Commit message: Added launch files for ur5 manipulation

File: trunk/mantis/mantis_config/urdf/mantis_sia20d.urdf (robot description, URDF)
Before this commit: robot mantis_sia20d, 23 links, 22 joints
Links:
- link sia20d_arm_palm: geometry collision mesh filename=package://mantis_config/config/meshes/vacuum_gripper.stl; visual mesh filename=package://mantis_config/config/meshes/vacuum_gripper.STL

File: trunk/mantis/mantis_config/urdf/mantis_ur5.urdf (robot description, URDF)
Before this commit: robot mantis_ur5, 27 links, 26 joints
Links:
- link ur5_arm_forearm_link: geometry collision mesh filename=package://ur5_description/meshes/collision/Forearm.dae; visual mesh filename=package://ur5_description/meshes/Forearm.dae
- link ur5_arm_gripper_body: geometry collision box size=0.044 0.088 0.0946; visual mesh filename=package://mantis_config/config/meshes/vacuum_gripper.STL
- link ur5_arm_kinect_keepout: geometry collision box size=0.2 0.32 0.9
- link ur5_arm_shoulder_link: geometry collision mesh filename=package://ur5_description/meshes/collision/Shoulder.dae; visual mesh filename=package://ur5_description/meshes/Shoulder.dae
- link ur5_arm_upper_arm_link: geometry collision mesh filename=package://ur5_description/meshes/collision/UpperArm.dae; visual mesh filename=package://ur5_description/meshes/UpperArm.dae
- link ur5_arm_wrist_1_link: geometry collision mesh filename=package://ur5_description/meshes/collision/Wrist1.dae; visual mesh filename=package://ur5_description/meshes/Wrist1.dae
- link ur5_arm_wrist_2_link: geometry collision mesh filename=package://ur5_description/meshes/collision/Wrist2.dae; visual mesh filename=package://ur5_description/meshes/Wrist2.dae
- link ur5_arm_wrist_3_link: geometry collision mesh filename=package://ur5_description/meshes/collision/Wrist3.dae; visual mesh filename=package://ur5_description/meshes/Wrist3.dae
Joints:
- removed joint ur5_arm_workcell_frame_to_kinect
- removed joint ur5_arm_workcell_frame_to_kinect_keepout
- removed joint ur5_to_gripper
- added joint ur5_arm_to_gripper: type fixed, parent ur5_arm_ee_link, child ur5_arm_gripper_frame, origin xyz=0 0 0 rpy=0 1.57 0
- added joint ur5_arm_ur5_arm_base_link_to_kinect: type fixed, parent ur5_arm_base_link, child ur5_arm_kinect, origin xyz=1.08 -0.72 0.82 rpy=0 0.5235 2.536
- added joint ur5_arm_ur5_arm_base_link_to_kinect_keepout: type fixed, parent ur5_arm_base_link, child ur5_arm_kinect_keepout, origin xyz=1.08 -0.72 0.45 rpy=0 0 2.536
- joint ur5_arm_elbow_joint: axis 0.0 1.0 0.0 -> 0 1 0
- joint ur5_arm_gripper_to_tcp: origin xyz=0.022 0 0.0946 rpy=0 0 0 -> xyz= 0 0.022 0.0946 rpy=0 0 0
- joint ur5_arm_shoulder_lift_joint: axis 0.0 1.0 0.0 -> 0 1 0
- joint ur5_arm_shoulder_pan_joint: axis 0.0 0.0 1.0 -> 0 0 1
- joint ur5_arm_wrist_1_joint: axis 0.0 1.0 0.0 -> 0 1 0
- joint ur5_arm_wrist_2_joint: axis 0.0 0.0 1.0 -> 0 0 1
- joint ur5_arm_wrist_3_joint: axis 0.0 1.0 0.0 -> 0 1 0

File: trunk/mantis/mantis_config/urdf/mantis_ur5_arm_workspace.xacro (robot description, xacro)
@@ -8,4 +8,5 @@
 	<!-- property list -->
 	<xacro:property name="workcell_height" value="1"/>
+	<xacro:property name="robot_stand_height" value="0.20"/>
 	<xacro:property name="vacuum_gripper_width" value="0.088"/>
 	<xacro:property name="arm2_prefix" value="ur5_arm_"/>
@@ -18,6 +19,6 @@
 	<!-- end of workcell definitions -->
 	<!-- instantiating sensor definitions -->
-	<xacro:sensor_definitions prefix="${arm2_prefix}" parent_link="workcell_frame"
-		x_val="-1.20" y_val="0" z_val="0.4" pitch="0.5235" yaw="0"/>
+	<xacro:sensor_definitions prefix="${arm2_prefix}" parent_link="${arm2_prefix}base_link"
+		x_val="1.08" y_val="-0.72" z_val="${0.82 - robot_stand_height}" pitch="0.5235" yaw="2.536"/>
 	<!-- end of sensor definitions -->
 	<!-- arm-workcell link definitions -->
@@ -25,5 +26,5 @@
 		<visual>
 			<geometry>
-				<cylinder radius="0.0735" length="0.20"/>
+				<cylinder radius="0.0735" length="${robot_stand_height}"/>
 			</geometry>
 			<material name="orange_transparent"/>
@@ -31,5 +32,5 @@
 		<collision>
 			<geometry>
-				<cylinder radius="0.0735" length="0.20"/>
+				<cylinder radius="0.0735" length="${robot_stand_height}"/>
 			</geometry>
 			<material name="blue_transparent"/>
@@ -50,5 +51,5 @@
 	<!-- end of arm workcell joint definitions-->
 	<!-- arm-gripper coupling joint definitions -->
-	<joint name="${arm2_name}_to_gripper" type="fixed">
+	<joint name="${arm2_prefix}to_gripper" type="fixed">
 		<parent link="${arm2_prefix}ee_link"/>
 		<child link="${arm2_prefix}gripper_frame"/>

File: trunk/mantis/mantis_config/urdf/vacuum_gripper_macro.xacro (robot description, xacro)
@@ -9,5 +9,9 @@
 		<link name="${prefix}gripper_body">
 			<visual>
-				<origin xyz="0 0.036 -0.1" rpy="0 0 0"/>
+				<!--origin xyz="0 0.036 -0.0473" rpy="0 0 0"/-->
+				<!--geometry>
+					<box size="${gripper_length} ${gripper_width} ${gripper_height}"/>
+				</geometry-->
+				<origin xyz="0 0 -0.048" rpy="0 0 0"/>
 				<geometry>
 					<mesh filename="package://mantis_config/config/meshes/vacuum_gripper.STL" />
@@ -18,5 +22,4 @@
 			</visual>
 			<collision>
-				<origin xyz="0 0.036 -0.0473" rpy="0 0 0"/>
 				<geometry>
 					<box size="${gripper_length} ${gripper_width} ${gripper_height}"/>
@@ -36,5 +39,5 @@
 			<parent link="${prefix}gripper_frame"/>
 			<child link="${prefix}tcp_frame"/>
-			<origin xyz="${gripper_length * 0.5} 0 ${gripper_height}" rpy="0 0 0"/>
+			<origin xyz=" 0 ${gripper_length * 0.5} ${gripper_height}" rpy="0 0 0"/>
 		</joint>
 	</xacro:macro>

Commit message: sia20d xacro uses the gripper definition in vacuum_xacro_macro

File: trunk/mantis/mantis_config/urdf/mantis_sia20d.urdf (robot description, URDF)
Before this commit: robot mantis_sia20d, 23 links, 22 joints
Links:
- removed link sia20d_arm_kinect
- removed link sia20d_arm_palm
- added link sia20d_arm_gripper_body; collision box size=0.044 0.088 0.0946; visual mesh filename=package://mantis_config/config/meshes/vacuum_gripper.STL
- added link sia20d_arm_gripper_frame
- added link sia20d_arm_kinect_link; collision box size=0.36 0.28 0.22
- added link sia20d_arm_tcp_frame
Joints:
- removed joint coupler-hand
- removed joint sia20d_arm_sia20d_arm_base_link_to_kinect
- removed joint tool-coupler
- added joint sia20d_arm_coupler_to_hand: type fixed, parent sia20d_arm_coupler, child sia20d_arm_gripper_frame, origin xyz=0 0.087 0 rpy=-1.570 0 0
- added joint sia20d_arm_gripper_to_palm: type fixed, parent sia20d_arm_gripper_frame, child sia20d_arm_gripper_body, origin xyz=0 0 0.0473 rpy=0 0 0
- added joint sia20d_arm_gripper_to_tcp: type fixed, parent sia20d_arm_gripper_frame, child sia20d_arm_tcp_frame, origin xyz= 0 0.022 0.0946 rpy=0 0 0
- added joint sia20d_arm_sia20d_arm_base_link_to_kinect_link: type fixed, parent sia20d_arm_base_link, child sia20d_arm_kinect_link, origin xyz=1.08 -0.72 0.82 rpy=0 0.5235 2.356
- added joint sia20d_arm_tool_to_coupler: type fixed, parent sia20d_arm_link_t, child sia20d_arm_coupler, origin xyz=0 0 0 rpy=1.570 0 -0.785
- joint sia20d_arm_kinect_frame_joint: parent sia20d_arm_kinect -> sia20d_arm_kinect_link

File: trunk/mantis/mantis_config/urdf/mantis_sia20d_arm_workspace.xacro (robot description, xacro)
@@ -2,5 +2,5 @@
 <robot name="mantis_sia20d" xmlns:xacro="http://ros.org/wiki/xacro">
 	<include filename="$(find mantis_config)/urdf/sia20d_mesh_macro.xacro"/>
-	<include filename="$(find mantis_config)/urdf/vacuum_gripper.xacro"/>
+	<!--include filename="$(find mantis_config)/urdf/vacuum_gripper.xacro"/-->
 	<include filename="$(find mantis_config)/urdf/vacuum_gripper_macro.xacro"/>
 	<include filename="$(find mantis_config)/urdf/mantis_workspace_components.xacro"/>
@@ -8,28 +8,29 @@
 	<!-- property list -->
 	<xacro:property name="workcell_height" value="1"/>
-	<xacro:property name="vacuum_gripper_width" value="0.088"/>
-	<xacro:property name="arm1_prefix" value="sia20d_arm_"/>
-	<xacro:property name="arm1_name" value="sia20d"/>
+	<xacro:property name="coupler_height" value="0.087"/>
+	<xacro:property name="arm_prefix" value="sia20d_arm_"/>
+	<xacro:property name="arm_name" value="sia20d"/>
+	<xacro:property name="coupler_height" value="0.087"/>
 	<!-- instantiating workcell definitions -->
 	<xacro:workcell_zone1_components/>
 	<!-- end of workcell definitions -->
 	<!-- instantiating sensor definitions -->
-	<!--xacro:sensor_definitions prefix="${arm1_prefix}" parent_link="workcell_frame"
+	<!--xacro:sensor_definitions prefix="${arm_prefix}" parent_link="workcell_frame"
 		x_val="1.20" y_val="0" z_val="0.4" pitch="0.5235" yaw="3.147"/-->
-	<xacro:sensor_definitions prefix="${arm1_prefix}" parent_link="${arm1_prefix}base_link"
+	<xacro:sensor_definitions prefix="${arm_prefix}" parent_link="${arm_prefix}base_link"
 		x_val="1.08" y_val="-0.72" z_val="0.82" pitch="0.5235" yaw="2.356"/>
 	<!-- end of sensor definitions -->
 	<!-- instantiating arm and gripper -->
-	<xacro:vacuum_gripper prefix="${arm1_prefix}"/>
-	<xacro:sia20d_mesh prefix="${arm1_prefix}"/>
+	<xacro:vacuum_gripper_definition prefix="${arm_prefix}"/>
+	<xacro:sia20d_mesh prefix="${arm_prefix}"/>
 	<!-- arm-workcell joint definitions -->
-	<joint name="${arm1_name}_to_workcell" type="fixed">
+	<joint name="${arm_name}_to_workcell" type="fixed">
 		<parent link="workcell_frame"/>
-		<child link="${arm1_prefix}base_link"/>
+		<child link="${arm_prefix}base_link"/>
 		<origin xyz="0.241 0 0" rpy="0 0 0"/>
 	</joint>
 	<!-- end of arm workcell joint definitions-->
 	<!-- arm-gripper coupling link definitions-->
-	<link name="${arm1_prefix}coupler">
+	<link name="${arm_prefix}coupler">
 		<visual>
 			<geometry>
@@ -51,13 +52,17 @@
 	<!-- end of arm-gripper coupling link definitions -->
 	<!-- arm-gripper coupling joint definitions -->
-	<joint name="tool-coupler" type="fixed">
-		<parent link="${arm1_prefix}link_t"/>
-		<child link="${arm1_prefix}coupler"/>
+	<!--joint name="tool-coupler" type="fixed"-->
+	<joint name="${arm_prefix}wrist_to_coupler" type="fixed">
+		<parent link="${arm_prefix}link_t"/>
+		<child link="${arm_prefix}coupler"/>
 		<origin xyz="0 0 0" rpy="1.570 0 -0.785"/>
 	</joint>
-	<joint name="coupler-hand" type="fixed">
-		<parent link="${arm1_prefix}coupler"/>
-		<child link="${arm1_prefix}palm"/>
-		<origin xyz="0 0.182 0.036" rpy="-1.570 0 0"/>
+	<!--joint name="coupler-hand" type="fixed"-->
+	<joint name="${arm_prefix}coupler_to_gripper" type="fixed">
+		<parent link="${arm_prefix}coupler"/>
+		<child link="${arm_prefix}gripper_frame"/>
+		<!--child link="${arm_prefix}palm"/-->
+		<origin xyz="0 ${coupler_height} 0" rpy="-1.570 0 0"/>
+		<!--origin xyz="0 0.182 0.036" rpy="-1.570 0 0"/-->
 	</joint>
 	<!-- end of arm-gripper coupling joint definitions -->
