Commit message: added option for using gui with joints to adjust "kinect" camera xyz, rpy. Changed macro.xacro to include visual model.

File: trunk/mantis/mantis_config/urdf/mantis_asus.urdf (robot description, URDF)
Before this commit: robot motoman_vacumm, 21 links, 20 joints
Joints:
- joint base-kinect: origin xyz=1.14 -0.055 1.5 rpy=0 1.25 3.13 -> xyz=1.16 -0.01 1.49 rpy=0.06 1.27 3.16
- joint kinect_ir_optical_frame_joint: axis (none) -> 1 0 0; limit (none) -> lower=-1 upper=1 effort=100 velocity=3.48; type fixed -> revolute

File: trunk/mantis/mantis_config/urdf/vacuum_gripper_macro.xacro (robot description, xacro)
@@ -9,13 +9,14 @@
 		<link name="${prefix}gripper_body">
 			<visual>
-				<!--origin xyz="0 0.036 -0.0473" rpy="0 0 0"/-->
+				<origin xyz="0 0.036 -0.1" rpy="0 0 0"/>
 				<geometry>
-					<box size="${gripper_length} ${gripper_width} ${gripper_height}"/>
+					<mesh filename="package://mantis_config/config/meshes/vacuum_gripper.STL" />
 				</geometry>
-				<material name="another_blue1">
-					<color rgba="0.40 0.40 0.80 1"/>
+				<material name="silver">
+					<color rgba="0.8 0.8 0.8 1"/>
 				</material>
 			</visual>
 			<collision>
+				<origin xyz="0 0.036 -0.0473" rpy="0 0 0"/>
 				<geometry>
 					<box size="${gripper_length} ${gripper_width} ${gripper_height}"/>

Commit message: changes made for new height of asus sensor (height changed to improve recognition results)

File: trunk/mantis/mantis_config/urdf/mantis_asus.urdf (robot description, URDF)
Before this commit: robot motoman_vacumm, 21 links, 20 joints
Joints:
- joint base-kinect: origin xyz=1.16 -0.01 1.49 rpy=0.06 1.27 3.16 -> xyz=1.15 -0.01 1.265 rpy=0.08 1.19 3.19

Commit message: Asus urdf with height change to minimum distance affordable from current configuration with not too much change to structural support of demo frame. Currently designed mounting leaves camera face about 61.2 in from tabletop. There is about 6 inches tubing that we can cut down easily and still keep the rest of the set up the same, so the camera face is currently about 55.2 in from the table top.

File: trunk/mantis/mantis_config/urdf/mantis_asus.urdf (robot description, URDF)
Before this commit: robot motoman_vacumm, 21 links, 20 joints
Joints:
- joint base-kinect: origin xyz=1.15 -0.01 1.265 rpy=0.08 1.19 3.19 -> xyz=1.15 -0.01 1.42 rpy=0.06 1.19 3.19
