Commit message: modified on of the kinect link names in order to match the frame_ids used by the point clouds published by the kinect (sensor) node

File: trunk/mantis/mantis_config/urdf/mantis_sensor_macro.xacro (robot description, xacro)
@@ -12,5 +12,5 @@
 		</material>
 		<!-- sensor main components -->
-		<link name="${prefix}kinect">
+		<link name="${prefix}kinect_link">
 			<collision>
 				<material name="${prefix}color_a"/>
@@ -66,5 +66,5 @@
 		<!-- sensor joints -->
 		<joint name="${prefix}kinect_frame_joint" type="fixed">
-			<parent link="${prefix}kinect"/>
+			<parent link="${prefix}kinect_link"/>
 			<child link="${prefix}kinect_frame"/>
 			<origin rpy="0 0 0" xyz="0 0 0"/>
@@ -92,7 +92,7 @@
 	  	<!-- end of sensor joints -->
 		<!-- world joints -->
-		<joint name="${prefix}${parent_link}_to_kinect" type="fixed">
+		<joint name="${prefix}${parent_link}_to_kinect_link" type="fixed">
 			<parent link="${parent_link}"/>
-			<child link="${prefix}kinect"/>
+			<child link="${prefix}kinect_link"/>
 			<origin xyz="${x_val} ${y_val} ${z_val}" rpy="0 ${pitch} ${yaw}"/>
 		</joint>

Commit message: added roll as parameter for joint "${prefix}${parent_link}_to_kinect_link" in mantis_sensor_macro.

File: trunk/mantis/mantis_config/urdf/mantis_sensor_macro.xacro (robot description, xacro)
@@ -1,5 +1,5 @@
 <?xml version="1.0" ?>
 <robot name="mantis_sensor" xmlns:xacro="http://ros.org/wiki/xacro">
-	<xacro:macro name="sensor_definitions" params="prefix parent_link x_val y_val z_val pitch yaw" >
+	<xacro:macro name="sensor_definitions" params="prefix parent_link x_val y_val z_val roll pitch yaw" >
 		<material name="${prefix}color_b">
 			<color rgba="0 0.8 1 0.4"/>
@@ -95,5 +95,5 @@
 			<parent link="${parent_link}"/>
 			<child link="${prefix}kinect_link"/>
-			<origin xyz="${x_val} ${y_val} ${z_val}" rpy="0 ${pitch} ${yaw}"/>
+			<origin xyz="${x_val} ${y_val} ${z_val}" rpy="${roll} ${pitch} ${yaw}"/>
 		</joint>
 		<joint name="${prefix}${parent_link}_to_kinect_keepout" type="fixed">
