Commit message: modified prefixes

File: trunk/mantis/mantis_config/urdf/mantis_ur5_arm_workspace.xacro (robot description, xacro)
@@ -40,5 +40,5 @@
 		<parent link="workcell_frame"/>
 		<child link="ur5_stand"/>
-		<origin xyz="-0.238 0 0.10"/>
+		<origin xyz="-0.238 0 ${robot_stand_height * 0.5}"/>
 	</joint>
 	<!-- end of arm-workcell link definitions -->
@@ -47,5 +47,5 @@
 		<parent link="ur5_stand"/>
 		<child link="${arm2_prefix}base_link"/>
-		<origin xyz="0 0 0.10" rpy="0 0 -3.14"/>
+		<origin xyz="0 0 ${robot_stand_height * 0.5}" rpy="0 0 -3.14"/>
 	</joint>
 	<!-- end of arm workcell joint definitions-->

Commit message: remapped recognition service names in both arm setup launch files

File: trunk/mantis/mantis_config/urdf/mantis_ur5_arm_workspace.xacro (robot description, xacro)
@@ -10,14 +10,14 @@
 	<xacro:property name="robot_stand_height" value="0.20"/>
 	<xacro:property name="vacuum_gripper_width" value="0.088"/>
-	<xacro:property name="arm2_prefix" value="ur5_arm_"/>
-	<xacro:property name="arm2_name" value="ur5"/>
+	<xacro:property name="arm_prefix" value="ur5_arm_"/>
+	<xacro:property name="arm_name" value="ur5"/>
 	<!-- instantiating arm and gripper -->
-	<xacro:ur5_robot prefix="${arm2_prefix}"/>
-	<xacro:vacuum_gripper_definition prefix="${arm2_prefix}"/>
+	<xacro:ur5_robot prefix="${arm_prefix}"/>
+	<xacro:vacuum_gripper_definition prefix="${arm_prefix}"/>
 	<!-- instantiating workcell definitions -->
 	<xacro:workcell_zone2_components/>
 	<!-- end of workcell definitions -->
 	<!-- instantiating sensor definitions -->
-	<xacro:sensor_definitions prefix="${arm2_prefix}" parent_link="${arm2_prefix}base_link"
+	<xacro:sensor_definitions prefix="${arm_prefix}" parent_link="${arm_prefix}base_link"
 		x_val="1.08" y_val="-0.72" z_val="${0.82 - robot_stand_height}" pitch="0.5235" yaw="2.536"/>
 	<!-- end of sensor definitions -->
@@ -44,14 +44,14 @@
 	<!-- end of arm-workcell link definitions -->
 	<!-- arm-workcell joint definitions -->
-	<joint name="${arm2_name}_to_stand" type="fixed">
+	<joint name="${arm_name}_to_stand" type="fixed">
 		<parent link="ur5_stand"/>
-		<child link="${arm2_prefix}base_link"/>
+		<child link="${arm_prefix}base_link"/>
 		<origin xyz="0 0 ${robot_stand_height * 0.5}" rpy="0 0 -3.14"/>
 	</joint>
 	<!-- end of arm workcell joint definitions-->
 	<!-- arm-gripper coupling joint definitions -->
-	<joint name="${arm2_prefix}to_gripper" type="fixed">
-		<parent link="${arm2_prefix}ee_link"/>
-		<child link="${arm2_prefix}gripper_frame"/>
+	<joint name="${arm_prefix}to_gripper" type="fixed">
+		<parent link="${arm_prefix}ee_link"/>
+		<child link="${arm_prefix}gripper_frame"/>
 		<origin xyz="0 0 0" rpy="0 1.57 0"/>
 	</joint>

Commit message: rotated base of ur5 by -45 degrees in mantis_ur5_arm_workspace.xacro

File: trunk/mantis/mantis_config/urdf/mantis_ur5_arm_workspace.xacro (robot description, xacro)
@@ -47,5 +47,5 @@
 		<parent link="ur5_stand"/>
 		<child link="${arm_prefix}base_link"/>
-		<origin xyz="0 0 ${robot_stand_height * 0.5}" rpy="0 0 -3.14"/>
+		<origin xyz="0 0 ${robot_stand_height * 0.5}" rpy="0 0 2.355"/>
 	</joint>
 	<!-- end of arm workcell joint definitions-->

Commit message: added roll to sensor_definitions. Changed values in sensor_definitions to match the current setup in the lab (probably not final setup, but should be close). changed rpy vlues in joiny ${arm_prefix}to_gripper so that the one functioning suction cup on the actual robot matches the tcp frame of the model robot.

File: trunk/mantis/mantis_config/urdf/mantis_ur5_arm_workspace.xacro (robot description, xacro)
@@ -12,4 +12,5 @@
 	<xacro:property name="arm_prefix" value="ur5_arm_"/>
 	<xacro:property name="arm_name" value="ur5"/>
+	<xacro:property name="temp_base_offset" value="0.045"/>
 	<!-- instantiating arm and gripper -->
 	<xacro:ur5_robot prefix="${arm_prefix}"/>
@@ -35,5 +36,5 @@
 	<!-- instantiating sensor definitions -->
 	<xacro:sensor_definitions prefix="${arm_prefix}" parent_link="ur5_stand"
-		x_val="-1.08" y_val="0.72" z_val="${0.82 - 0.5 * robot_stand_height}" pitch="0.5235" yaw="-0.604"/>
+		x_val="-0.75" y_val="-0.03" z_val="1.37" pitch="1.19" yaw="0.0" roll="0.07" />
 	<!--xacro:sensor_definitions prefix="${arm_prefix}" parent_link="${arm_prefix}base_link"
 		x_val="1.08" y_val="-0.72" z_val="${0.82 - robot_stand_height}" pitch="0.5235" yaw="2.536"/-->
@@ -49,5 +50,5 @@
 		<parent link="ur5_stand"/>
 		<child link="${arm_prefix}base_link"/>
-		<origin xyz="0 0 ${robot_stand_height * 0.5}" rpy="0 0 2.355"/>
+		<origin xyz="0 0 ${robot_stand_height * 0.5 + temp_base_offset}" rpy="0 0 2.355"/>
 	</joint>
 	<!-- end of arm workcell joint definitions-->
@@ -56,5 +57,5 @@
 		<parent link="${arm_prefix}ee_link"/>
 		<child link="${arm_prefix}gripper_frame"/>
-		<origin xyz="0 0 0" rpy="0 1.57 0"/>
+		<origin xyz="0 0 0" rpy="-1.57 0 -1.57"/> <!-- 0 1.57 0 -->
 	</joint>
 	<!-- end of arm-gripper coupling joint definitions -->

Commit message: changed camera/sensor position/definitions to match new semi-premanent location.

File: trunk/mantis/mantis_config/urdf/mantis_ur5_arm_workspace.xacro (robot description, xacro)
@@ -12,5 +12,5 @@
 	<xacro:property name="arm_prefix" value="ur5_arm_"/>
 	<xacro:property name="arm_name" value="ur5"/>
-	<xacro:property name="temp_base_offset" value="0.045"/>
+	<xacro:property name="temp_base_offset" value="0.0"/>
 	<!-- instantiating arm and gripper -->
 	<xacro:ur5_robot prefix="${arm_prefix}"/>
@@ -36,5 +36,5 @@
 	<!-- instantiating sensor definitions -->
 	<xacro:sensor_definitions prefix="${arm_prefix}" parent_link="ur5_stand"
-		x_val="-0.75" y_val="-0.03" z_val="1.37" pitch="1.19" yaw="0.0" roll="0.07" />
+		x_val="-0.9" y_val="-0.03" z_val="1.17" pitch="1.19" yaw="0.0" roll="0.015" />
 	<!--xacro:sensor_definitions prefix="${arm_prefix}" parent_link="${arm_prefix}base_link"
 		x_val="1.08" y_val="-0.72" z_val="${0.82 - robot_stand_height}" pitch="0.5235" yaw="2.536"/-->

Commit message: Vaccum gripper xacro tcp frame location was modified

File: trunk/mantis/mantis_config/urdf/mantis_ur5_arm_workspace.xacro (robot description, xacro)
@@ -36,5 +36,5 @@
 	<!-- instantiating sensor definitions -->
 	<xacro:sensor_definitions prefix="${arm_prefix}" parent_link="ur5_stand"
-		x_val="-0.9" y_val="-0.03" z_val="1.17" pitch="1.19" yaw="0.0" roll="0.015" />
+		x_val="-0.915" y_val="-0.03" z_val="1.17" pitch="1.19" yaw="0.0" roll="0.015" />
 	<!--xacro:sensor_definitions prefix="${arm_prefix}" parent_link="${arm_prefix}base_link"
 		x_val="1.08" y_val="-0.72" z_val="${0.82 - robot_stand_height}" pitch="0.5235" yaw="2.536"/-->

File: trunk/mantis/mantis_config/urdf/vacuum_gripper_macro.xacro (robot description, xacro)
@@ -39,5 +39,5 @@
 			<parent link="${prefix}gripper_frame"/>
 			<child link="${prefix}tcp_frame"/>
-			<origin xyz=" 0 ${gripper_length * 0.5} ${gripper_height}" rpy="0 0 0"/>
+			<origin xyz=" 0 ${gripper_length * 0.5} ${0.12}" rpy="0 0 0"/>
 		</joint>
 	</xacro:macro>
