Commit message: modified xacro and planning scene yaml file, to include obstacles and sensor definitions

File: trunk/mantis/mantis_config/urdf/mantis.urdf (robot description, URDF)
Before this commit: robot motoman_vacumm, 11 links, 10 joints
Links:
- added link kinect; collision box size=0.36 0.28 0.22
- added link kinect_frame; collision box size=0.064 0.28 0.04; visual box size=0.064 0.28 0.04
- added link kinect_ir_link; visual sphere radius=0.0005
- added link kinect_ir_optical_frame
- added link kinect_keepout; collision box size=0.25 2.69 2
- added link kinect_rgb_link; visual sphere radius=0.0005
- added link kinect_rgb_optical_frame
- added link power_supply; collision box size=0.400 0.250 0.115; visual box size=0.400 0.250 0.115
- added link table_keepout_1; collision box size=2.08 0.25 2
- added link table_keepout_2; collision box size=0.25 2.69 2
- link table: geometry collision box size=1.83 2.44 0.25; visual box size=1.83 2.44 0.25
Joints:
- added joint base-kinect: type fixed, parent base_link, child kinect, origin xyz=1.08 -0.72 0.82 rpy=0 0.5235 2.356
- added joint base-power_supply: type fixed, parent base_link, child power_supply, origin xyz=0 -0.260 0.050 rpy=0 0 0
- added joint kinect_frame_joint: type fixed, parent kinect, child kinect_frame, origin xyz=0 0 0 rpy=0 0 0
- added joint kinect_ir_joint: type fixed, parent kinect_frame, child kinect_ir_link, origin xyz=0 0 0 rpy=0 0 0
- added joint kinect_ir_optical_frame_joint: type fixed, parent kinect_ir_link, child kinect_ir_optical_frame, origin xyz=0 0 0 rpy=-1.57 0 -1.57
- added joint kinect_rgb_joint: type fixed, parent kinect_ir_link, child kinect_rgb_link, origin xyz=0 -0.03 0 rpy=0 0 0
- added joint kinect_rgb_optical_frame_joint: type fixed, parent kinect_rgb_link, child kinect_rgb_optical_frame, origin xyz=0 0 0 rpy=-1.57 0 -1.57
- added joint table-keepout_1: type fixed, parent table, child table_keepout_1, origin xyz=0 -1.34 1 rpy=0 0 0
- added joint table-keepout_2: type fixed, parent table, child table_keepout_2, origin xyz=-1.025 0 1 rpy=0 0 0
- added joint table-kinect: type fixed, parent table, child kinect_keepout, origin xyz=.5 0 1 rpy=0 0 0
- joint base-table: child base_link -> table; origin xyz=0 -0.8 1 rpy=0 0 1.57 -> xyz=1.19 0.22 -0.125 rpy=0 0 -0.785; parent table -> base_link

File: trunk/mantis/mantis_config/urdf/mantis.xacro (robot description, xacro)
@@ -20,5 +20,5 @@
 		</material>
 	</xacro:macro>
-	<!-- adding coupling link -->
+	<!-- arm-gripper coupling links -->
 	<link name="coupler">
 		<visual>
@@ -39,5 +39,6 @@
 		</collision>
 	</link>
-	<!-- adding joints for coupler/gripper -->
+	<!-- end of arm-gripper coupling links -->
+	<!-- arm-gripper coupling joints -->
 	<joint name="tool-coupler" type="fixed">
 		<parent link="link_t"/>
@@ -50,18 +51,176 @@
 		<origin xyz="0 0.182 0.036" rpy="-1.570 0 0"/>
 	</joint>
+	<!-- end of arm-gripper coupling joints -->
 	<!-- environment objects -->
 	<link name="table">
 		<visual>
-			<xacro:table_elements/>
-		</visual>
-		<collision>
-			<xacro:table_elements/>
-		</collision>
-	</link>
+			<geometry>
+				<box size="1.83 2.44 0.25"/>
+			</geometry>
+			<material name="">
+				<color rgba="1 0 1 1"/>
+			</material>
+		</visual>
+		<collision>
+			<geometry>
+				<box size="1.83 2.44 0.25"/>
+			</geometry>
+			<material name="">
+				<color rgba="1 0 1 1"/>
+			</material>
+		</collision>
+	</link>
+	<link name="table_keepout_1">
+		<collision>
+			<geometry>
+				<box size="2.08 0.25 2"/>
+			</geometry>
+			<material name="">
+				<color rgba="1 0.2 1 0.1"/>
+			</material>
+		</collision>
+	</link>
+	<link name="table_keepout_2">
+		<collision>
+			<geometry>
+				<box size="0.25 2.69 2"/>
+			</geometry>
+			<material name="">
+				<color rgba="1 0.2 1 0.1"/>
+			</material>
+		</collision>
+	</link>
+	<link name="power_supply">
+		<visual>
+			<geometry>
+				<box size="0.400 0.250 0.115"/>
+			</geometry>
+			<material name="">
+				<color rgba="1 0.2 1 0.1"/>
+			</material>
+		</visual>
+		<collision>
+			<geometry>
+				<box size="0.400 0.250 0.115"/>
+			</geometry>
+			<material name="">
+				<color rgba="1 0.2 1 0.1"/>
+			</material>
+		</collision>
+	</link>
+	<link name="kinect_keepout">
+		<collision>
+			<geometry>
+				<box size="0.25 2.69 2"/>
+			</geometry>
+			<material name="">
+				<color rgba="1 0.2 1 0.1"/>
+			</material>
+		</collision>
+	</link>
+	<link name="kinect">
+		<collision>
+			<geometry>
+				<box size="0.36 0.28 0.22"/>
+			</geometry>
+			<material name="">
+				<color rgba="1 0.8 1 0.1"/>
+			</material>
+		</collision>
+	</link>
+	<!-- end of environment objects -->
 	<!-- environment joints -->
 	<joint name="base-table" type="fixed">
+		<parent link="base_link"/>
+		<child link="table"/>
+		<origin xyz="1.19 0.22 -0.125" rpy="0 0 -0.785"/>
+	</joint>
+	<joint name="base-kinect" type="fixed">
+		<parent link="base_link"/>
+		<child link="kinect"/>
+		<origin rpy="0 0.5235 2.356" xyz="1.08 -0.72 0.82"/>
+	</joint>
+	<joint name="table-keepout_1" type="fixed">
 		<parent link="table"/>
-		<child link="base_link"/>
-		<origin xyz="0 ${-0.40 * table_length} ${table_height}" rpy="0 0 1.57"/>
-	</joint>
+		<child link="table_keepout_1"/>
+		<origin xyz="0 -1.34 1" rpy="0 0 0"/>
+	</joint>
+	<joint name="table-keepout_2" type="fixed">
+		<parent link="table"/>
+		<child link="table_keepout_2"/>
+		<origin xyz="-1.025 0 1" rpy="0 0 0"/>
+	</joint>
+	<joint name="base-power_supply" type="fixed">
+		<parent link="base_link"/>
+		<child link="power_supply"/>
+		<origin xyz="0 -0.260 0.050" rpy="0 0 0"/>
+	</joint>
+	<joint name="table-kinect" type="fixed">
+		<parent link="table"/>
+		<child link="kinect_keepout"/>
+		<origin xyz=".5 0 1" rpy="0 0 0"/>
+	</joint>
+	<!-- end of environment joints -->
+  	<!-- sensor links -->
+	<link name="kinect_frame">
+		<visual>
+			<origin rpy="0 0 0" xyz="0 0 0"/>
+			<geometry>
+				<box size="0.064 0.28 0.04"/>
+			</geometry>
+			<material name="silver"/>
+		</visual>
+		<collision>
+			<origin rpy="0 0 0" xyz="0 0 0"/>
+			<geometry>
+				<box size="0.064 0.28 0.04"/>
+			</geometry>
+		</collision>
+	</link>
+	<link name="kinect_ir_link">
+		<visual>
+			<origin rpy="0 0 0" xyz="0 0 0"/>
+			<geometry>
+				<sphere radius="0.0005"/>
+			</geometry>
+		</visual>
+	</link>
+	<link name="kinect_rgb_link">
+		<visual>
+			<origin rpy="0 0 0" xyz="0 0 0"/>
+			<geometry>
+				<sphere radius="0.0005"/>
+			</geometry>
+		</visual>
+	</link>
+	<link name="kinect_ir_optical_frame"/>
+	<link name="kinect_rgb_optical_frame"/>
+	<!-- end of sensor links -->
+	<!-- sensor joints -->
+	<joint name="kinect_frame_joint" type="fixed">
+		<parent link="kinect"/>
+		<child link="kinect_frame"/>
+		<origin rpy="0 0 0" xyz="0 0 0"/>
+	</joint>
+	<joint name="kinect_ir_joint" type="fixed">
+		<parent link="kinect_frame"/>
+		<child link="kinect_ir_link"/>
+		<origin rpy="0 0 0" xyz="0 0 0"/>
+	</joint>
+	<joint name="kinect_ir_optical_frame_joint" type="fixed">
+		<parent link="kinect_ir_link"/>
+		<child link="kinect_ir_optical_frame"/>
+		<origin rpy="-1.57 0 -1.57" xyz="0 0 0"/>
+	</joint>
+	<joint name="kinect_rgb_joint" type="fixed">
+		<parent link="kinect_ir_link"/>
+		<child link="kinect_rgb_link"/>
+		<origin rpy="0 0 0" xyz="0 -0.03 0"/>
+	</joint>
+	<joint name="kinect_rgb_optical_frame_joint" type="fixed">
+		<parent link="kinect_rgb_link"/>
+		<child link="kinect_rgb_optical_frame"/>
+		<origin rpy="-1.57 0 -1.57" xyz="0 0 0"/>
+	</joint>
+  	<!-- end of sensor joints -->
 </robot>

Commit message: Changed name of vacuum_gripper.stl/STL.  Windows does not differentiate between files with different cases.  Updated URDFs in Mantis config to reflect latest files.

File: trunk/mantis/mantis_config/urdf/mantis.urdf (robot description, URDF)
Before this commit: robot motoman_vacumm, 21 links, 20 joints
Links:
- link palm: geometry collision mesh filename=package://mantis_config/config/meshes/vacuum_gripper_col.stl; visual mesh filename=package://mantis_config/config/meshes/vacuum_gripper_vis.STL

File: trunk/mantis/mantis_config/urdf/mantis_asus.urdf (robot description, URDF)
Before this commit: robot motoman_vacumm, 21 links, 20 joints
Links:
- link palm: geometry collision mesh filename=package://mantis_config/config/meshes/vacuum_gripper_col.stl; visual mesh filename=package://mantis_config/config/meshes/vacuum_gripper_vis.STL

File: trunk/mantis/mantis_config/urdf/mantis_sia20d.urdf (robot description, URDF)
Before this commit: robot mantis_sia20d, 25 links, 24 joints
Links:
- link sia20d_arm_gripper_body: geometry collision box size=0.044 0.088 0.0946; visual mesh filename=package://mantis_config/config/meshes/vacuum_gripper_vis.STL

File: trunk/mantis/mantis_config/urdf/mantis_ur5.urdf (robot description, URDF)
Before this commit: robot mantis_ur5, 27 links, 26 joints
Links:
- link ur5_arm_gripper_body: geometry collision box size=0.044 0.088 0.0946; visual mesh filename=package://mantis_config/config/meshes/vacuum_gripper_vis.STL

File: trunk/mantis/mantis_config/urdf/vacuum_gripper.xacro (robot description, xacro)
@@ -6,5 +6,5 @@
 				<origin xyz="0 0.036 -0.1" rpy="0 0 0"/>
 				<geometry>
-					<mesh filename="package://mantis_config/config/meshes/vacuum_gripper.STL" />
+					<mesh filename="package://mantis_config/config/meshes/vacuum_gripper_vis.STL" />
 				</geometry>
 				<material name="silver">
@@ -15,5 +15,5 @@
 				<origin xyz="0 0.036 -0.1" rpy="0 0 0"/>
 				<geometry>
-					<mesh filename="package://mantis_config/config/meshes/vacuum_gripper.stl" />
+					<mesh filename="package://mantis_config/config/meshes/vacuum_gripper_col.stl" />
 				</geometry>
 				<material name="another_blue2">

File: trunk/mantis/mantis_config/urdf/vacuum_gripper_macro.xacro (robot description, xacro)
@@ -15,5 +15,5 @@
 				<origin xyz="0 0 -0.048" rpy="0 0 0"/>
 				<geometry>
-					<mesh filename="package://mantis_config/config/meshes/vacuum_gripper.STL" />
+					<mesh filename="package://mantis_config/config/meshes/vacuum_gripper_vis.STL" />
 				</geometry>
 				<material name="silver">
