Commit message: xacro with a temporary offset for the current testing phase setup

File: trunk/mantis/mantis_config/urdf/mantis_sia20d_arm_workspace.xacro (robot description, xacro)
@@ -12,4 +12,5 @@
 	<xacro:property name="arm_name" value="sia20d"/>
 	<xacro:property name="coupler_height" value="0.087"/>
+	<xacro:property name="temp_base_offset" value="0.045"/>
 	<!-- instantiating workcell definitions -->
 	<xacro:workcell_zone1_components/>
@@ -29,5 +30,5 @@
 		<parent link="workcell_frame"/>
 		<child link="${arm_prefix}base_link"/>
-		<origin xyz="0.241 0 0" rpy="0 0 0"/>
+		<origin xyz="0.241 0 ${temp_base_offset}" rpy="0 0 0"/>
 	</joint>
 	<!-- end of arm workcell joint definitions-->

Commit message: updated orientation of gripper relative to interface mount

File: trunk/mantis/mantis_config/urdf/mantis_sia20d_arm_workspace.xacro (robot description, xacro)
@@ -65,5 +65,5 @@
 		<child link="${arm_prefix}gripper_frame"/>
 		<!--child link="${arm_prefix}palm"/-->
-		<origin xyz="0 ${coupler_height} 0" rpy="-1.570 0 0"/>
+		<origin xyz="0 ${coupler_height} 0" rpy="-1.570 3.14 0"/>
 		<!--origin xyz="0 0.182 0.036" rpy="-1.570 0 0"/-->
 	</joint>

Commit message: changes sensor location/definitions to match the semi-temporary setup in the lab (will change slightly with addition of full camera case/enclosure).

File: trunk/mantis/mantis_config/urdf/mantis_sia20d_arm_workspace.xacro (robot description, xacro)
@@ -12,5 +12,5 @@
 	<xacro:property name="arm_name" value="sia20d"/>
 	<xacro:property name="coupler_height" value="0.087"/>
-	<xacro:property name="temp_base_offset" value="0.045"/>
+	<xacro:property name="temp_base_offset" value="0.0"/>
 	<!-- instantiating workcell definitions -->
 	<xacro:workcell_zone1_components/>
@@ -21,5 +21,5 @@
 		rpy="0.06+0.06 1.19 3.19+0.06" xyz="1.15-.16 -0.01 1.42+.16"-->
 	<xacro:sensor_definitions prefix="${arm_prefix}" parent_link="${arm_prefix}base_link"
-		x_val="0.99" y_val="-0.04" z_val="1.52" roll="0.12" pitch="1.19" yaw="3.25"/>
+		x_val="0.99" y_val="-0.09" z_val="1.25" roll="0.055" pitch="1.12" yaw="3.15"/>
 	<!-- end of sensor definitions -->
 	<!-- instantiating arm and gripper -->

Commit message: added an adjustment parameter for suction gripper height which changes with suction size and number of bellows. Currently sia20d has a smaller suction gripper.

File: trunk/mantis/mantis_config/urdf/mantis_sia20d_arm_workspace.xacro (robot description, xacro)
@@ -24,5 +24,5 @@
 	<!-- end of sensor definitions -->
 	<!-- instantiating arm and gripper -->
-	<xacro:vacuum_gripper_definition prefix="${arm_prefix}"/>
+	<xacro:vacuum_gripper_definition prefix="${arm_prefix}" gripper_adjustment="-0.010"/>
 	<xacro:sia20d_mesh prefix="${arm_prefix}"/>
 	<!-- arm-workcell joint definitions -->

File: trunk/mantis/mantis_config/urdf/mantis_ur5_arm_workspace.xacro (robot description, xacro)
@@ -15,5 +15,5 @@
 	<!-- instantiating arm and gripper -->
 	<xacro:ur5_robot prefix="${arm_prefix}"/>
-	<xacro:vacuum_gripper_definition prefix="${arm_prefix}"/>
+	<xacro:vacuum_gripper_definition prefix="${arm_prefix}" gripper_adjustment="0.0"/>
 	<!-- instantiating workcell definitions -->
 	<xacro:workcell_zone2_components/>

File: trunk/mantis/mantis_config/urdf/vacuum_gripper_macro.xacro (robot description, xacro)
@@ -5,5 +5,5 @@
 	<xacro:property name="gripper_width" value="0.088"/>
 	<xacro:property name="gripper_height" value="0.0946"/>
-	<xacro:macro name="vacuum_gripper_definition" params="prefix">
+	<xacro:macro name="vacuum_gripper_definition" params="prefix gripper_adjustment">
 		<link name="${prefix}gripper_frame"/>
 		<link name="${prefix}gripper_body">
@@ -39,5 +39,5 @@
 			<parent link="${prefix}gripper_frame"/>
 			<child link="${prefix}tcp_frame"/>
-			<origin xyz=" 0 ${gripper_length * 0.5} ${0.12}" rpy="0 0 0"/>
+			<origin xyz=" 0 ${gripper_length * 0.5 + gripper_adjustment} ${0.12}" rpy="0 0 0"/>
 		</joint>
 	</xacro:macro>

Commit message: fixed some issues with the concurrent arm move supervisor

File: trunk/mantis/mantis_config/urdf/mantis_sia20d_arm_workspace.xacro (robot description, xacro)
@@ -24,5 +24,5 @@
 	<!-- end of sensor definitions -->
 	<!-- instantiating arm and gripper -->
-	<xacro:vacuum_gripper_definition prefix="${arm_prefix}" gripper_adjustment="-0.010"/>
+	<xacro:vacuum_gripper_definition prefix="${arm_prefix}" gripper_adjustment="0.035"/>
 	<xacro:sia20d_mesh prefix="${arm_prefix}"/>
 	<!-- arm-workcell joint definitions -->

File: trunk/mantis/mantis_config/urdf/vacuum_gripper_macro.xacro (robot description, xacro)
@@ -39,5 +39,5 @@
 			<parent link="${prefix}gripper_frame"/>
 			<child link="${prefix}tcp_frame"/>
-			<origin xyz=" 0 ${gripper_length * 0.5 + gripper_adjustment} ${0.12}" rpy="0 0 0"/>
+			<origin xyz=" 0 ${gripper_length * 0.5} ${0.12 + gripper_adjustment}" rpy="0 0 0"/>
 		</joint>
 	</xacro:macro>
