Commit message: fix ABB xacro references after directory re-org

File: branches/moveit_dev/abb/irb_2400_arm_navigation/urdf/irb_2400.urdf (robot description, URDF)
Before this commit: robot irb_2400, 8 links, 7 joints
Links:
- link base_link: geometry collision mesh filename=package://irb_2400_arm_navigation/meshes/collision/base_lin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; visual mesh filename=package://irb_2400_arm_navigation/meshes/visual/base_link.S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
- link link_1: geometry collision mesh filename=package://irb_2400_arm_navigation/meshes/collision/link_1.S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; visual mesh filename=package://irb_2400_arm_navigation/meshes/visual/link_1.STL
- link link_2: geometry collision mesh filename=package://irb_2400_arm_navigation/meshes/collision/link_2_w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; visual mesh filename=package://irb_2400_arm_navigation/meshes/visual/link_2.STL
- link link_3: geometry collision mesh filename=package://irb_2400_arm_navigation/meshes/collision/link_3.S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; visual mesh filename=package://irb_2400_arm_navigation/meshes/visual/link_3.STL
- link link_4: geometry collision mesh filename=package://irb_2400_arm_navigation/meshes/collision/link_4.S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; visual mesh filename=package://irb_2400_arm_navigation/meshes/visual/link_4.STL
- link link_5: geometry collision mesh filename=package://irb_2400_arm_navigation/meshes/collision/link_5.S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; visual mesh filename=package://irb_2400_arm_navigation/meshes/visual/link_5.STL
- link link_6: geometry collision mesh filename=package://irb_2400_arm_navigation/meshes/collision/link_6.S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; visual mesh filename=package://irb_2400_arm_navigation/meshes/visual/link_6.STL
Joints:
- joint joint_5: origin xyz=0.497 0 -4.4409E-16 rpy=0 0 0 -> xyz=0.497 0 0 rpy=0 0 0
- joint joint_6: origin xyz=0.085 -4.1563E-17 2.2204E-16 rpy=0 0 0 -> xyz=0.085 0 0 rpy=0 0 0

File: branches/moveit_dev/abb/irb_2400_arm_navigation/urdf/irb_2400.xacro (robot description, xacro)
@@ -1,5 +1,5 @@
 <?xml version="1.0" ?>
 <robot name="irb_2400" xmlns:xacro="http://ros.org/wiki/xacro">
-	<include filename="$(find abb_common)/urdf/irb_2400_macro.xacro"/>
+	<include filename="irb_2400_macro.xacro"/>
 	<xacro:irb_2400 prefix=""/>
 </robot>

File: branches/moveit_dev/abb/irb_2400_arm_navigation/urdf/irb_2400_macro.xacro (robot description, xacro)
@@ -10,5 +10,5 @@
       			<geometry>
         			<mesh
-          			filename="package://abb_common/meshes/irb_2400/visual/base_link.STL" />
+          			filename="package://irb_2400_arm_navigation/meshes/visual/base_link.STL" />
       			</geometry>
       			<material
@@ -20,5 +20,5 @@
  			<collision>
 				<geometry>
-					<mesh filename="package://abb_common/meshes/irb_2400/collision/base_link.STL" />
+					<mesh filename="package://irb_2400_arm_navigation/meshes/collision/base_link.STL" />
 				</geometry>
 				<material name="yellow">
@@ -34,5 +34,5 @@
       			<geometry>
         			<mesh
-          			filename="package://abb_common/meshes/irb_2400/visual/link_1.STL" />
+          			filename="package://irb_2400_arm_navigation/meshes/visual/link_1.STL" />
       			</geometry>
       			<material name="abb_orange"/>
@@ -43,5 +43,5 @@
         			rpy="0 0 0" />
 				<geometry>
-					<mesh filename="package://abb_common/meshes/irb_2400/collision/link_1.STL" />
+					<mesh filename="package://irb_2400_arm_navigation/meshes/collision/link_1.STL" />
 				</geometry>
 				<material name="yellow"/>
@@ -55,5 +55,5 @@
       			<geometry>
         			<mesh
-          			filename="package://abb_common/meshes/irb_2400/visual/link_2.STL" />
+          			filename="package://irb_2400_arm_navigation/meshes/visual/link_2.STL" />
       			</geometry>
       			<material name="abb_orange"/>
@@ -64,5 +64,5 @@
         			rpy="0 0 0" />
 				<geometry>
-					<mesh filename="package://abb_common/meshes/irb_2400/collision/link_2_whole.STL" />
+					<mesh filename="package://irb_2400_arm_navigation/meshes/collision/link_2_whole.STL" />
 				</geometry>
 				<material name="yellow"/>
@@ -76,5 +76,5 @@
 			  	<geometry>
 					<mesh
-				  	filename="package://abb_common/meshes/irb_2400/visual/link_3.STL" />
+				  	filename="package://irb_2400_arm_navigation/meshes/visual/link_3.STL" />
 			  	</geometry>
 			  	<material name="abb_orange"/>
@@ -85,5 +85,5 @@
         			rpy="0 0 0" />
 				<geometry>
-					<mesh filename="package://abb_common/meshes/irb_2400/collision/link_3.STL" />
+					<mesh filename="package://irb_2400_arm_navigation/meshes/collision/link_3.STL" />
 				</geometry>
 				<material name="yellow"/>
@@ -97,5 +97,5 @@
 				  <geometry>
 					<mesh
-					  filename="package://abb_common/meshes/irb_2400/visual/link_4.STL" />
+					  filename="package://irb_2400_arm_navigation/meshes/visual/link_4.STL" />
 				  </geometry>
 				  <material name="abb_orange"/>
@@ -106,5 +106,5 @@
         			rpy="0 0 0" />
 				<geometry>
-					<mesh filename="package://abb_common/meshes/irb_2400/collision/link_4.STL" />
+					<mesh filename="package://irb_2400_arm_navigation/meshes/collision/link_4.STL" />
 				</geometry>
 				<material name="yellow"/>
@@ -118,5 +118,5 @@
 				<geometry>
 					<mesh
-					  filename="package://abb_common/meshes/irb_2400/visual/link_5.STL" />
+					  filename="package://irb_2400_arm_navigation/meshes/visual/link_5.STL" />
 				</geometry>
 				<material name="abb_orange"/>
@@ -127,5 +127,5 @@
         			rpy="0 0 0" />
 				<geometry>
-					<mesh filename="package://abb_common/meshes/irb_2400/collision/link_5.STL" />
+					<mesh filename="package://irb_2400_arm_navigation/meshes/collision/link_5.STL" />
 				</geometry>
 				<material name="yellow"/>
@@ -139,5 +139,5 @@
 				<geometry>
 					<mesh
-					  filename="package://abb_common/meshes/irb_2400/visual/link_6.STL" />
+					  filename="package://irb_2400_arm_navigation/meshes/visual/link_6.STL" />
 				</geometry>
 				<material name="abb_orange"/>
@@ -148,5 +148,5 @@
         			rpy="0 0 0" />
 				<geometry>
-					<mesh filename="package://abb_common/meshes/irb_2400/collision/link_6.STL" />
+					<mesh filename="package://irb_2400_arm_navigation/meshes/collision/link_6.STL" />
 				</geometry>
 				<material name="yellow"/>

File: branches/moveit_dev/abb/irb_5400_arm_navigation/urdf/irb_5400.urdf (robot description, URDF)
Before this commit: robot irb_5400, 8 links, 7 joints
Links:
- link base_link: geometry collision mesh filename=../meshes/collision/BASE_LINK.STL; visual mesh filename=../meshes/visual/BASE_LINK.STL
- link link_1: geometry collision mesh filename=../meshes/collision/LINK_1.STL; visual mesh filename=../meshes/visual/LINK_1.STL
- link link_2: geometry collision mesh filename=../meshes/collision/LINK_2.STL; visual mesh filename=../meshes/visual/LINK_2.STL
- link link_3: geometry collision mesh filename=../meshes/collision/LINK_3.STL; visual mesh filename=../meshes/visual/LINK_3.STL
- link link_4: geometry collision mesh filename=../meshes/collision/LINK_4.STL; visual mesh filename=../meshes/visual/LINK_4.STL
- link link_5: geometry collision mesh filename=../meshes/collision/LINK_5.STL; visual mesh filename=../meshes/visual/LINK_5.STL
- link link_6: geometry collision mesh filename=../meshes/collision/LINK_6.STL; visual mesh filename=../meshes/visual/LINK_6.STL

File: branches/moveit_dev/abb/irb_5400_arm_navigation/urdf/irb_5400.xacro (robot description, xacro)
@@ -1,5 +1,5 @@
 <?xml version="1.0" ?>
 <robot name="irb_5400" xmlns:xacro="http://ros.org/wiki/xacro">
-	<include filename="$(find abb_common)/urdf/irb_5400_macro.xacro" />
+	<include filename="irb_5400_macro.xacro" />
 	<xacro:irb_5400 prefix=""/>
 </robot>

File: branches/moveit_dev/abb/irb_5400_arm_navigation/urdf/irb_5400_macro.xacro (robot description, xacro)
@@ -6,5 +6,5 @@
       <visual>
         <geometry>
-          <mesh filename="package://abb_common/meshes/irb_5400/visual/BASE_LINK.STL" />
+          <mesh filename="../meshes/visual/BASE_LINK.STL" />
         </geometry>
         <material name="orange">
@@ -14,5 +14,5 @@
       <collision>
         <geometry>
-          <mesh filename="package://abb_common/meshes/irb_5400/collision/BASE_LINK.STL" />
+          <mesh filename="../meshes/collision/BASE_LINK.STL" />
         </geometry>
         <material name="yellow">
@@ -24,5 +24,5 @@
       <visual>
         <geometry>
-          <mesh filename="package://abb_common/meshes/irb_5400/visual/LINK_1.STL" />
+          <mesh filename="../meshes/visual/LINK_1.STL" />
         </geometry>
         <material name="orange" />
@@ -30,5 +30,5 @@
       <collision>
         <geometry>
-          <mesh filename="package://abb_common/meshes/irb_5400/collision/LINK_1.STL" />
+          <mesh filename="../meshes/collision/LINK_1.STL" />
         </geometry>
         <material name="yellow"/>
@@ -38,5 +38,5 @@
       <visual>
         <geometry>
-          <mesh filename="package://abb_common/meshes/irb_5400/visual/LINK_2.STL" />
+          <mesh filename="../meshes/visual/LINK_2.STL" />
         </geometry>
         <material name="lt_black">
@@ -46,5 +46,5 @@
       <collision>
         <geometry>
-          <mesh filename="package://abb_common/meshes/irb_5400/collision/LINK_2.STL" />
+          <mesh filename="../meshes/collision/LINK_2.STL" />
         </geometry>
         <material name="yellow"/>
@@ -54,5 +54,5 @@
       <visual>
         <geometry>
-          <mesh filename="package://abb_common/meshes/irb_5400/visual/LINK_3.STL" />
+          <mesh filename="../meshes/visual/LINK_3.STL" />
         </geometry>
         <material name="orange" />
@@ -60,5 +60,5 @@
       <collision>
         <geometry>
-          <mesh filename="package://abb_common/meshes/irb_5400/collision/LINK_3.STL" />
+          <mesh filename="../meshes/collision/LINK_3.STL" />
         </geometry>
         <material name="yellow"/>
@@ -68,5 +68,5 @@
       <visual>
         <geometry>
-          <mesh filename="package://abb_common/meshes/irb_5400/visual/LINK_4.STL" />
+          <mesh filename="../meshes/visual/LINK_4.STL" />
         </geometry>
         <material name="lt_black" />
@@ -74,5 +74,5 @@
       <collision>
         <geometry>
-          <mesh filename="package://abb_common/meshes/irb_5400/collision/LINK_4.STL" />
+          <mesh filename="../meshes/collision/LINK_4.STL" />
         </geometry>
         <material name="yellow"/>
@@ -82,5 +82,5 @@
       <visual>
         <geometry>
-          <mesh filename="package://abb_common/meshes/irb_5400/visual/LINK_5.STL" />
+          <mesh filename="../meshes/visual/LINK_5.STL" />
         </geometry>
         <material name="lt_black" />
@@ -88,5 +88,5 @@
       <collision>
         <geometry>
-          <mesh filename="package://abb_common/meshes/irb_5400/collision/LINK_5.STL" />
+          <mesh filename="../meshes/collision/LINK_5.STL" />
         </geometry>
         <material name="yellow"/>
@@ -96,5 +96,5 @@
       <visual>
         <geometry>
-          <mesh filename="package://abb_common/meshes/irb_5400/visual/LINK_6.STL" />
+          <mesh filename="../meshes/visual/LINK_6.STL" />
         </geometry>
         <material name="lt_black" />
@@ -102,5 +102,5 @@
       <collision>
         <geometry>
-          <mesh filename="package://abb_common/meshes/irb_5400/collision/LINK_6.STL" />
+          <mesh filename="../meshes/collision/LINK_6.STL" />
         </geometry>
         <material name="yellow"/>
