Commit message: mantis demo stable version as of 01052013

File: branches/mantis_demo_01032013/mantis/mantis_config/urdf/mantis_sensor_macro.xacro (robot description, xacro)
@@ -21,10 +21,10 @@
 		</link>
 		<link name="${prefix}kinect_keepout">
-			<collision>
+			<!--collision>
 				<material name="${prefix}color_b"/>
 				<geometry>
 					<box size="0.2 0.32 ${z_val + 0.08}"/>
 				</geometry>
-			</collision>
+			</collision-->
 		</link>
 		<!-- end of sensor main components -->

File: branches/mantis_demo_01032013/mantis/mantis_config/urdf/mantis_sia20d_arm_workspace.xacro (robot description, xacro)
@@ -21,5 +21,5 @@
 		rpy="0.06+0.06 1.19 3.19+0.06" xyz="1.15-.16 -0.01 1.42+.16"-->
 	<xacro:sensor_definitions prefix="${arm_prefix}" parent_link="${arm_prefix}base_link"
-		x_val="0.955" y_val="-0.002" z_val="1.174" roll="0.04" pitch="1.959" yaw="0"/>
+		x_val="0.930" y_val="0.175" z_val="1.174" roll="0.0" pitch="1.959" yaw="0.02"/>
 	<!-- end of sensor definitions -->
 	<!-- instantiating arm and gripper -->
