Commit message: changed solid model to reflect vacuum gripper with one suction cup

File: branches/mantis_demo_01032013/mantis/mantis_config/urdf/vacuum_gripper.xacro (robot description, xacro)
@@ -6,5 +6,5 @@
 				<origin xyz="0 0.036 -0.1" rpy="0 0 0"/>
 				<geometry>
-					<mesh filename="package://mantis_config/config/meshes/vacuum_gripper_vis.STL" />
+					<mesh filename="package://mantis_config/config/meshes/vacuum_gripper_one_suction_cup.STL" />
 				</geometry>
 				<material name="silver">
