Commit message: in vacuum_gripper_macro.xacro: loads single vacuum cup model

File: branches/mantis_demo_01032013/mantis/mantis_config/urdf/vacuum_gripper_macro.xacro (robot description, xacro)
@@ -15,5 +15,5 @@
 				<origin xyz="0 0 -0.048" rpy="0 0 0"/>
 				<geometry>
-					<mesh filename="package://mantis_config/config/meshes/vacuum_gripper_vis.STL" />
+					<mesh filename="package://mantis_config/config/meshes/vacuum_gripper_one_suction_cup.STL" />
 				</geometry>
 				<material name="silver">
