Commit message: Manually merged trunk revisions r1233 (URDF formatting and robot mesh colours), r1234 (m430 incorrect joint limits), r1279 (update m430 meshes) and r1280 (minor launch file updates) into fanuc stack in fuerte dev branch.

File: branches/fuerte_dev/fanuc/fanuc_config/urdf/M16iB20_macro.xacro (robot description, xacro)
@@ -2,283 +2,163 @@
 <robot xmlns:xacro="http://ros.org/wiki/xacro">
 	<xacro:macro name="M16iB20" params="prefix">
-	<!-- links -->
-		  <link name="${prefix}base_link">
-		    <visual>
-		      <origin
-			xyz="0 0 0"
-			rpy="0 0 0" />
-		      <geometry>
-			<mesh
-			  filename="package://fanuc_config/meshes/m_16iB20/visual/base_link.STL" />
-		      </geometry>
-		      <material
-			name="">
-			<color
-			  rgba="1 1 0 1" />
-		      </material>
-		    </visual>
-		    <collision>
-		      <origin
-			xyz="0 0 0"
-			rpy="0 0 0" />
-		      <geometry>
-			<mesh
-			  filename="package://fanuc_config/meshes/m_16iB20/collision/base_link.STL" />
-		      </geometry>
-		    </collision>
-		  </link>
-		  <link name="${prefix}link_1">
-		    <visual>
-		      <origin
-			xyz="0 0 0"
-			rpy="0 0 0" />
-		      <geometry>
-			<mesh
-			  filename="package://fanuc_config/meshes/m_16iB20/visual/Link_1.STL" />
-		      </geometry>
-		      <material
-			name="">
-			<color
-			  rgba="1 1 0 1" />
-		      </material>
-		    </visual>
-		    <collision>
-		      <origin
-			xyz="0 0 0"
-			rpy="0 0 0" />
-		      <geometry>
-			<mesh
-			  filename="package://fanuc_config/meshes/m_16iB20/collision/Link_1.STL" />
-		      </geometry>
-		    </collision>
-		  </link>
-		  <link name="${prefix}link_2">
-		    <visual>
-		      <origin
-			xyz="0 0 0"
-			rpy="0 0 0" />
-		      <geometry>
-			<mesh
-			  filename="package://fanuc_config/meshes/m_16iB20/visual/Link_2.STL" />
-		      </geometry>
-		      <material
-			name="">
-			<color
-			  rgba="1 1 0 1" />
-		      </material>
-		    </visual>
-		    <collision>
-		      <origin
-			xyz="0 0 0"
-			rpy="0 0 0" />
-		      <geometry>
-			<mesh
-			  filename="package://fanuc_config/meshes/m_16iB20/collision/Link_2.STL" />
-		      </geometry>
-		    </collision>
-		  </link>
-		  <link name="${prefix}link_3">
-		    <visual>
-		      <origin
-			xyz="0 0 0"
-			rpy="0 0 0" />
-		      <geometry>
-			<mesh
-			  filename="package://fanuc_config/meshes/m_16iB20/visual/Link_3.STL" />
-		      </geometry>
-		      <material
-			name="">
-			<color
-			  rgba="1 1 0 1" />
-		      </material>
-		    </visual>
-		    <collision>
-		      <origin
-			xyz="0 0 0"
-			rpy="0 0 0" />
-		      <geometry>
-			<mesh
-			  filename="package://fanuc_config/meshes/m_16iB20/collision/Link_3.STL" />
-		      </geometry>
-		    </collision>
-		  </link>
-		  <link name="${prefix}link_4">
-		    <visual>
-		      <origin
-			xyz="0 0 0"
-			rpy="0 0 0" />
-		      <geometry>
-			<mesh
-			  filename="package://fanuc_config/meshes/m_16iB20/visual/Link_4.STL" />
-		      </geometry>
-		      <material
-			name="">
-			<color
-			  rgba="1 1 0 1" />
-		      </material>
-		    </visual>
-		    <collision>
-		      <origin
-			xyz="0 0 0"
-			rpy="0 0 0" />
-		      <geometry>
-			<mesh
-			  filename="package://fanuc_config/meshes/m_16iB20/collision/Link_4.STL" />
-		      </geometry>
-		    </collision>
-		  </link>
-		  <link name="${prefix}link_5">
-		    <visual>
-		      <origin
-			xyz="0 0 0"
-			rpy="0 0 0" />
-		      <geometry>
-			<mesh
-			  filename="package://fanuc_config/meshes/m_16iB20/visual/Link_5.STL" />
-		      </geometry>
-		      <material
-			name="">
-			<color
-			  rgba="1 1 0 1" />
-		      </material>
-		    </visual>
-		    <collision>
-		      <origin
-			xyz="0 0 0"
-			rpy="0 0 0" />
-		      <geometry>
-			<mesh
-			  filename="package://fanuc_config/meshes/m_16iB20/collision/Link_5.STL" />
-		      </geometry>
-		    </collision>
-		  </link>
-		  <link name="${prefix}link_6">
-		    <visual>
-		      <origin
-			xyz="0 0 0"
-			rpy="0 0 0" />
-		      <geometry>
-			<mesh
-			  filename="package://fanuc_config/meshes/m_16iB20/visual/Link_6.STL" />
-		      </geometry>
-		      <material
-			name="">
-			<color
-			  rgba="1 1 0 1" />
-		      </material>
-		    </visual>
-		    <collision>
-		      <origin
-			xyz="0 0 0"
-			rpy="0 0 0" />
-		      <geometry>
-			<mesh
-			  filename="package://fanuc_config/meshes/m_16iB20/collision/Link_6.STL" />
-		      </geometry>
-		    </collision>
-		  </link>
-          <link name="${prefix}tool0"/>
-	<!-- joints -->
-		  <joint name="${prefix}joint_1" type="revolute">
-		    <origin
-		      xyz="0 0 0.245"
-		      rpy="0 0 0" />
-		    <parent
-		      link="base_link" />
-		    <child
-		      link="link_1" />
-		    <axis
-		      xyz="0 0 1" />
-		    <limit
-		      lower="-2.967"
-		      upper="2.967"
-		      effort="0"
-		      velocity="2.879" />
-		  </joint>
-		  <joint name="${prefix}joint_2" type="revolute">
-		    <origin
-		      xyz="0.15 0.18759 0.28"
-		      rpy="0 0 0" />
-		    <parent
-		      link="link_1" />
-		    <child
-		      link="link_2" />
-		    <axis
-		      xyz="0 1 0" />
-		    <limit
-		      lower="-1.38"
-		      upper="2.78"
-		      effort="0"
-		      velocity="2.879" />
-		  </joint>
-		  <joint name="${prefix}joint_3" type="revolute">
-		    <origin
-		      xyz="0 -0.18759 0.77"
-		      rpy="0 0 0" />
-		    <parent
-		      link="link_2" />
-		    <child
-		      link="link_3" />
-		    <axis
-		      xyz="0 -1 0" />
-		    <limit
-		      lower="-4.08"
-		      upper="1.38"
-		      effort="0"
-		      velocity="3.054" />
-		  </joint>
-		  <joint name="${prefix}joint_4" type="revolute">
-		    <origin
-		      xyz="0.18425 0 0.1"
-		      rpy="0 0 0" />
-		    <parent
-		      link="link_3" />
-		    <child
-		      link="link_4" />
-		    <axis
-		      xyz="-1 0 0" />
-		    <limit
-		      lower="-3.48"
-		      upper="3.48"
-		      effort="0"
-		      velocity="6.108" />
-		  </joint>
-		  <joint name="${prefix}joint_5" type="revolute">
-		    <origin
-		      xyz="0.55575 0 0"
-		      rpy="0 0 0" />
-		    <parent
-		      link="link_4" />
-		    <child
-		      link="link_5" />
-		    <axis
-		      xyz="0 -1 0" />
-		    <limit
-		      lower="-2.43"
-		      upper="2.43"
-		      effort="0"
-		      velocity="5.934" />
-		  </joint>
-		  <joint name="${prefix}joint_6" type="revolute">
-		    <origin
-		      xyz="0.1 0 0"
-		      rpy="0 0 0" />
-		    <parent
-		      link="link_5" />
-		    <child
-		      link="link_6" />
-		    <axis
-		      xyz="-1 0 0" />
-		    <limit
-		      lower="-7.84"
-		      upper="7.84"
-		      effort="0"
-		      velocity="9.075" />
-		  </joint>
-		  <joint name="${prefix}joint_6-tool0" type="fixed">
-		      <parent link="${prefix}link_6"/>
-	              <child link="${prefix}tool0"/>
-          	      <origin xyz="0 0 0" rpy="0 0 0"/>
-	          </joint>
+		<!-- links -->
+		<link name="${prefix}base_link">
+			<visual>
+				<origin xyz="0 0 0" rpy="0 0 0"/>
+				<geometry>
+					<mesh filename="package://fanuc_config/meshes/m_16iB20/visual/base_link.STL"/>
+				</geometry>
+				<material name="fyel">
+					<color rgba="0.9 0.9 0 1" />
+				</material>
+			</visual>
+			<collision>
+				<origin xyz="0 0 0" rpy="0 0 0"/>
+				<geometry>
+					<mesh filename="package://fanuc_config/meshes/m_16iB20/collision/base_link.STL"/>
+				</geometry>
+			</collision>
+		</link>
+		<link name="${prefix}link_1">
+			<visual>
+				<origin xyz="0 0 0" rpy="0 0 0"/>
+				<geometry>
+					<mesh filename="package://fanuc_config/meshes/m_16iB20/visual/Link_1.STL"/>
+				</geometry>
+				<material name="fyel" />
+			</visual>
+			<collision>
+				<origin xyz="0 0 0" rpy="0 0 0"/>
+				<geometry>
+					<mesh filename="package://fanuc_config/meshes/m_16iB20/collision/Link_1.STL"/>
+				</geometry>
+			</collision>
+		</link>
+		<link name="${prefix}link_2">
+			<visual>
+				<origin xyz="0 0 0" rpy="0 0 0"/>
+				<geometry>
+					<mesh filename="package://fanuc_config/meshes/m_16iB20/visual/Link_2.STL"/>
+				</geometry>
+				<material name="fyel" />
+			</visual>
+			<collision>
+				<origin xyz="0 0 0" rpy="0 0 0"/>
+				<geometry>
+					<mesh filename="package://fanuc_config/meshes/m_16iB20/collision/Link_2.STL"/>
+				</geometry>
+			</collision>
+		</link>
+		<link name="${prefix}link_3">
+			<visual>
+				<origin xyz="0 0 0" rpy="0 0 0"/>
+				<geometry>
+					<mesh filename="package://fanuc_config/meshes/m_16iB20/visual/Link_3.STL"/>
+				</geometry>
+				<material name="fyel" />
+			</visual>
+			<collision>
+				<origin xyz="0 0 0" rpy="0 0 0"/>
+				<geometry>
+					<mesh filename="package://fanuc_config/meshes/m_16iB20/collision/Link_3.STL"/>
+				</geometry>
+			</collision>
+		</link>
+		<link name="${prefix}link_4">
+			<visual>
+				<origin xyz="0 0 0" rpy="0 0 0"/>
+				<geometry>
+					<mesh filename="package://fanuc_config/meshes/m_16iB20/visual/Link_4.STL"/>
+				</geometry>
+				<material name="fyel" />
+			</visual>
+			<collision>
+				<origin xyz="0 0 0" rpy="0 0 0"/>
+				<geometry>
+					<mesh filename="package://fanuc_config/meshes/m_16iB20/collision/Link_4.STL"/>
+				</geometry>
+			</collision>
+		</link>
+		<link name="${prefix}link_5">
+			<visual>
+				<origin xyz="0 0 0" rpy="0 0 0"/>
+				<geometry>
+					<mesh filename="package://fanuc_config/meshes/m_16iB20/visual/Link_5.STL"/>
+				</geometry>
+				<material name="fyel" />
+			</visual>
+			<collision>
+				<origin xyz="0 0 0" rpy="0 0 0"/>
+				<geometry>
+					<mesh filename="package://fanuc_config/meshes/m_16iB20/collision/Link_5.STL"/>
+				</geometry>
+			</collision>
+		</link>
+		<link name="${prefix}link_6">
+			<visual>
+				<origin xyz="0 0 0" rpy="0 0 0"/>
+				<geometry>
+					<mesh filename="package://fanuc_config/meshes/m_16iB20/visual/Link_6.STL"/>
+				</geometry>
+				<material name="fblack">
+					<color rgba="0.1 0.1 0.1 1"/>
+				</material>
+			</visual>
+			<collision>
+				<origin xyz="0 0 0" rpy="0 0 0"/>
+				<geometry>
+					<mesh filename="package://fanuc_config/meshes/m_16iB20/collision/Link_6.STL"/>
+				</geometry>
+			</collision>
+		</link>
+		<link name="${prefix}tool0"/>
+		<!-- joints -->
+		<joint name="${prefix}joint_1" type="revolute">
+			<origin xyz="0 0 0.245" rpy="0 0 0"/>
+			<parent link="base_link"/>
+			<child link="link_1"/>
+			<axis xyz="0 0 1"/>
+			<limit lower="-2.967" upper="2.967" effort="0" velocity="2.879"/>
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
File: branches/fuerte_dev/fanuc/fanuc_config/urdf/m430iA2F.urdf (robot description, URDF)
Before this commit: robot m430iA2F, 7 links, 6 joints
Joints:
- joint joint_1: limit lower=-3.1415 upper=3.1415 effort=0 velocity=5.23598775598 -> lower=-3.1415 upper=3.1415 effort=0 velocity=5.24; origin xyz=-6.0758E-19 1.2493E-16 0.44 rpy=0 0 0 -> xyz=0 0 0.44 rpy=0 0 0
- joint joint_2: limit lower=-2.00707 upper=2.00707 effort=0 velocity=5.58505360638 -> lower=-2.01 upper=2.01 effort=0 velocity=5.59; origin xyz=-1.4097E-17 0.171 -4.4409E-16 rpy=0 0 0 -> xyz=0 0.171 0 rpy=0 0 0
- joint joint_3: limit lower=-1.771457 upper=1.771457 effort=0 velocity=5.58505360638 -> lower=-3.34 upper=3.34 effort=0 velocity=5.59; origin xyz=1.2197E-19 -0.171 0.350 rpy=0 0 0 -> xyz=0 -0.171 0.35 rpy=0 0 0
- joint joint_4: limit lower=-2.617917 upper=2.617917 effort=0 velocity=6.28318530718 -> lower=-2.62 upper=2.62 effort=0 velocity=6.28; origin xyz=-2.6075E-17 -0.06 0.55 rpy=0 0 0 -> xyz=0 -0.06 0.55 rpy=0 0 0
- joint joint_5: limit lower=-4.71225 upper=4.71225 effort=0 velocity=20.9439510239 -> lower=-4.71 upper=4.71 effort=0 velocity=20.94; origin xyz=1.4734E-16 -0.035 0.065 rpy=0 0 0 -> xyz=0 -0.035 0.065 rpy=0 0 0

File: branches/fuerte_dev/fanuc/fanuc_config/urdf/m_10iA_macro.xacro (robot description, xacro)
@@ -1,323 +1,160 @@
-<?xml version="1.0" ?>
+<?xml version="1.0"?>
 <robot xmlns:xacro="http://ros.org/wiki/xacro">
 	<xacro:macro name="m10iA" params="prefix">
-		<!-- link list -->
+		<!-- links -->
 		<link name="${prefix}base_link">
 			<visual>
-     			<origin
-        		xyz="0 0 0"
-       			rpy="-1.578 0 0" />
-      			<geometry>
-        			<mesh
-          			filename="package://fanuc_config/meshes/m_10iA/visual/base_link.stl" />
-      			</geometry>
-      			<material
-        			name="grey">
-        			<color
-          			rgba="0.75 0.75 0.75 1" />
-      			</material>
-    		</visual>
- 			<collision>
-     			<origin
-        		xyz="0 0 0"
-       			rpy="-1.578 0 0" />
+				<origin xyz="0 0 0" rpy="-1.578 0 0"/>
 				<geometry>
-					<mesh filename="package://fanuc_config/meshes/m_10iA/collision/base_link.stl" />
+					<mesh filename="package://fanuc_config/meshes/m_10iA/visual/base_link.stl"/>
 				</geometry>
-				<material name="yellow">
-					<color rgba="1 1 0 1"/>
+				<material name="fgrey">
+					<color rgba="0.20 0.20 0.20 1"/>
 				</material>
+			</visual>
+			<collision>
+				<origin xyz="0 0 0" rpy="-1.578 0 0"/>
+				<geometry>
+					<mesh filename="package://fanuc_config/meshes/m_10iA/collision/base_link.stl"/>
+				</geometry>
 			</collision>
 		</link>
 		<link name="${prefix}link_1">
 			<visual>
-      			<origin
-        			xyz="0 0 0"
-        			rpy="0 0 0" />
-      			<geometry>
-        			<mesh
-          			filename="package://fanuc_config/meshes/m_10iA/visual/link_1.stl" />
-      			</geometry>
-      			<material name="grey"/>
-    		</visual>
+				<origin xyz="0 0 0" rpy="0 0 0"/>
+				<geometry>
+					<mesh filename="package://fanuc_config/meshes/m_10iA/visual/link_1.stl"/>
+				</geometry>
+				<material name="fyel">
+					<color rgba="0.9 0.9 0 1"/>
+				</material>
+			</visual>
 			<collision>
-      			<origin
-        			xyz="0 0 0"
-        			rpy="0 0 0" />
+				<origin xyz="0 0 0" rpy="0 0 0"/>
 				<geometry>
-					<mesh filename="package://fanuc_config/meshes/m_10iA/collision/link_1.stl" />
+					<mesh filename="package://fanuc_config/meshes/m_10iA/collision/link_1.stl"/>
 				</geometry>
-				<material name="yellow"/>
 			</collision>
 		</link>
 		<link name="${prefix}link_2">
-		    <visual>
-      			<origin
-        			xyz="0 0 0"
-        			rpy="0 0 0" />
-      			<geometry>
-        			<mesh
-          			filename="package://fanuc_config/meshes/m_10iA/visual/link_2.stl" />
-      			</geometry>
-      			<material name="grey"/>
-    		</visual>
+			<visual>
+				<origin xyz="0 0 0" rpy="0 0 0"/>
+				<geometry>
+					<mesh filename="package://fanuc_config/meshes/m_10iA/visual/link_2.stl"/>
+				</geometry>
+				<material name="fyel"/>
+			</visual>
 			<collision>
-      			<origin
-        			xyz="0 0 0"
-        			rpy="0 0 0" />
+				<origin xyz="0 0 0" rpy="0 0 0"/>
 				<geometry>
-					<mesh filename="package://fanuc_config/meshes/m_10iA/collision/link_2.stl" />
+					<mesh filename="package://fanuc_config/meshes/m_10iA/collision/link_2.stl"/>
 				</geometry>
-				<material name="yellow"/>
 			</collision>
 		</link>
 		<link name="${prefix}link_3">
 			<visual>
-				<origin
-					xyz="0 0 0"
-					rpy="0 0 0" />
-			  	<geometry>
-					<mesh
-				  	filename="package://fanuc_config/meshes/m_10iA/visual/link_3.stl" />
-			  	</geometry>
-			  	<material name="grey"/>
+				<origin xyz="0 0 0" rpy="0 0 0"/>
+				<geometry>
+					<mesh filename="package://fanuc_config/meshes/m_10iA/visual/link_3.stl"/>
+				</geometry>
+				<material name="fyel"/>
 			</visual>
 			<collision>
-      			<origin
-        			xyz="0 0 0"
-        			rpy="0 0 0" />
+				<origin xyz="0 0 0" rpy="0 0 0"/>
 				<geometry>
-					<mesh filename="package://fanuc_config/meshes/m_10iA/collision/link_3.stl" />
+					<mesh filename="package://fanuc_config/meshes/m_10iA/collision/link_3.stl"/>
 				</geometry>
-				<material name="yellow"/>
 			</collision>
 		</link>
 		<link name="${prefix}link_4">
 			<visual>
-				  <origin
-					xyz="0 0 0"
-					rpy="0 0 0" />
-				  <geometry>
-					<mesh
-					  filename="package://fanuc_config/meshes/m_10iA/visual/link_4.stl" />
-				  </geometry>
-				  <material name="grey"/>
+				<origin xyz="0 0 0" rpy="0 0 0"/>
+				<geometry>
+					<mesh filename="package://fanuc_config/meshes/m_10iA/visual/link_4.stl"/>
+				</geometry>
+				<material name="fyel"/>
 			</visual>
 			<collision>
-      			<origin
-        			xyz="0 0 0"
-        			rpy="0 0 0" />
+				<origin xyz="0 0 0" rpy="0 0 0"/>
 				<geometry>
-					<mesh filename="package://fanuc_config/meshes/m_10iA/collision/link_4.stl" />
+					<mesh filename="package://fanuc_config/meshes/m_10iA/collision/link_4.stl"/>
 				</geometry>
-				<material name="yellow"/>
 			</collision>
 		</link>
 		<link name="${prefix}link_5">
 			<visual>
-				<origin
-					xyz="0 0 0"
-					rpy="0 0 0" />
+				<origin xyz="0 0 0" rpy="0 0 0"/>
 				<geometry>
-					<mesh
-					  filename="package://fanuc_config/meshes/m_10iA/visual/link_5.stl" />
+					<mesh filename="package://fanuc_config/meshes/m_10iA/visual/link_5.stl"/>
 				</geometry>
-				<material name="grey"/>
+				<material name="fyel"/>
 			</visual>
 			<collision>
-      			<origin
-        			xyz="0 0 0"
-        			rpy="0 0 0" />
+				<origin xyz="0 0 0" rpy="0 0 0"/>
 				<geometry>
-					<mesh filename="package://fanuc_config/meshes/m_10iA/collision/link_5.stl" />
+					<mesh filename="package://fanuc_config/meshes/m_10iA/collision/link_5.stl"/>
 				</geometry>
-				<material name="yellow"/>
 			</collision>
 		</link>
 		<link name="${prefix}link_6">
 			<visual>
-				<origin
-					xyz="0 0 0"
-					rpy="0 0 0" />
+				<origin xyz="0 0 0" rpy="0 0 0"/>
 				<geometry>
-					<mesh
-					  filename="package://fanuc_config/meshes/m_10iA/visual/link_6.stl" />
+					<mesh filename="package://fanuc_config/meshes/m_10iA/visual/link_6.stl"/>
 				</geometry>
-				<material name="grey"/>
+				<material name="fblack">
+					<color rgba="0.1 0.1 0.1 1"/>
+				</material>
 			</visual>
 			<collision>
-      			<origin
-        			xyz="0 0 0"
-        			rpy="0 0 0" />
+				<origin xyz="0 0 0" rpy="0 0 0"/>
 				<geometry>
-					<mesh filename="package://fanuc_config/meshes/m_10iA/collision/link_6.stl" />
+					<mesh filename="package://fanuc_config/meshes/m_10iA/collision/link_6.stl"/>
 				</geometry>
-				<material name="yellow"/>
 			</collision>
 		</link>
 		<link name="${prefix}tool0"/>
-		<!-- end of link list -->
-		<!-- joint list -->
+		<!-- joints -->
 		<joint name="${prefix}joint_1" type="revolute">
-			<origin
-      			xyz="0 0 0"
-      			rpy="0 0 0" />
-			<parent
-			  link="base_link" />
-			<child
-			  link="link_1" />
-			<axis
-			  xyz="0 0 1" />
-			<limit
-			  lower="-5.93"
-			  upper="5.93"
-			  effort="0"
-			  velocity="3.665" />
-			<calibration
-			  rising="0"
-			  falling="0" />
-			<dynamics
-			  damping="0"
-			  friction="0" />
-<!--			<safety_controller
-			  soft_lower_limit="0"
-			  soft_upper_limit="0"
-			  k_position="0"
-			  k_velocity="0" /> -->
+			<origin xyz="0 0 0" rpy="0 0 0"/>
+			<parent link="base_link"/>
+			<child link="link_1"/>
+			<axis xyz="0 0 1"/>
+			<limit lower="-5.93" upper="5.93" effort="0" velocity="3.665"/>
 		</joint>
 		<joint name="${prefix}joint_2" type="revolute">
-			<origin
-			  xyz="0.15 -0.04 0.45"
-      		  rpy="0 0 0" />
-			<parent
-			  link="link_1" />
-			<child
-			  link="link_2" />
-			<axis
-			  xyz="0 1 0" />
-			<limit
-			  lower="-4.36"
-			  upper="4.36"
-			  effort="0"
-			  velocity="3.32" />
-			<calibration
-			  rising="0"
-			  falling="0" />
-			<dynamics
-			  damping="0"
-			  friction="0" />
-<!--			<safety_controller
-			  soft_lower_limit="0"
-			  soft_upper_limit="0"
-			  k_position="0"
-			  k_velocity="0" /> -->
-  		</joint>
+			<origin xyz="0.15 -0.04 0.45" rpy="0 0 0"/>
+			<parent link="link_1"/>
+			<child link="link_2"/>
+			<axis xyz="0 1 0"/>
+			<limit lower="-4.36" upper="4.36" effort="0" velocity="3.32"/>
+		</joint>
 		<joint name="${prefix}joint_3" type="revolute">
-			<origin
-			  xyz="0 -0.0225 0.6"
-    		  rpy="0 0 0" />
-			<parent
-			  link="link_2" />
-			<child
-			  link="link_3" />
-			<axis
-			  xyz="0 1 0" />
-			<limit
-			  lower="-5.06"
-			  upper="5.06"
-			  effort="0"
-			  velocity="3.665" />
-			<calibration
-			  rising="0"
-			  falling="0" />
-			<dynamics
-			  damping="0"
-			  friction="0" />
-<!--			<safety_controller
-			  soft_lower_limit="0"
-			  soft_upper_limit="0"
-			  k_position="0"
-			  k_velocity="0" /> -->
+			<origin xyz="0 -0.0225 0.6" rpy="0 0 0"/>
+			<parent link="link_2"/>
+			<child link="link_3"/>
+			<axis xyz="0 1 0"/>
+			<limit lower="-5.06" upper="5.06" effort="0" velocity="3.665"/>
 		</joint>
 		<joint name="${prefix}joint_4" type="revolute">
-			<origin
-			  xyz="0.1805 0.0625 0.2"
-    		  rpy="0 0 0" />
-			<parent
-			  link="link_3" />
-			<child
-			  link="link_4" />
-			<axis
-			  xyz="1 0 0" />
-			<limit
-			  lower="-6.63"
-			  upper="6.63"
-			  effort="0"
-			  velocity="6.98" />
-			<calibration
-			  rising="0"
-			  falling="0" />
-			<dynamics
-			  damping="0"
-			  friction="0" />
-<!--			<safety_controller
-			  soft_lower_limit="0"
-			  soft_upper_limit="0"
-			  k_position="0"
-			  k_velocity="0" /> -->
+			<origin xyz="0.1805 0.0625 0.2" rpy="0 0 0"/>
+			<parent link="link_3"/>
+			<child link="link_4"/>
+			<axis xyz="1 0 0"/>
+			<limit lower="-6.63" upper="6.63" effort="0" velocity="6.98"/>
 		</joint>
 		<joint name="${prefix}joint_5" type="revolute">
-			<origin
-			  xyz="0.4595 -0.0565 0"
-      		  rpy="0 0 0" />
-			<parent
-			  link="link_4" />
-			<child
-			  link="link_5" />
-			<axis
-			  xyz="0 1 0" />
-			<limit
-			  lower="-6.63"
-			  upper="6.63"
-			  effort="0"
-			  velocity="3.98" />
-			<calibration
-			  rising="0"
-			  falling="0" />
-			<dynamics
-			  damping="0"
-			  friction="0" />
-<!--			<safety_controller
-			  soft_lower_limit="0"
-			  soft_upper_limit="0"
-			  k_position="0"
-			  k_velocity="0" /> -->
+			<origin xyz="0.4595 -0.0565 0" rpy="0 0 0"/>
+			<parent link="link_4"/>
+			<child link="link_5"/>
+			<axis xyz="0 1 0"/>
+			<limit lower="-6.63" upper="6.63" effort="0" velocity="3.98"/>
 		</joint>
 		<joint name="${prefix}joint_6" type="revolute">
-			<origin
-			  xyz="0.1 0.0565 0"
-    		  rpy="0 0 0" />
-			<parent
-			  link="link_5" />
-			<child
-			  link="link_6" />
-			<axis
-			  xyz="1 0 0" />
-			<limit
-			  lower="-12.566"
-			  upper="12.566"
-			  effort="0"
-			  velocity="10.47" />
-			<calibration
-			  rising="0"
-			  falling="0" />
-			<dynamics
-			  damping="0"
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