Commit message: Manually merged trunk revisions r1233 (URDF formatting and robot mesh colours), r1234 (m430 incorrect joint limits), r1279 (update m430 meshes) and r1280 (minor launch file updates) into fanuc stack in fuerte dev branch.

File: branches/fuerte_dev/fanuc/fanuc_config/urdf/m_430iA2F_macro.xacro (robot description, xacro)
@@ -1,20 +1,20 @@
-<?xml version="1.0" ?>
+<?xml version="1.0"?>
 <robot xmlns:xacro="http://ros.org/wiki/xacro">
-    <xacro:macro name="m430iA2F" params="prefix">
-        <!-- links -->
+	<xacro:macro name="m430iA2F" params="prefix">
+		<!-- links -->
 		<link name="${prefix}base_link">
 			<visual>
-				<origin xyz="0 0 0" rpy="0 0 0" />
+				<origin xyz="0 0 0" rpy="0 0 0"/>
 				<geometry>
-					<mesh filename="package://fanuc_config/meshes/m_430iA/visual/base_link.stl" />
+					<mesh filename="package://fanuc_config/meshes/m_430iA/visual/base_link.stl"/>
 				</geometry>
 				<material name="white">
-					<color rgba="1 1 1 1" />
+					<color rgba="0.9 0.9 0.9 1"/>
 				</material>
 			</visual>
 			<collision>
-				<origin xyz="0 0 0" rpy="0 0 0" />
+				<origin xyz="0 0 0" rpy="0 0 0"/>
 				<geometry>
-					<mesh filename="package://fanuc_config/meshes/m_430iA/collision/base_link.stl" />
+					<mesh filename="package://fanuc_config/meshes/m_430iA/collision/base_link.stl"/>
 				</geometry>
 			</collision>
@@ -22,16 +22,16 @@
 		<link name="${prefix}link_1">
 			<visual>
-				<origin xyz="0 0 0" rpy="0 0 0" />
+				<origin xyz="0 0 0" rpy="0 0 0"/>
 				<geometry>
-					<mesh filename="package://fanuc_config/meshes/m_430iA/visual/link_1.stl" />
+					<mesh filename="package://fanuc_config/meshes/m_430iA/visual/link_1.stl"/>
 				</geometry>
 				<material name="">
-					<color rgba="0.89804 0.89804 0.89804 1" />
+					<color rgba="0.89804 0.89804 0.89804 1"/>
 				</material>
 			</visual>
 			<collision>
-				<origin xyz="0 0 0" rpy="0 0 0" />
+				<origin xyz="0 0 0" rpy="0 0 0"/>
 				<geometry>
-					<mesh filename="package://fanuc_config/meshes/m_430iA/collision/link_1.stl" />
+					<mesh filename="package://fanuc_config/meshes/m_430iA/collision/link_1.stl"/>
 				</geometry>
 			</collision>
@@ -39,16 +39,16 @@
 		<link name="${prefix}link_2">
 			<visual>
-				<origin xyz="0 0 0" rpy="0 0 0" />
+				<origin xyz="0 0 0" rpy="0 0 0"/>
 				<geometry>
-					<mesh filename="package://fanuc_config/meshes/m_430iA/visual/link_2.stl" />
+					<mesh filename="package://fanuc_config/meshes/m_430iA/visual/link_2.stl"/>
 				</geometry>
 				<material name="">
-					<color rgba="0.89804 0.89804 0.89804 1" />
+					<color rgba="0.89804 0.89804 0.89804 1"/>
 				</material>
 			</visual>
 			<collision>
-				<origin xyz="0 0 0" rpy="0 0 0" />
+				<origin xyz="0 0 0" rpy="0 0 0"/>
 				<geometry>
-					<mesh filename="package://fanuc_config/meshes/m_430iA/collision/link_2.stl" />
+					<mesh filename="package://fanuc_config/meshes/m_430iA/collision/link_2.stl"/>
 				</geometry>
 			</collision>
@@ -56,16 +56,22 @@
 		<link name="${prefix}link_3">
 			<visual>
-				<origin xyz="0 0 0.053" rpy="0 0 0" />
+				<!-- coordinate origin for link_3 is not at mate centre, -->
+				<!-- so compensate (53mm dZ between link_3-link_2 mate -->
+				<!-- and coordinate origin) -->
+				<!-- origin xyz="0 0 0" rpy="0 0 0"/ -->
+				<origin xyz="0 0 0.053" rpy="0 0 0"/>
 				<geometry>
-					<mesh filename="package://fanuc_config/meshes/m_430iA/visual/link_3.stl" />
+					<mesh filename="package://fanuc_config/meshes/m_430iA/visual/link_3.stl"/>
 				</geometry>
 				<material name="">
-					<color rgba="0.89804 0.89804 0.89804 1" />
+					<color rgba="0.89804 0.89804 0.89804 1"/>
 				</material>
 			</visual>
 			<collision>
-				<origin xyz="0 0 0.053" rpy="0 0 0" />
+				<!-- see earlier comment -->
+				<!-- origin xyz="0 0 0" rpy="0 0 0"/ -->
+				<origin xyz="0 0 0.053" rpy="0 0 0"/>
 				<geometry>
-					<mesh filename="package://fanuc_config/meshes/m_430iA/collision/link_3.stl" />
+					<mesh filename="package://fanuc_config/meshes/m_430iA/collision/link_3.stl"/>
 				</geometry>
 			</collision>
@@ -73,16 +79,16 @@
 		<link name="${prefix}link_4">
 			<visual>
-				<origin xyz="0 0 0" rpy="0 0 0" />
+				<origin xyz="0 0 0" rpy="0 0 0"/>
 				<geometry>
-					<mesh filename="package://fanuc_config/meshes/m_430iA/visual/link_4.stl" />
+					<mesh filename="package://fanuc_config/meshes/m_430iA/visual/link_4.stl"/>
 				</geometry>
 				<material name="">
-					<color rgba="0.89804 0.89804 0.89804 1" />
+					<color rgba="0.89804 0.89804 0.89804 1"/>
 				</material>
 			</visual>
 			<collision>
-				<origin xyz="0 0 0" rpy="0 0 0" />
+				<origin xyz="0 0 0" rpy="0 0 0"/>
 				<geometry>
-					<mesh filename="package://fanuc_config/meshes/m_430iA/collision/link_4.stl" />
+					<mesh filename="package://fanuc_config/meshes/m_430iA/collision/link_4.stl"/>
 				</geometry>
 			</collision>
@@ -90,88 +96,65 @@
 		<link name="${prefix}link_5">
 			<visual>
-				<origin xyz="0 0 0" rpy="0 0 0" />
+				<origin xyz="0 0 0" rpy="0 0 0"/>
 				<geometry>
-					<mesh filename="package://fanuc_config/meshes/m_430iA/visual/link_5.stl" />
+					<mesh filename="package://fanuc_config/meshes/m_430iA/visual/link_5.stl"/>
 				</geometry>
 				<material name="">
-					<color rgba="0.75294 0.75294 0.75294 1" />
+					<color rgba="0.75294 0.75294 0.75294 1"/>
 				</material>
 			</visual>
 			<collision>
-				<origin xyz="0 0 0" rpy="0 0 0" />
+				<origin xyz="0 0 0" rpy="0 0 0"/>
 				<geometry>
-					<mesh filename="package://fanuc_config/meshes/m_430iA/collision/link_5.stl" />
+					<mesh filename="package://fanuc_config/meshes/m_430iA/collision/link_5.stl"/>
 				</geometry>
 			</collision>
 		</link>
-        <link name="${prefix}tool0"/>
-        <!-- joints -->
-        <joint name="${prefix}joint_1" type="revolute">
-            <origin xyz="-6.0758E-19 1.2493E-16 0.44" rpy="0 0 0" />
-            <parent link="${prefix}base_link" />
-            <child link="${prefix}link_1" />
-            <axis xyz="0 0 1" />
-            <limit lower="-3.1415" upper="3.1415" effort="0"
-                velocity="5.23598775598" />
-            <!-- calibration rising="0" falling="0" />
-            <dynamics damping="0" friction="0" />
-            <safety_controller soft_lower_limit="0"
-                soft_upper_limit="0" k_position="0" k_velocity="0" / -->
-        </joint>
-        <joint name="${prefix}joint_2" type="revolute">
-            <origin xyz="-1.4097E-17 0.171 -4.4409E-16" rpy="0 0 0" />
-            <parent link="${prefix}link_1" />
-            <child link="${prefix}link_2" />
-            <axis xyz="0 1 0" />
-            <limit lower="-2.00707" upper="2.00707" effort="0"
-                velocity="5.58505360638" />
-            <!-- calibration rising="0" falling="0" />
-            <dynamics damping="0" friction="0" />
-            <safety_controller soft_lower_limit="0"
-                soft_upper_limit="0" k_position="0" k_velocity="0" / -->
-        </joint>
-        <joint name="${prefix}joint_3" type="revolute">
-            <!-- origin xyz="1.2197E-19 -0.171 0.403" rpy="0 0 0" / -->
-            <origin xyz="1.2197E-19 -0.171 0.350" rpy="0 0 0" />
-            <parent link="${prefix}link_2" />
-            <child link="${prefix}link_3" />
-            <axis xyz="0 1 0" />
-            <limit lower="-1.771457" upper="1.771457" effort="0"
-                velocity="5.58505360638" />
-            <!-- calibration rising="0" falling="0" />
-            <dynamics damping="0" friction="0" />
-            <safety_controller soft_lower_limit="0"
-                soft_upper_limit="0" k_position="0" k_velocity="0" / -->
-        </joint>
-        <joint name="${prefix}joint_4" type="revolute">
-            <!-- origin xyz="-2.6075E-17 -0.06 0.497" rpy="0 0 0" / -->
-            <origin xyz="-2.6075E-17 -0.06 0.55" rpy="0 0 0" />
-            <parent link="${prefix}link_3" />
-            <child link="${prefix}link_4" />
-            <axis xyz="0 1 0" />
-            <limit lower="-2.617917" upper="2.617917" effort="0"
-                velocity="6.28318530718" />
-            <!-- calibration rising="0" falling="0" />
-            <dynamics damping="0" friction="0" />
-            <safety_controller soft_lower_limit="0"
-                soft_upper_limit="0" k_position="0" k_velocity="0" / -->
-        </joint>
+		<link name="${prefix}tool0"/>
+		<!-- joints -->
+		<joint name="${prefix}joint_1" type="revolute">
+			<origin xyz="0 0 0.44" rpy="0 0 0"/>
+			<parent link="${prefix}base_link"/>
+			<child link="${prefix}link_1"/>
+			<axis xyz="0 0 1"/>
+			<limit lower="-3.1415" upper="3.1415" effort="0" velocity="5.24"/>
+		</joint>
+		<joint name="${prefix}joint_2" type="revolute">
+			<origin xyz="0 0.171 0" rpy="0 0 0"/>
+			<parent link="${prefix}link_1"/>
+			<child link="${prefix}link_2"/>
+			<axis xyz="0 1 0"/>
+			<limit lower="-2.01" upper="2.01" effort="0" velocity="5.59"/>
+		</joint>
+		<joint name="${prefix}joint_3" type="revolute">
+			<!-- see earlier comment -->
+			<!-- origin xyz="0 -0.171 0.403" rpy="0 0 0"/ -->
+			<origin xyz="0 -0.171 0.35" rpy="0 0 0"/>
+			<parent link="${prefix}link_2"/>
+			<child link="${prefix}link_3"/>
+			<axis xyz="0 1 0"/>
+			<limit lower="-3.34" upper="3.34" effort="0" velocity="5.59"/>
+		</joint>
+		<joint name="${prefix}joint_4" type="revolute">
+			<!-- see earlier comment -->
+			<!-- origin xyz="0 -0.06 0.497" rpy="0 0 0"/ -->
+			<origin xyz="0 -0.06 0.55" rpy="0 0 0"/>
+			<parent link="${prefix}link_3"/>
+			<child link="${prefix}link_4"/>
+			<axis xyz="0 1 0"/>
+			<limit lower="-2.62" upper="2.62" effort="0" velocity="6.28"/>
+		</joint>
 		<joint name="${prefix}joint_5" type="revolute">
-			<origin xyz="1.4734E-16 -0.035 0.065" rpy="0 0 0" />
-			<parent link="${prefix}link_4" />
-			<child link="${prefix}link_5" />
-			<axis xyz="0 0 1" />
-			<limit lower="-4.71225" upper="4.71225" effort="0"
-                velocity="20.9439510239" />
-            <!-- calibration rising="0" falling="0" />
-            <dynamics damping="0" friction="0" />
-            <safety_controller soft_lower_limit="0"
-                soft_upper_limit="0" k_position="0" k_velocity="0" / -->
+			<origin xyz="0 -0.035 0.065" rpy="0 0 0"/>
+			<parent link="${prefix}link_4"/>
+			<child link="${prefix}link_5"/>
+			<axis xyz="0 0 1"/>
+			<limit lower="-4.71" upper="4.71" effort="0" velocity="20.94"/>
 		</joint>
-        <joint name="${prefix}joint_5-tool0" type="fixed">
-            <parent link="${prefix}link_5"/>
-            <child link="${prefix}tool0"/>
-            <origin xyz="0 0 0" rpy="0 0 0"/>
-        </joint>
-    </xacro:macro>
+		<joint name="${prefix}joint_5-tool0" type="fixed">
+			<parent link="${prefix}link_5"/>
+			<child link="${prefix}tool0"/>
+			<origin xyz="0 0 0" rpy="0 0 0"/>
+		</joint>
+	</xacro:macro>
 </robot>
