Commit message: corrected lower joint limit so that it's not a larger value that the upper joint limit.  Regenerated urdf file to reflect changes in xacro

File: branches/fuerte_dev/fanuc/fanuc_config/urdf/M16iB20.urdf (robot description, URDF)
Before this commit: robot M16iB20, 8 links, 7 joints
Joints:
- joint joint_2: limit lower=-1.39 upper=2.78 effort=0 velocity=2.8 -> lower=-1.38 upper=2.78 effort=0 velocity=2.8
- joint joint_3: limit lower=-4.21 upper=1.45 effort=0 velocity=3.0 -> lower=-4.08 upper=1.38 effort=0 velocity=3.0
- joint joint_5: limit lower=-2.44 upper=2.44 effort=0 velocity=5.9 -> lower=-2.43 upper=2.43 effort=0 velocity=5.9
- joint joint_6: axis -1 0 -0.0013212 -> -1 0 0; limit lower=-7.85 upper=7.85 effort=0 velocity=9.0 -> lower=-7.84 upper=7.84 effort=0 velocity=9.0

File: branches/fuerte_dev/fanuc/fanuc_config/urdf/M16iB20_macro.xacro (robot description, xacro)
@@ -343,5 +343,5 @@
 		      xyz="0 -1 0" />
 		    <limit
-		      lower="4.08"
+		      lower="-4.08"
 		      upper="1.38"
 		      effort="0"

Commit message: Merging trunk changes in fanuc package.

File: branches/fuerte_dev/fanuc/fanuc_config/urdf/M16iB20.urdf (robot description, URDF)
Before this commit: robot M16iB20, 8 links, 7 joints
Links:
- link base_link: mass 48654.354928172 -> None
- link link_1: mass 48654.354928172 -> None
- link link_2: mass 48654.354928172 -> None
- link link_3: mass 48654.354928172 -> None
- link link_4: mass 48654.354928172 -> None
- link link_5: mass 48654.354928172 -> None
- link link_6: mass 48654.354928172 -> None
Joints:
- joint joint_1: limit lower=-2.967 upper=2.967 effort=0 velocity=2.8 -> lower=-2.967 upper=2.967 effort=0 velocity=2.879; origin xyz=0 0 0.24477 rpy=0 0 0 -> xyz=0 0 0.245 rpy=0 0 0
- joint joint_2: limit lower=-1.38 upper=2.78 effort=0 velocity=2.8 -> lower=-1.38 upper=2.78 effort=0 velocity=2.879
- joint joint_3: limit lower=-4.08 upper=1.38 effort=0 velocity=3.0 -> lower=-4.08 upper=1.38 effort=0 velocity=3.054; origin xyz=0 -0.18815 0.77 rpy=0 0 0 -> xyz=0 -0.18759 0.77 rpy=0 0 0
- joint joint_4: limit lower=-3.48 upper=3.48 effort=0 velocity=6.1 -> lower=-3.48 upper=3.48 effort=0 velocity=6.108; origin xyz=0.1847 0 0.1 rpy=0 0 0 -> xyz=0.18425 0 0.1 rpy=0 0 0
- joint joint_5: limit lower=-2.43 upper=2.43 effort=0 velocity=5.9 -> lower=-2.43 upper=2.43 effort=0 velocity=5.934; origin xyz=0.55575 0.00019326 0.00073427 rpy=0 0 0 -> xyz=0.55575 0 0 rpy=0 0 0
- joint joint_6: limit lower=-7.84 upper=7.84 effort=0 velocity=9.0 -> lower=-7.84 upper=7.84 effort=0 velocity=9.075; origin xyz=0.10014 0 0.00013231 rpy=0 0 0 -> xyz=0.1 0 0 rpy=0 0 0

File: branches/fuerte_dev/fanuc/fanuc_config/urdf/M16iB20_macro.xacro (robot description, xacro)
@@ -4,18 +4,4 @@
 	<!-- links -->
 		  <link name="${prefix}base_link">
-		    <inertial>
-		      <origin
-			xyz="0 9.68920591007408E-05 0.538248432765216"
-			rpy="0 0 0" />
-		      <mass
-			value="48654.354928172" />
-		      <inertia
-			ixx="51563.7946245021"
-			ixy="0.552841467322453"
-			ixz="-212.267889356987"
-			iyy="49495.9076886951"
-			iyz="1.80688027777408"
-			izz="54368.3241585813" />
-		    </inertial>
 		    <visual>
 		      <origin
@@ -43,18 +29,4 @@
 		  </link>
 		  <link name="${prefix}link_1">
-		    <inertial>
-		      <origin
-			xyz="0.0335399435995477 9.68920591007463E-05 0.293476071945811"
-			rpy="0 0 0" />
-		      <mass
-			value="48654.354928172" />
-		      <inertia
-			ixx="51563.7946245021"
-			ixy="0.552841467322453"
-			ixz="-212.267889356987"
-			iyy="49495.9076886951"
-			iyz="1.80688027777408"
-			izz="54368.3241585813" />
-		    </inertial>
 		    <visual>
 		      <origin
@@ -82,18 +54,4 @@
 		  </link>
 		  <link name="${prefix}link_2">
-		    <inertial>
-		      <origin
-			xyz="-0.116459985096576 -0.187496105761522 0.0134762050463809"
-			rpy="0 0 0" />
-		      <mass
-			value="48654.354928172" />
-		      <inertia
-			ixx="51563.7946245021"
-			ixy="0.552841467322453"
-			ixz="-212.267889356987"
-			iyy="49495.9076886951"
-			iyz="1.80688027777408"
-			izz="54368.3241585813" />
-		    </inertial>
 		    <visual>
 		      <origin
@@ -121,18 +79,4 @@
 		  </link>
 		  <link name="${prefix}link_3">
-		    <inertial>
-		      <origin
-			xyz="-0.116459985097232 0.000649393837860671 -0.7565234388513"
-			rpy="0 0 0" />
-		      <mass
-			value="48654.354928172" />
-		      <inertia
-			ixx="51563.7946245021"
-			ixy="0.552841467322453"
-			ixz="-212.267889356987"
-			iyy="49495.9076886951"
-			iyz="1.80688027777408"
-			izz="54368.3241585813" />
-		    </inertial>
 		    <visual>
 		      <origin
@@ -160,18 +104,4 @@
 		  </link>
 		  <link name="${prefix}link_4">
-		    <inertial>
-		      <origin
-			xyz="-0.301157421773673 0.000649393837861561 -0.856523437562654"
-			rpy="0 0 0" />
-		      <mass
-			value="48654.354928172" />
-		      <inertia
-			ixx="51563.7946245021"
-			ixy="0.552841467322453"
-			ixz="-212.267889356987"
-			iyy="49495.9076886951"
-			iyz="1.80688027777408"
-			izz="54368.3241585813" />
-		    </inertial>
 		    <visual>
 		      <origin
@@ -199,18 +129,4 @@
 		  </link>
 		  <link name="${prefix}link_5">
-		    <inertial>
-		      <origin
-			xyz="-0.856906936709003 0.000456131051686355 -0.857257705801685"
-			rpy="0 0 0" />
-		      <mass
-			value="48654.354928172" />
-		      <inertia
-			ixx="51563.7946245021"
-			ixy="0.552841467322453"
-			ixz="-212.267889356987"
-			iyy="49495.9076886951"
-			iyz="1.80688027777408"
-			izz="54368.3241585813" />
-		    </inertial>
 		    <visual>
 		      <origin
@@ -238,18 +154,4 @@
 		  </link>
 		  <link name="${prefix}link_6">
-		    <inertial>
-		      <origin
-			xyz="-0.957051849301239 0.000456131051686355 -0.857390019418947"
-			rpy="0 0 0" />
-		      <mass
-			value="48654.354928172" />
-		      <inertia
-			ixx="51563.7946245021"
-			ixy="0.552841467322453"
-			ixz="-212.267889356987"
-			iyy="49495.9076886951"
-			iyz="1.80688027777408"
-			izz="54368.3241585813" />
-		    </inertial>
 		    <visual>
 		      <origin
@@ -276,9 +178,9 @@
 		    </collision>
 		  </link>
-        	  <link name="${prefix}tool0"/>
+          <link name="${prefix}tool0"/>
 	<!-- joints -->
 		  <joint name="${prefix}joint_1" type="revolute">
 		    <origin
-		      xyz="0 0 0.24477"
+		      xyz="0 0 0.245"
 		      rpy="0 0 0" />
 		    <parent
@@ -292,16 +194,5 @@
 		      upper="2.967"
 		      effort="0"
-		      velocity="2.8" />
-		    <calibration
-		      rising="0"
-		      falling="0" />
-		    <dynamics
-		      damping="0"
-		      friction="0" />
-		    <!--safety_controller
-		      soft_lower_limit="0"
-		      soft_upper_limit="0"
-		      k_position="0"
-		      k_velocity="0" /-->
+		      velocity="2.879" />
 		  </joint>
 		  <joint name="${prefix}joint_2" type="revolute">
@@ -319,20 +210,9 @@
 		      upper="2.78"
 		      effort="0"
-		      velocity="2.8" />
-		    <calibration
-		      rising="0"
-		      falling="0" />
-		    <dynamics
-		      damping="0"
-		      friction="0" />
-		    <!--safety_controller
-		      soft_lower_limit="0"
-		      soft_upper_limit="0"
-		      k_position="0"
-		      k_velocity="0" /-->
+		      velocity="2.879" />
 		  </joint>
 		  <joint name="${prefix}joint_3" type="revolute">
 		    <origin
-		      xyz="0 -0.18815 0.77"
+		      xyz="0 -0.18759 0.77"
 		      rpy="0 0 0" />
 		    <parent
@@ -346,20 +226,9 @@
 		      upper="1.38"
 		      effort="0"
-		      velocity="3.0" />
-		    <calibration
-		      rising="0"
-		      falling="0" />
-		    <dynamics
-		      damping="0"
-		      friction="0" />
-		    <!--safety_controller
-		      soft_lower_limit="0"
-		      soft_upper_limit="0"
-		      k_position="0"
-		      k_velocity="0" /-->
+		      velocity="3.054" />
 		  </joint>
 		  <joint name="${prefix}joint_4" type="revolute">
 		    <origin
-		      xyz="0.1847 0 0.1"
+		      xyz="0.18425 0 0.1"
 		      rpy="0 0 0" />
 		    <parent
@@ -373,20 +242,9 @@
 		      upper="3.48"
 		      effort="0"
-		      velocity="6.1" />
-		    <calibration
-		      rising="0"
-		      falling="0" />
-		    <dynamics
-		      damping="0"
-		      friction="0" />
-		    <!--safety_controller
-		      soft_lower_limit="0"
-		      soft_upper_limit="0"
-		      k_position="0"
-		      k_velocity="0" /-->
+		      velocity="6.108" />
 		  </joint>
 		  <joint name="${prefix}joint_5" type="revolute">
 		    <origin
-		      xyz="0.55575 0.00019326 0.00073427"
+		      xyz="0.55575 0 0"
 		      rpy="0 0 0" />
 		    <parent
@@ -400,20 +258,9 @@
 		      upper="2.43"
 		      effort="0"
-		      velocity="5.9" />
-		    <calibration
-		      rising="0"
-		      falling="0" />
-		    <dynamics
-		      damping="0"
-		      friction="0" />
-		    <!--safety_controller
-		      soft_lower_limit="0"
-		      soft_upper_limit="0"
-		      k_position="0"
-		      k_velocity="0" /-->
+		      velocity="5.934" />
 		  </joint>
 		  <joint name="${prefix}joint_6" type="revolute">
 		    <origin
-		      xyz="0.10014 0 0.00013231"
+		      xyz="0.1 0 0"
 		      rpy="0 0 0" />
 		    <parent
@@ -427,16 +274,5 @@
 		      upper="7.84"
 		      effort="0"
-		      velocity="9.0" />
-		    <calibration
-		      rising="0"
-		      falling="0" />
-		    <dynamics
-		      damping="0"
-		      friction="0" />
-		    <!--safety_controller
-		      soft_lower_limit="0"
-		      soft_upper_limit="0"
-		      k_position="0"
-		      k_velocity="0" /-->
+		      velocity="9.075" />
 		  </joint>
 		  <joint name="${prefix}joint_6-tool0" type="fixed">

Commit message: Backport fix for incorrect M-16iB/20 joint limits from trunk Fanuc into fuerte-dev branch.
NB: manual merge.

File: branches/fuerte_dev/fanuc/fanuc_config/urdf/M16iB20.urdf (robot description, URDF)
Before this commit: robot M16iB20, 8 links, 7 joints
Joints:
- joint joint_1: limit lower=-2.967 upper=2.967 effort=0 velocity=2.879 -> lower=-2.9671 upper=2.9671 effort=0 velocity=2.8798
- joint joint_2: limit lower=-1.38 upper=2.78 effort=0 velocity=2.879 -> lower=-1.5708 upper=2.7925 effort=0 velocity=2.8798
- joint joint_3: limit lower=-4.08 upper=1.38 effort=0 velocity=3.054 -> lower=-2.9671 upper=5.0615 effort=0 velocity=3.0543
- joint joint_4: limit lower=-3.48 upper=3.48 effort=0 velocity=6.108 -> lower=-3.4907 upper=3.4907 effort=0 velocity=6.1087
- joint joint_5: limit lower=-2.43 upper=2.43 effort=0 velocity=5.934 -> lower=-2.4435 upper=2.4435 effort=0 velocity=5.9341
- joint joint_6: limit lower=-7.84 upper=7.84 effort=0 velocity=9.075 -> lower=-7.8540 upper=7.8540 effort=0 velocity=9.0757

File: branches/fuerte_dev/fanuc/fanuc_config/urdf/M16iB20_macro.xacro (robot description, xacro)
@@ -119,5 +119,5 @@
 			<child link="link_1"/>
 			<axis xyz="0 0 1"/>
-			<limit lower="-2.967" upper="2.967" effort="0" velocity="2.879"/>
+			<limit effort="0" lower="-2.9671" upper="2.9671" velocity="2.8798" />
 		</joint>
 		<joint name="${prefix}joint_2" type="revolute">
@@ -126,5 +126,5 @@
 			<child link="link_2"/>
 			<axis xyz="0 1 0"/>
-			<limit lower="-1.38" upper="2.78" effort="0" velocity="2.879"/>
+			<limit effort="0" lower="-1.5708" upper="2.7925" velocity="2.8798" />
 		</joint>
 		<joint name="${prefix}joint_3" type="revolute">
@@ -133,5 +133,5 @@
 			<child link="link_3"/>
 			<axis xyz="0 -1 0"/>
-			<limit lower="-4.08" upper="1.38" effort="0" velocity="3.054"/>
+		<limit effort="0" lower="-2.9671" upper="5.0615" velocity="3.0543" />
 		</joint>
 		<joint name="${prefix}joint_4" type="revolute">
@@ -140,5 +140,5 @@
 			<child link="link_4"/>
 			<axis xyz="-1 0 0"/>
-			<limit lower="-3.48" upper="3.48" effort="0" velocity="6.108"/>
+			<limit effort="0" lower="-3.4907" upper="3.4907" velocity="6.1087" />
 		</joint>
 		<joint name="${prefix}joint_5" type="revolute">
@@ -147,5 +147,5 @@
 			<child link="link_5"/>
 			<axis xyz="0 -1 0"/>
-			<limit lower="-2.43" upper="2.43" effort="0" velocity="5.934"/>
+			<limit effort="0" lower="-2.4435" upper="2.4435" velocity="5.9341" />
 		</joint>
 		<joint name="${prefix}joint_6" type="revolute">
@@ -154,5 +154,5 @@
 			<child link="link_6"/>
 			<axis xyz="-1 0 0"/>
-			<limit lower="-7.84" upper="7.84" effort="0" velocity="9.075"/>
+			<limit effort="0" lower="-7.8540" upper="7.8540" velocity="9.0757" />
 		</joint>
 		<joint name="${prefix}joint_6-tool0" type="fixed">
