Commit message: Reverting problematic merge of changes from Fanuc trunk.

File: branches/groovy/fanuc/fanuc_config/urdf/M16iB20.urdf (robot description, URDF)
Before this commit: robot m16ib20, 8 links, 7 joints
Links:
- link base_link: geometry collision mesh filename=package://fanuc_config/meshes/m_16iB20/collision/base_link.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; visual mesh filename=package://fanuc_config/meshes/m_16iB20/visual/base_link.STL
- link link_1: geometry collision mesh filename=package://fanuc_config/meshes/m_16iB20/collision/Link_1.STL; visual mesh filename=package://fanuc_config/meshes/m_16iB20/visual/Link_1.STL
- link link_2: geometry collision mesh filename=package://fanuc_config/meshes/m_16iB20/collision/Link_2.STL; visual mesh filename=package://fanuc_config/meshes/m_16iB20/visual/Link_2.STL
- link link_3: geometry collision mesh filename=package://fanuc_config/meshes/m_16iB20/collision/Link_3.STL; visual mesh filename=package://fanuc_config/meshes/m_16iB20/visual/Link_3.STL
- link link_4: geometry collision mesh filename=package://fanuc_config/meshes/m_16iB20/collision/Link_4.STL; visual mesh filename=package://fanuc_config/meshes/m_16iB20/visual/Link_4.STL
- link link_5: geometry collision mesh filename=package://fanuc_config/meshes/m_16iB20/collision/Link_5.STL; visual mesh filename=package://fanuc_config/meshes/m_16iB20/visual/Link_5.STL
- link link_6: geometry collision mesh filename=package://fanuc_config/meshes/m_16iB20/collision/Link_6.STL; visual mesh filename=package://fanuc_config/meshes/m_16iB20/visual/Link_6.STL

File: branches/groovy/fanuc/fanuc_config/urdf/M16iB20.xacro (robot description, xacro)
@@ -1,5 +1,5 @@
 <?xml version="1.0" ?>
-<robot name="m16ib20" xmlns:xacro="http://ros.org/wiki/xacro">
-	<include filename="$(find fanuc_config)/urdf/m16ib20_macro.xacro"/>
-	<xacro:m16ib20 prefix=""/>
+<robot name="M16iB20" xmlns:xacro="http://ros.org/wiki/xacro">
+	<include filename="$(find fanuc_config)/urdf/M16iB20_macro.xacro"/>
+	<xacro:M16iB20 prefix=""/>
 </robot>

File: branches/groovy/fanuc/fanuc_config/urdf/M16iB20_macro.xacro (robot description, xacro)
@@ -1,164 +1,284 @@
 <?xml version="1.0" ?>
 <robot xmlns:xacro="http://ros.org/wiki/xacro">
-	<xacro:macro name="m16ib20" params="prefix">
-		<!-- links -->
-		<link name="${prefix}base_link">
-			<visual>
-				<origin xyz="0 0 0" rpy="0 0 0"/>
-				<geometry>
-					<mesh filename="package://fanuc_config/meshes/m16ib20/visual/base_link.STL"/>
-				</geometry>
-				<material name="fyel">
-					<color rgba="0.9 0.9 0 1" />
-				</material>
-			</visual>
-			<collision>
-				<origin xyz="0 0 0" rpy="0 0 0"/>
-				<geometry>
-					<mesh filename="package://fanuc_config/meshes/m16ib20/collision/base_link.STL"/>
-				</geometry>
-			</collision>
-		</link>
-		<link name="${prefix}link_1">
-			<visual>
-				<origin xyz="0 0 0" rpy="0 0 0"/>
-				<geometry>
-					<mesh filename="package://fanuc_config/meshes/m16ib20/visual/Link_1.STL"/>
-				</geometry>
-				<material name="fyel" />
-			</visual>
-			<collision>
-				<origin xyz="0 0 0" rpy="0 0 0"/>
-				<geometry>
-					<mesh filename="package://fanuc_config/meshes/m16ib20/collision/Link_1.STL"/>
-				</geometry>
-			</collision>
-		</link>
-		<link name="${prefix}link_2">
-			<visual>
-				<origin xyz="0 0 0" rpy="0 0 0"/>
-				<geometry>
-					<mesh filename="package://fanuc_config/meshes/m16ib20/visual/Link_2.STL"/>
-				</geometry>
-				<material name="fyel" />
-			</visual>
-			<collision>
-				<origin xyz="0 0 0" rpy="0 0 0"/>
-				<geometry>
-					<mesh filename="package://fanuc_config/meshes/m16ib20/collision/Link_2.STL"/>
-				</geometry>
-			</collision>
-		</link>
-		<link name="${prefix}link_3">
-			<visual>
-				<origin xyz="0 0 0" rpy="0 0 0"/>
-				<geometry>
-					<mesh filename="package://fanuc_config/meshes/m16ib20/visual/Link_3.STL"/>
-				</geometry>
-				<material name="fyel" />
-			</visual>
-			<collision>
-				<origin xyz="0 0 0" rpy="0 0 0"/>
-				<geometry>
-					<mesh filename="package://fanuc_config/meshes/m16ib20/collision/Link_3.STL"/>
-				</geometry>
-			</collision>
-		</link>
-		<link name="${prefix}link_4">
-			<visual>
-				<origin xyz="0 0 0" rpy="0 0 0"/>
-				<geometry>
-					<mesh filename="package://fanuc_config/meshes/m16ib20/visual/Link_4.STL"/>
-				</geometry>
-				<material name="fyel" />
-			</visual>
-			<collision>
-				<origin xyz="0 0 0" rpy="0 0 0"/>
-				<geometry>
-					<mesh filename="package://fanuc_config/meshes/m16ib20/collision/Link_4.STL"/>
-				</geometry>
-			</collision>
-		</link>
-		<link name="${prefix}link_5">
-			<visual>
-				<origin xyz="0 0 0" rpy="0 0 0"/>
-				<geometry>
-					<mesh filename="package://fanuc_config/meshes/m16ib20/visual/Link_5.STL"/>
-				</geometry>
-				<material name="fyel" />
-			</visual>
-			<collision>
-				<origin xyz="0 0 0" rpy="0 0 0"/>
-				<geometry>
-					<mesh filename="package://fanuc_config/meshes/m16ib20/collision/Link_5.STL"/>
-				</geometry>
-			</collision>
-		</link>
-		<link name="${prefix}link_6">
-			<visual>
-				<origin xyz="0 0 0" rpy="0 0 0"/>
-				<geometry>
-					<mesh filename="package://fanuc_config/meshes/m16ib20/visual/Link_6.STL"/>
-				</geometry>
-				<material name="fblack">
-					<color rgba="0.1 0.1 0.1 1"/>
-				</material>
-			</visual>
-			<collision>
-				<origin xyz="0 0 0" rpy="0 0 0"/>
-				<geometry>
-					<mesh filename="package://fanuc_config/meshes/m16ib20/collision/Link_6.STL"/>
-				</geometry>
-			</collision>
-		</link>
-		<link name="${prefix}tool0"/>
-		<!-- joints -->
-		<joint name="${prefix}joint_1" type="revolute">
-			<origin xyz="0 0 0.245" rpy="0 0 0"/>
-			<parent link="base_link"/>
-			<child link="link_1"/>
-			<axis xyz="0 0 1"/>
-			<limit lower="-2.967" upper="2.967" effort="0" velocity="2.879"/>
-		</joint>
-		<joint name="${prefix}joint_2" type="revolute">
-			<origin xyz="0.15 0.18759 0.28" rpy="0 0 0"/>
-			<parent link="link_1"/>
-			<child link="link_2"/>
-			<axis xyz="0 1 0"/>
-			<limit lower="-1.38" upper="2.78" effort="0" velocity="2.879"/>
-		</joint>
-		<joint name="${prefix}joint_3" type="revolute">
-			<origin xyz="0 -0.18759 0.77" rpy="0 0 0"/>
-			<parent link="link_2"/>
-			<child link="link_3"/>
-			<axis xyz="0 -1 0"/>
-			<limit lower="-4.08" upper="1.38" effort="0" velocity="3.054"/>
-		</joint>
-		<joint name="${prefix}joint_4" type="revolute">
-			<origin xyz="0.18425 0 0.1" rpy="0 0 0"/>
-			<parent link="link_3"/>
-			<child link="link_4"/>
-			<axis xyz="-1 0 0"/>
-			<limit lower="-3.48" upper="3.48" effort="0" velocity="6.108"/>
-		</joint>
-		<joint name="${prefix}joint_5" type="revolute">
-			<origin xyz="0.55575 0 0" rpy="0 0 0"/>
-			<parent link="link_4"/>
-			<child link="link_5"/>
-			<axis xyz="0 -1 0"/>
-			<limit lower="-2.43" upper="2.43" effort="0" velocity="5.934"/>
-		</joint>
-		<joint name="${prefix}joint_6" type="revolute">
-			<origin xyz="0.1 0 0" rpy="0 0 0"/>
-			<parent link="link_5"/>
-			<child link="link_6"/>
-			<axis xyz="-1 0 0"/>
-			<limit lower="-7.84" upper="7.84" effort="0" velocity="9.075"/>
-		</joint>
-		<joint name="${prefix}joint_6-tool0" type="fixed">
-			<parent link="${prefix}link_6"/>
-			<child link="${prefix}tool0"/>
-			<origin xyz="0 0 0" rpy="0 0 0"/>
-		</joint>
+	<xacro:macro name="M16iB20" params="prefix">
+	<!-- links -->
+		  <link name="${prefix}base_link">
+		    <visual>
+		      <origin
+			xyz="0 0 0"
+			rpy="0 0 0" />
+		      <geometry>
+			<mesh
+			  filename="package://fanuc_config/meshes/m_16iB20/visual/base_link.STL" />
+		      </geometry>
+		      <material
+			name="">
+			<color
+			  rgba="1 1 0 1" />
+		      </material>
+		    </visual>
+		    <collision>
+		      <origin
+			xyz="0 0 0"
+			rpy="0 0 0" />
+		      <geometry>
+			<mesh
+			  filename="package://fanuc_config/meshes/m_16iB20/collision/base_link.STL" />
+		      </geometry>
+		    </collision>
+		  </link>
+		  <link name="${prefix}link_1">
+		    <visual>
+		      <origin
+			xyz="0 0 0"
+			rpy="0 0 0" />
+		      <geometry>
+			<mesh
+			  filename="package://fanuc_config/meshes/m_16iB20/visual/Link_1.STL" />
+		      </geometry>
+		      <material
+			name="">
+			<color
+			  rgba="1 1 0 1" />
+		      </material>
+		    </visual>
+		    <collision>
+		      <origin
+			xyz="0 0 0"
+			rpy="0 0 0" />
+		      <geometry>
+			<mesh
+			  filename="package://fanuc_config/meshes/m_16iB20/collision/Link_1.STL" />
+		      </geometry>
+		    </collision>
+		  </link>
+		  <link name="${prefix}link_2">
+		    <visual>
+		      <origin
+			xyz="0 0 0"
+			rpy="0 0 0" />
+		      <geometry>
+			<mesh
+			  filename="package://fanuc_config/meshes/m_16iB20/visual/Link_2.STL" />
+		      </geometry>
+		      <material
+			name="">
+			<color
+			  rgba="1 1 0 1" />
+		      </material>
+		    </visual>
+		    <collision>
+		      <origin
+			xyz="0 0 0"
+			rpy="0 0 0" />
+		      <geometry>
+			<mesh
+			  filename="package://fanuc_config/meshes/m_16iB20/collision/Link_2.STL" />
+		      </geometry>
+		    </collision>
+		  </link>
+		  <link name="${prefix}link_3">
+		    <visual>
+		      <origin
+			xyz="0 0 0"
+			rpy="0 0 0" />
+		      <geometry>
+			<mesh
+			  filename="package://fanuc_config/meshes/m_16iB20/visual/Link_3.STL" />
+		      </geometry>
+		      <material
+			name="">
+			<color
+			  rgba="1 1 0 1" />
+		      </material>
+		    </visual>
+		    <collision>
+		      <origin
+			xyz="0 0 0"
+			rpy="0 0 0" />
+		      <geometry>
+			<mesh
+			  filename="package://fanuc_config/meshes/m_16iB20/collision/Link_3.STL" />
+		      </geometry>
+		    </collision>
+		  </link>
+		  <link name="${prefix}link_4">
+		    <visual>
+		      <origin
+			xyz="0 0 0"
+			rpy="0 0 0" />
+		      <geometry>
+			<mesh
+			  filename="package://fanuc_config/meshes/m_16iB20/visual/Link_4.STL" />
+		      </geometry>
+		      <material
+			name="">
+			<color
+			  rgba="1 1 0 1" />
+		      </material>
+		    </visual>
+		    <collision>
+		      <origin
+			xyz="0 0 0"
+			rpy="0 0 0" />
+		      <geometry>
+			<mesh
+			  filename="package://fanuc_config/meshes/m_16iB20/collision/Link_4.STL" />
+		      </geometry>
+		    </collision>
+		  </link>
+		  <link name="${prefix}link_5">
+		    <visual>
+		      <origin
+			xyz="0 0 0"
+			rpy="0 0 0" />
+		      <geometry>
+			<mesh
+			  filename="package://fanuc_config/meshes/m_16iB20/visual/Link_5.STL" />
+		      </geometry>
+		      <material
+			name="">
+			<color
+			  rgba="1 1 0 1" />
+		      </material>
+		    </visual>
+		    <collision>
+		      <origin
+			xyz="0 0 0"
+			rpy="0 0 0" />
+		      <geometry>
+			<mesh
+			  filename="package://fanuc_config/meshes/m_16iB20/collision/Link_5.STL" />
+		      </geometry>
+		    </collision>
+		  </link>
+		  <link name="${prefix}link_6">
+		    <visual>
+		      <origin
+			xyz="0 0 0"
+			rpy="0 0 0" />
+		      <geometry>
+			<mesh
+			  filename="package://fanuc_config/meshes/m_16iB20/visual/Link_6.STL" />
+		      </geometry>
+		      <material
+			name="">
+			<color
+			  rgba="1 1 0 1" />
+		      </material>
+		    </visual>
+		    <collision>
+		      <origin
+			xyz="0 0 0"
+			rpy="0 0 0" />
+		      <geometry>
+			<mesh
+			  filename="package://fanuc_config/meshes/m_16iB20/collision/Link_6.STL" />
+		      </geometry>
+		    </collision>
+		  </link>
+          <link name="${prefix}tool0"/>
+	<!-- joints -->
+		  <joint name="${prefix}joint_1" type="revolute">
+		    <origin
+		      xyz="0 0 0.245"
+		      rpy="0 0 0" />
+		    <parent
+		      link="base_link" />
+		    <child
+		      link="link_1" />
+		    <axis
+		      xyz="0 0 1" />
+		    <limit
+		      lower="-2.967"
+		      upper="2.967"
+		      effort="0"
+		      velocity="2.879" />
+		  </joint>
+		  <joint name="${prefix}joint_2" type="revolute">
+		    <origin
+		      xyz="0.15 0.18759 0.28"
+		      rpy="0 0 0" />
+		    <parent
+		      link="link_1" />
+		    <child
+		      link="link_2" />
+		    <axis
+		      xyz="0 1 0" />
+		    <limit
+		      lower="-1.38"
+		      upper="2.78"
+		      effort="0"
+		      velocity="2.879" />
+		  </joint>
+		  <joint name="${prefix}joint_3" type="revolute">
+		    <origin
+		      xyz="0 -0.18759 0.77"
+		      rpy="0 0 0" />
+		    <parent
+		      link="link_2" />
+		    <child
+		      link="link_3" />
+		    <axis
+		      xyz="0 -1 0" />
+		    <limit
+		      lower="-4.08"
+		      upper="1.38"
+		      effort="0"
+		      velocity="3.054" />
+		  </joint>
+		  <joint name="${prefix}joint_4" type="revolute">
+		    <origin
+		      xyz="0.18425 0 0.1"
+		      rpy="0 0 0" />
+		    <parent
+		      link="link_3" />
+		    <child
+		      link="link_4" />
+		    <axis
+		      xyz="-1 0 0" />
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
File: branches/groovy/fanuc/fanuc_config/urdf/m10iA.urdf (robot description, URDF)
Before this commit: robot m10ia, 8 links, 7 joints
Links:
- link base_link: geometry collision mesh filename=package://fanuc_config/meshes/m_10iA/collision/base_link.stl; visual mesh filename=package://fanuc_config/meshes/m_10iA/visual/base_link.stl
- link link_1: geometry collision mesh filename=package://fanuc_config/meshes/m_10iA/collision/link_1.stl; visual mesh filename=package://fanuc_config/meshes/m_10iA/visual/link_1.stl
- link link_2: geometry collision mesh filename=package://fanuc_config/meshes/m_10iA/collision/link_2.stl; visual mesh filename=package://fanuc_config/meshes/m_10iA/visual/link_2.stl
- link link_3: geometry collision mesh filename=package://fanuc_config/meshes/m_10iA/collision/link_3.stl; visual mesh filename=package://fanuc_config/meshes/m_10iA/visual/link_3.stl
- link link_4: geometry collision mesh filename=package://fanuc_config/meshes/m_10iA/collision/link_4.stl; visual mesh filename=package://fanuc_config/meshes/m_10iA/visual/link_4.stl
- link link_5: geometry collision mesh filename=package://fanuc_config/meshes/m_10iA/collision/link_5.stl; visual mesh filename=package://fanuc_config/meshes/m_10iA/visual/link_5.stl
- link link_6: geometry collision mesh filename=package://fanuc_config/meshes/m_10iA/collision/link_6.stl; visual mesh filename=package://fanuc_config/meshes/m_10iA/visual/link_6.stl

File: branches/groovy/fanuc/fanuc_config/urdf/m10iA.xacro (robot description, xacro)
@@ -1,5 +1,5 @@
 <?xml version="1.0" ?>
-<robot name="m10ia" xmlns:xacro="http://ros.org/wiki/xacro">
-	<include filename="$(find fanuc_config)/urdf/m10ia_macro.xacro"/>
-	<xacro:m10ia prefix=""/>
+<robot name="m10iA" xmlns:xacro="http://ros.org/wiki/xacro">
+	<include filename="$(find fanuc_config)/urdf/m_10iA_macro.xacro"/>
+	<xacro:m10iA prefix=""/>
 </robot>

File: branches/groovy/fanuc/fanuc_config/urdf/m430iA2F.urdf (robot description, URDF)
Before this commit: robot m430ia2f, 7 links, 6 joints
Links:
- link base_link: geometry collision mesh filename=package://fanuc_config/meshes/m_430iA/collision/base_link.s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; visual mesh filename=package://fanuc_config/meshes/m_430iA/visual/base_link.stl
- link link_1: geometry collision mesh filename=package://fanuc_config/meshes/m_430iA/collision/link_1.stl; visual mesh filename=package://fanuc_config/meshes/m_430iA/visual/link_1.stl
- link link_2: geometry collision mesh filename=package://fanuc_config/meshes/m_430iA/collision/link_2.stl; visual mesh filename=package://fanuc_config/meshes/m_430iA/visual/link_2.stl
- link link_3: geometry collision mesh filename=package://fanuc_config/meshes/m_430iA/collision/link_3.stl; visual mesh filename=package://fanuc_config/meshes/m_430iA/visual/link_3.stl
- link link_4: geometry collision mesh filename=package://fanuc_config/meshes/m_430iA/collision/link_4.stl; visual mesh filename=package://fanuc_config/meshes/m_430iA/visual/link_4.stl
- link link_5: geometry collision mesh filename=package://fanuc_config/meshes/m_430iA/collision/link_5.stl; visual mesh filename=package://fanuc_config/meshes/m_430iA/visual/link_5.stl
Joints:
- joint joint_1: limit lower=-3.1415 upper=3.1415 effort=0 velocity=5.24 -> lower=-3.1415 upper=3.1415 effort=0 velocity=5.23598775598
- joint joint_2: limit lower=-2.01 upper=2.01 effort=0 velocity=5.59 -> lower=-2.00707 upper=2.00707 effort=0 velocity=5.58505360638
- joint joint_3: limit lower=-3.49 upper=3.49 effort=0 velocity=5.59 -> lower=-1.771457 upper=1.771457 effort=0 velocity=5.58505360638
- joint joint_4: limit lower=-2.62 upper=2.62 effort=0 velocity=6.28 -> lower=-2.617917 upper=2.617917 effort=0 velocity=6.28318530718
- joint joint_5: limit lower=-4.71 upper=4.71 effort=0 velocity=20.94 -> lower=-4.71225 upper=4.71225 effort=0 velocity=20.9439510239

File: branches/groovy/fanuc/fanuc_config/urdf/m430iA2F.xacro (robot description, xacro)
@@ -1,5 +1,5 @@
 <?xml version="1.0" ?>
-<robot name="m430ia2f" xmlns:xacro="http://ros.org/wiki/xacro">
-	<include filename="$(find fanuc_config)/urdf/m430ia2f_macro.xacro"/>
-	<xacro:m430ia2f prefix=""/>
+<robot name="m430iA2F" xmlns:xacro="http://ros.org/wiki/xacro">
+	<include filename="$(find fanuc_config)/urdf/m_430iA2F_macro.xacro"/>
+	<xacro:m430iA2F prefix=""/>
 </robot>
