Commit message: Update model support packages for the M-10iA, M-16iB and the M-430iA to work with the new package layout.
Also remove files and references from other models not supported by the packages (ie: remove m10ia from m430ia package).

File: branches/fanuc_pkg_rename/fanuc_m10ia_support/urdf/m10ia.urdf (robot description, URDF)
Before this commit: robot m10ia, 8 links, 7 joints
Links:
- link base_link: geometry collision mesh filename=package://fanuc_m10ia_support/meshes/m10ia/collision/base_l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; visual mesh filename=package://fanuc_m10ia_support/meshes/m10ia/visual/base_link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
- link link_1: geometry collision mesh filename=package://fanuc_m10ia_support/meshes/m10ia/collision/link_1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; visual mesh filename=package://fanuc_m10ia_support/meshes/m10ia/visual/link_1.stl
- link link_2: geometry collision mesh filename=package://fanuc_m10ia_support/meshes/m10ia/collision/link_2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; visual mesh filename=package://fanuc_m10ia_support/meshes/m10ia/visual/link_2.stl
- link link_3: geometry collision mesh filename=package://fanuc_m10ia_support/meshes/m10ia/collision/link_3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; visual mesh filename=package://fanuc_m10ia_support/meshes/m10ia/visual/link_3.stl
- link link_4: geometry collision mesh filename=package://fanuc_m10ia_support/meshes/m10ia/collision/link_4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; visual mesh filename=package://fanuc_m10ia_support/meshes/m10ia/visual/link_4.stl
- link link_5: geometry collision mesh filename=package://fanuc_m10ia_support/meshes/m10ia/collision/link_5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; visual mesh filename=package://fanuc_m10ia_support/meshes/m10ia/visual/link_5.stl
- link link_6: geometry collision mesh filename=package://fanuc_m10ia_support/meshes/m10ia/collision/link_6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; visual mesh filename=package://fanuc_m10ia_support/meshes/m10ia/visual/link_6.stl

File: branches/fanuc_pkg_rename/fanuc_m10ia_support/urdf/m10ia.xacro (robot description, xacro)
@@ -1,5 +1,5 @@
 <?xml version="1.0" ?>
-<robot name="m10ia" xmlns:xacro="http://ros.org/wiki/xacro">
-	<include filename="$(find fanuc_config)/urdf/m10ia_macro.xacro"/>
-	<xacro:m10ia prefix=""/>
+<robot name="fanuc_m10ia" xmlns:xacro="http://ros.org/wiki/xacro">
+	<include filename="$(find fanuc_m10ia_support)/urdf/m10ia_macro.xacro"/>
+	<xacro:fanuc_m10ia prefix=""/>
 </robot>

File: branches/fanuc_pkg_rename/fanuc_m10ia_support/urdf/m10ia_macro.xacro (robot description, xacro)
@@ -1,5 +1,5 @@
 <?xml version="1.0"?>
 <robot xmlns:xacro="http://ros.org/wiki/xacro">
-	<xacro:macro name="m10ia" params="prefix">
+	<xacro:macro name="fanuc_m10ia" params="prefix">
 		<!-- links -->
 		<link name="${prefix}base_link">
@@ -7,5 +7,5 @@
 				<origin xyz="0 0 0" rpy="-1.578 0 0"/>
 				<geometry>
-					<mesh filename="package://fanuc_config/meshes/m10ia/visual/base_link.stl"/>
+					<mesh filename="package://fanuc_m10ia_support/meshes/m10ia/visual/base_link.stl"/>
 				</geometry>
 				<material name="fgrey">
@@ -16,5 +16,5 @@
 				<origin xyz="0 0 0" rpy="-1.578 0 0"/>
 				<geometry>
-					<mesh filename="package://fanuc_config/meshes/m10ia/collision/base_link.stl"/>
+					<mesh filename="package://fanuc_m10ia_support/meshes/m10ia/collision/base_link.stl"/>
 				</geometry>
 			</collision>
@@ -24,5 +24,5 @@
 				<origin xyz="0 0 0" rpy="0 0 0"/>
 				<geometry>
-					<mesh filename="package://fanuc_config/meshes/m10ia/visual/link_1.stl"/>
+					<mesh filename="package://fanuc_m10ia_support/meshes/m10ia/visual/link_1.stl"/>
 				</geometry>
 				<material name="fyel">
@@ -33,5 +33,5 @@
 				<origin xyz="0 0 0" rpy="0 0 0"/>
 				<geometry>
-					<mesh filename="package://fanuc_config/meshes/m10ia/collision/link_1.stl"/>
+					<mesh filename="package://fanuc_m10ia_support/meshes/m10ia/collision/link_1.stl"/>
 				</geometry>
 			</collision>
@@ -41,5 +41,5 @@
 				<origin xyz="0 0 0" rpy="0 0 0"/>
 				<geometry>
-					<mesh filename="package://fanuc_config/meshes/m10ia/visual/link_2.stl"/>
+					<mesh filename="package://fanuc_m10ia_support/meshes/m10ia/visual/link_2.stl"/>
 				</geometry>
 				<material name="fyel"/>
@@ -48,5 +48,5 @@
 				<origin xyz="0 0 0" rpy="0 0 0"/>
 				<geometry>
-					<mesh filename="package://fanuc_config/meshes/m10ia/collision/link_2.stl"/>
+					<mesh filename="package://fanuc_m10ia_support/meshes/m10ia/collision/link_2.stl"/>
 				</geometry>
 			</collision>
@@ -56,5 +56,5 @@
 				<origin xyz="0 0 0" rpy="0 0 0"/>
 				<geometry>
-					<mesh filename="package://fanuc_config/meshes/m10ia/visual/link_3.stl"/>
+					<mesh filename="package://fanuc_m10ia_support/meshes/m10ia/visual/link_3.stl"/>
 				</geometry>
 				<material name="fyel"/>
@@ -63,5 +63,5 @@
 				<origin xyz="0 0 0" rpy="0 0 0"/>
 				<geometry>
-					<mesh filename="package://fanuc_config/meshes/m10ia/collision/link_3.stl"/>
+					<mesh filename="package://fanuc_m10ia_support/meshes/m10ia/collision/link_3.stl"/>
 				</geometry>
 			</collision>
@@ -71,5 +71,5 @@
 				<origin xyz="0 0 0" rpy="0 0 0"/>
 				<geometry>
-					<mesh filename="package://fanuc_config/meshes/m10ia/visual/link_4.stl"/>
+					<mesh filename="package://fanuc_m10ia_support/meshes/m10ia/visual/link_4.stl"/>
 				</geometry>
 				<material name="fyel"/>
@@ -78,5 +78,5 @@
 				<origin xyz="0 0 0" rpy="0 0 0"/>
 				<geometry>
-					<mesh filename="package://fanuc_config/meshes/m10ia/collision/link_4.stl"/>
+					<mesh filename="package://fanuc_m10ia_support/meshes/m10ia/collision/link_4.stl"/>
 				</geometry>
 			</collision>
@@ -86,5 +86,5 @@
 				<origin xyz="0 0 0" rpy="0 0 0"/>
 				<geometry>
-					<mesh filename="package://fanuc_config/meshes/m10ia/visual/link_5.stl"/>
+					<mesh filename="package://fanuc_m10ia_support/meshes/m10ia/visual/link_5.stl"/>
 				</geometry>
 				<material name="fyel"/>
@@ -93,5 +93,5 @@
 				<origin xyz="0 0 0" rpy="0 0 0"/>
 				<geometry>
-					<mesh filename="package://fanuc_config/meshes/m10ia/collision/link_5.stl"/>
+					<mesh filename="package://fanuc_m10ia_support/meshes/m10ia/collision/link_5.stl"/>
 				</geometry>
 			</collision>
@@ -101,5 +101,5 @@
 				<origin xyz="0 0 0" rpy="0 0 0"/>
 				<geometry>
-					<mesh filename="package://fanuc_config/meshes/m10ia/visual/link_6.stl"/>
+					<mesh filename="package://fanuc_m10ia_support/meshes/m10ia/visual/link_6.stl"/>
 				</geometry>
 				<material name="fblack">
@@ -110,5 +110,5 @@
 				<origin xyz="0 0 0" rpy="0 0 0"/>
 				<geometry>
-					<mesh filename="package://fanuc_config/meshes/m10ia/collision/link_6.stl"/>
+					<mesh filename="package://fanuc_m10ia_support/meshes/m10ia/collision/link_6.stl"/>
 				</geometry>
 			</collision>

File: branches/fanuc_pkg_rename/fanuc_m16ib_support/urdf/m16ib20.urdf (robot description, URDF)
Before this commit: robot m16ib20, 8 links, 7 joints
Links:
- link base_link: geometry collision mesh filename=package://fanuc_m16ib_support/meshes/m16ib20/collision/base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; visual mesh filename=package://fanuc_m16ib_support/meshes/m16ib20/visual/base_li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
- link link_1: geometry collision mesh filename=package://fanuc_m16ib_support/meshes/m16ib20/collision/Link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; visual mesh filename=package://fanuc_m16ib_support/meshes/m16ib20/visual/Link_1.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
- link link_2: geometry collision mesh filename=package://fanuc_m16ib_support/meshes/m16ib20/collision/Link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; visual mesh filename=package://fanuc_m16ib_support/meshes/m16ib20/visual/Link_2.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
- link link_3: geometry collision mesh filename=package://fanuc_m16ib_support/meshes/m16ib20/collision/Link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; visual mesh filename=package://fanuc_m16ib_support/meshes/m16ib20/visual/Link_3.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
- link link_4: geometry collision mesh filename=package://fanuc_m16ib_support/meshes/m16ib20/collision/Link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; visual mesh filename=package://fanuc_m16ib_support/meshes/m16ib20/visual/Link_4.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
- link link_5: geometry collision mesh filename=package://fanuc_m16ib_support/meshes/m16ib20/collision/Link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; visual mesh filename=package://fanuc_m16ib_support/meshes/m16ib20/visual/Link_5.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
- link link_6: geometry collision mesh filename=package://fanuc_m16ib_support/meshes/m16ib20/collision/Link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; visual mesh filename=package://fanuc_m16ib_support/meshes/m16ib20/visual/Link_6.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

File: branches/fanuc_pkg_rename/fanuc_m16ib_support/urdf/m16ib20.xacro (robot description, xacro)
@@ -1,5 +1,5 @@
 <?xml version="1.0" ?>
-<robot name="m16ib20" xmlns:xacro="http://ros.org/wiki/xacro">
-	<include filename="$(find fanuc_config)/urdf/m16ib20_macro.xacro"/>
-	<xacro:m16ib20 prefix=""/>
+<robot name="fanuc_m16ib20" xmlns:xacro="http://ros.org/wiki/xacro">
+	<include filename="$(find fanuc_m16ib_support)/urdf/m16ib20_macro.xacro"/>
+	<xacro:fanuc_m16ib20 prefix=""/>
 </robot>

File: branches/fanuc_pkg_rename/fanuc_m16ib_support/urdf/m16ib20_macro.xacro (robot description, xacro)
@@ -1,5 +1,5 @@
 <?xml version="1.0" ?>
 <robot xmlns:xacro="http://ros.org/wiki/xacro">
-	<xacro:macro name="m16ib20" params="prefix">
+	<xacro:macro name="fanuc_m16ib20" params="prefix">
 		<!-- links -->
 		<link name="${prefix}base_link">
@@ -7,5 +7,5 @@
 				<origin xyz="0 0 0" rpy="0 0 0"/>
 				<geometry>
-					<mesh filename="package://fanuc_config/meshes/m16ib20/visual/base_link.STL"/>
+					<mesh filename="package://fanuc_m16ib_support/meshes/m16ib20/visual/base_link.STL"/>
 				</geometry>
 				<material name="fyel">
@@ -16,5 +16,5 @@
 				<origin xyz="0 0 0" rpy="0 0 0"/>
 				<geometry>
-					<mesh filename="package://fanuc_config/meshes/m16ib20/collision/base_link.STL"/>
+					<mesh filename="package://fanuc_m16ib_support/meshes/m16ib20/collision/base_link.STL"/>
 				</geometry>
 			</collision>
@@ -24,5 +24,5 @@
 				<origin xyz="0 0 0" rpy="0 0 0"/>
 				<geometry>
-					<mesh filename="package://fanuc_config/meshes/m16ib20/visual/Link_1.STL"/>
+					<mesh filename="package://fanuc_m16ib_support/meshes/m16ib20/visual/Link_1.STL"/>
 				</geometry>
 				<material name="fyel" />
@@ -31,5 +31,5 @@
 				<origin xyz="0 0 0" rpy="0 0 0"/>
 				<geometry>
-					<mesh filename="package://fanuc_config/meshes/m16ib20/collision/Link_1.STL"/>
+					<mesh filename="package://fanuc_m16ib_support/meshes/m16ib20/collision/Link_1.STL"/>
 				</geometry>
 			</collision>
@@ -39,5 +39,5 @@
 				<origin xyz="0 0 0" rpy="0 0 0"/>
 				<geometry>
-					<mesh filename="package://fanuc_config/meshes/m16ib20/visual/Link_2.STL"/>
+					<mesh filename="package://fanuc_m16ib_support/meshes/m16ib20/visual/Link_2.STL"/>
 				</geometry>
 				<material name="fyel" />
@@ -46,5 +46,5 @@
 				<origin xyz="0 0 0" rpy="0 0 0"/>
 				<geometry>
-					<mesh filename="package://fanuc_config/meshes/m16ib20/collision/Link_2.STL"/>
+					<mesh filename="package://fanuc_m16ib_support/meshes/m16ib20/collision/Link_2.STL"/>
 				</geometry>
 			</collision>
@@ -54,5 +54,5 @@
 				<origin xyz="0 0 0" rpy="0 0 0"/>
 				<geometry>
-					<mesh filename="package://fanuc_config/meshes/m16ib20/visual/Link_3.STL"/>
+					<mesh filename="package://fanuc_m16ib_support/meshes/m16ib20/visual/Link_3.STL"/>
 				</geometry>
 				<material name="fyel" />
@@ -61,5 +61,5 @@
 				<origin xyz="0 0 0" rpy="0 0 0"/>
 				<geometry>
-					<mesh filename="package://fanuc_config/meshes/m16ib20/collision/Link_3.STL"/>
+					<mesh filename="package://fanuc_m16ib_support/meshes/m16ib20/collision/Link_3.STL"/>
 				</geometry>
 			</collision>
@@ -69,5 +69,5 @@
 				<origin xyz="0 0 0" rpy="0 0 0"/>
 				<geometry>
-					<mesh filename="package://fanuc_config/meshes/m16ib20/visual/Link_4.STL"/>
+					<mesh filename="package://fanuc_m16ib_support/meshes/m16ib20/visual/Link_4.STL"/>
 				</geometry>
 				<material name="fyel" />
@@ -76,5 +76,5 @@
 				<origin xyz="0 0 0" rpy="0 0 0"/>
 				<geometry>
-					<mesh filename="package://fanuc_config/meshes/m16ib20/collision/Link_4.STL"/>
+					<mesh filename="package://fanuc_m16ib_support/meshes/m16ib20/collision/Link_4.STL"/>
 				</geometry>
 			</collision>
@@ -84,5 +84,5 @@
 				<origin xyz="0 0 0" rpy="0 0 0"/>
 				<geometry>
-					<mesh filename="package://fanuc_config/meshes/m16ib20/visual/Link_5.STL"/>
+					<mesh filename="package://fanuc_m16ib_support/meshes/m16ib20/visual/Link_5.STL"/>
 				</geometry>
 				<material name="fyel" />
@@ -91,5 +91,5 @@
 				<origin xyz="0 0 0" rpy="0 0 0"/>
 				<geometry>
-					<mesh filename="package://fanuc_config/meshes/m16ib20/collision/Link_5.STL"/>
+					<mesh filename="package://fanuc_m16ib_support/meshes/m16ib20/collision/Link_5.STL"/>
 				</geometry>
 			</collision>
@@ -99,5 +99,5 @@
 				<origin xyz="0 0 0" rpy="0 0 0"/>
 				<geometry>
-					<mesh filename="package://fanuc_config/meshes/m16ib20/visual/Link_6.STL"/>
+					<mesh filename="package://fanuc_m16ib_support/meshes/m16ib20/visual/Link_6.STL"/>
 				</geometry>
 				<material name="fblack">
@@ -108,5 +108,5 @@
 				<origin xyz="0 0 0" rpy="0 0 0"/>
 				<geometry>
-					<mesh filename="package://fanuc_config/meshes/m16ib20/collision/Link_6.STL"/>
+					<mesh filename="package://fanuc_m16ib_support/meshes/m16ib20/collision/Link_6.STL"/>
 				</geometry>
 			</collision>

File: branches/fanuc_pkg_rename/fanuc_m430ia_support/urdf/m430ia2f.urdf (robot description, URDF)
Before this commit: robot m430ia2f, 7 links, 6 joints
Links:
- link base_link: geometry collision mesh filename=package://fanuc_m430ia_support/meshes/m430ia2f/collision/ba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; visual mesh filename=package://fanuc_m430ia_support/meshes/m430ia2f/visual/base_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
- link link_1: geometry collision mesh filename=package://fanuc_m430ia_support/meshes/m430ia2f/collision/li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; visual mesh filename=package://fanuc_m430ia_support/meshes/m430ia2f/visual/link_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
- link link_2: geometry collision mesh filename=package://fanuc_m430ia_support/meshes/m430ia2f/collision/li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; visual mesh filename=package://fanuc_m430ia_support/meshes/m430ia2f/visual/link_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
- link link_3: geometry collision mesh filename=package://fanuc_m430ia_support/meshes/m430ia2f/collision/li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; visual mesh filename=package://fanuc_m430ia_support/meshes/m430ia2f/visual/link_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
- link link_4: geometry collision mesh filename=package://fanuc_m430ia_support/meshes/m430ia2f/collision/li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; visual mesh filename=package://fanuc_m430ia_support/meshes/m430ia2f/visual/link_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
- link link_5: geometry collision mesh filename=package://fanuc_m430ia_support/meshes/m430ia2f/collision/li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; visual mesh filename=package://fanuc_m430ia_support/meshes/m430ia2f/visual/link_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

File: branches/fanuc_pkg_rename/fanuc_m430ia_support/urdf/m430ia2f.xacro (robot description, xacro)
@@ -1,5 +1,5 @@
 <?xml version="1.0" ?>
-<robot name="m430ia2f" xmlns:xacro="http://ros.org/wiki/xacro">
-	<include filename="$(find fanuc_config)/urdf/m430ia2f_macro.xacro"/>
-	<xacro:m430ia2f prefix=""/>
+<robot name="fanuc_m430ia2f" xmlns:xacro="http://ros.org/wiki/xacro">
+	<include filename="$(find fanuc_m430ia_support)/urdf/m430ia2f_macro.xacro"/>
+	<xacro:fanuc_m430ia2f prefix=""/>
 </robot>

File: branches/fanuc_pkg_rename/fanuc_m430ia_support/urdf/m430ia2f_macro.xacro (robot description, xacro)
@@ -1,5 +1,5 @@
 <?xml version="1.0"?>
 <robot xmlns:xacro="http://ros.org/wiki/xacro">
-	<xacro:macro name="m430ia2f" params="prefix">
+	<xacro:macro name="fanuc_m430ia2f" params="prefix">
 		<!-- links -->
 		<link name="${prefix}base_link">
@@ -7,5 +7,5 @@
 				<origin xyz="0 0 0" rpy="0 0 0"/>
 				<geometry>
-					<mesh filename="package://fanuc_config/meshes/m430ia2f/visual/base_link.stl"/>
+					<mesh filename="package://fanuc_m430ia_support/meshes/m430ia2f/visual/base_link.stl"/>
 				</geometry>
 				<material name="white">
@@ -16,5 +16,5 @@
 				<origin xyz="0 0 0" rpy="0 0 0"/>
 				<geometry>
-					<mesh filename="package://fanuc_config/meshes/m430ia2f/collision/base_link.stl"/>
+					<mesh filename="package://fanuc_m430ia_support/meshes/m430ia2f/collision/base_link.stl"/>
 				</geometry>
 			</collision>
@@ -24,5 +24,5 @@
 				<origin xyz="0 0 0" rpy="0 0 0"/>
 				<geometry>
-					<mesh filename="package://fanuc_config/meshes/m430ia2f/visual/link_1.stl"/>
+					<mesh filename="package://fanuc_m430ia_support/meshes/m430ia2f/visual/link_1.stl"/>
 				</geometry>
 				<material name="">
@@ -33,5 +33,5 @@
 				<origin xyz="0 0 0" rpy="0 0 0"/>
 				<geometry>
-					<mesh filename="package://fanuc_config/meshes/m430ia2f/collision/link_1.stl"/>
+					<mesh filename="package://fanuc_m430ia_support/meshes/m430ia2f/collision/link_1.stl"/>
 				</geometry>
 			</collision>
@@ -41,5 +41,5 @@
 				<origin xyz="0 0 0" rpy="0 0 0"/>
 				<geometry>
-					<mesh filename="package://fanuc_config/meshes/m430ia2f/visual/link_2.stl"/>
+					<mesh filename="package://fanuc_m430ia_support/meshes/m430ia2f/visual/link_2.stl"/>
 				</geometry>
 				<material name="">
@@ -50,5 +50,5 @@
 				<origin xyz="0 0 0" rpy="0 0 0"/>
 				<geometry>
-					<mesh filename="package://fanuc_config/meshes/m430ia2f/collision/link_2.stl"/>
+					<mesh filename="package://fanuc_m430ia_support/meshes/m430ia2f/collision/link_2.stl"/>
 				</geometry>
 			</collision>
@@ -62,5 +62,5 @@
 				<origin xyz="0 0 0.053" rpy="0 0 0"/>
 				<geometry>
-					<mesh filename="package://fanuc_config/meshes/m430ia2f/visual/link_3.stl"/>
+					<mesh filename="package://fanuc_m430ia_support/meshes/m430ia2f/visual/link_3.stl"/>
 				</geometry>
 				<material name="">
@@ -73,5 +73,5 @@
 				<origin xyz="0 0 0.053" rpy="0 0 0"/>
 				<geometry>
-					<mesh filename="package://fanuc_config/meshes/m430ia2f/collision/link_3.stl"/>
+					<mesh filename="package://fanuc_m430ia_support/meshes/m430ia2f/collision/link_3.stl"/>
 				</geometry>
 			</collision>
@@ -81,5 +81,5 @@
 				<origin xyz="0 0 0" rpy="0 0 0"/>
 				<geometry>
-					<mesh filename="package://fanuc_config/meshes/m430ia2f/visual/link_4.stl"/>
+					<mesh filename="package://fanuc_m430ia_support/meshes/m430ia2f/visual/link_4.stl"/>
 				</geometry>
 				<material name="">
@@ -90,5 +90,5 @@
 				<origin xyz="0 0 0" rpy="0 0 0"/>
 				<geometry>
-					<mesh filename="package://fanuc_config/meshes/m430ia2f/collision/link_4.stl"/>
+					<mesh filename="package://fanuc_m430ia_support/meshes/m430ia2f/collision/link_4.stl"/>
 				</geometry>
 			</collision>
@@ -98,5 +98,5 @@
 				<origin xyz="0 0 0" rpy="0 0 0"/>
 				<geometry>
-					<mesh filename="package://fanuc_config/meshes/m430ia2f/visual/link_5.stl"/>
+					<mesh filename="package://fanuc_m430ia_support/meshes/m430ia2f/visual/link_5.stl"/>
 				</geometry>
 				<material name="">
@@ -107,5 +107,5 @@
 				<origin xyz="0 0 0" rpy="0 0 0"/>
 				<geometry>
-					<mesh filename="package://fanuc_config/meshes/m430ia2f/collision/link_5.stl"/>
+					<mesh filename="package://fanuc_m430ia_support/meshes/m430ia2f/collision/link_5.stl"/>
 				</geometry>
 			</collision>
