Commit message: Launchfile, xacro, urdf and CMakeLists.txt cleanup.
Formatting, layout and dependencies.

File: branches/fanuc_pkg_rename/fanuc_m10ia_support/urdf/m10ia_macro.xacro (robot description, xacro)
@@ -1,4 +1,5 @@
 <?xml version="1.0"?>
 <robot xmlns:xacro="http://ros.org/wiki/xacro">
+	<xacro:include filename="$(find fanuc_assets)/urdf/common_materials.xacro"/>
 	<xacro:macro name="fanuc_m10ia" params="prefix">
 		<!-- links -->
@@ -9,7 +10,5 @@
 					<mesh filename="package://fanuc_m10ia_support/meshes/m10ia/visual/base_link.stl"/>
 				</geometry>
-				<material name="fgrey">
-					<color rgba="0.20 0.20 0.20 1"/>
-				</material>
+				<xacro:material_fanuc_grey />
 			</visual>
 			<collision>
@@ -26,7 +25,5 @@
 					<mesh filename="package://fanuc_m10ia_support/meshes/m10ia/visual/link_1.stl"/>
 				</geometry>
-				<material name="fyel">
-					<color rgba="0.9 0.9 0 1"/>
-				</material>
+				<xacro:material_fanuc_yellow />
 			</visual>
 			<collision>
@@ -43,5 +40,5 @@
 					<mesh filename="package://fanuc_m10ia_support/meshes/m10ia/visual/link_2.stl"/>
 				</geometry>
-				<material name="fyel"/>
+				<xacro:material_fanuc_yellow />
 			</visual>
 			<collision>
@@ -58,5 +55,5 @@
 					<mesh filename="package://fanuc_m10ia_support/meshes/m10ia/visual/link_3.stl"/>
 				</geometry>
-				<material name="fyel"/>
+				<xacro:material_fanuc_yellow />
 			</visual>
 			<collision>
@@ -73,5 +70,5 @@
 					<mesh filename="package://fanuc_m10ia_support/meshes/m10ia/visual/link_4.stl"/>
 				</geometry>
-				<material name="fyel"/>
+				<xacro:material_fanuc_yellow />
 			</visual>
 			<collision>
@@ -88,5 +85,5 @@
 					<mesh filename="package://fanuc_m10ia_support/meshes/m10ia/visual/link_5.stl"/>
 				</geometry>
-				<material name="fyel"/>
+				<xacro:material_fanuc_yellow />
 			</visual>
 			<collision>
@@ -103,7 +100,5 @@
 					<mesh filename="package://fanuc_m10ia_support/meshes/m10ia/visual/link_6.stl"/>
 				</geometry>
-				<material name="fblack">
-					<color rgba="0.1 0.1 0.1 1"/>
-				</material>
+				<xacro:material_fanuc_black />
 			</visual>
 			<collision>

File: branches/fanuc_pkg_rename/fanuc_m16ib_support/urdf/m16ib20_macro.xacro (robot description, xacro)
@@ -1,4 +1,5 @@
 <?xml version="1.0" ?>
 <robot xmlns:xacro="http://ros.org/wiki/xacro">
+	<xacro:include filename="$(find fanuc_assets)/urdf/common_materials.xacro"/>
 	<xacro:macro name="fanuc_m16ib20" params="prefix">
 		<!-- links -->
@@ -9,7 +10,5 @@
 					<mesh filename="package://fanuc_m16ib_support/meshes/m16ib20/visual/base_link.STL"/>
 				</geometry>
-				<material name="fyel">
-					<color rgba="0.9 0.9 0 1" />
-				</material>
+				<xacro:material_fanuc_yellow />
 			</visual>
 			<collision>
@@ -26,5 +25,5 @@
 					<mesh filename="package://fanuc_m16ib_support/meshes/m16ib20/visual/Link_1.STL"/>
 				</geometry>
-				<material name="fyel" />
+				<xacro:material_fanuc_yellow />
 			</visual>
 			<collision>
@@ -41,5 +40,5 @@
 					<mesh filename="package://fanuc_m16ib_support/meshes/m16ib20/visual/Link_2.STL"/>
 				</geometry>
-				<material name="fyel" />
+				<xacro:material_fanuc_yellow />
 			</visual>
 			<collision>
@@ -56,5 +55,5 @@
 					<mesh filename="package://fanuc_m16ib_support/meshes/m16ib20/visual/Link_3.STL"/>
 				</geometry>
-				<material name="fyel" />
+				<xacro:material_fanuc_yellow />
 			</visual>
 			<collision>
@@ -71,5 +70,5 @@
 					<mesh filename="package://fanuc_m16ib_support/meshes/m16ib20/visual/Link_4.STL"/>
 				</geometry>
-				<material name="fyel" />
+				<xacro:material_fanuc_yellow />
 			</visual>
 			<collision>
@@ -86,5 +85,5 @@
 					<mesh filename="package://fanuc_m16ib_support/meshes/m16ib20/visual/Link_5.STL"/>
 				</geometry>
-				<material name="fyel" />
+				<xacro:material_fanuc_yellow />
 			</visual>
 			<collision>
@@ -101,7 +100,5 @@
 					<mesh filename="package://fanuc_m16ib_support/meshes/m16ib20/visual/Link_6.STL"/>
 				</geometry>
-				<material name="fblack">
-					<color rgba="0.1 0.1 0.1 1"/>
-				</material>
+				<xacro:material_fanuc_black />
 			</visual>
 			<collision>

File: branches/fanuc_pkg_rename/fanuc_m430ia_support/urdf/m430ia2f_macro.xacro (robot description, xacro)
@@ -1,4 +1,5 @@
 <?xml version="1.0"?>
 <robot xmlns:xacro="http://ros.org/wiki/xacro">
+	<include filename="$(find fanuc_assets)/urdf/common_materials.xacro"/>
 	<xacro:macro name="fanuc_m430ia2f" params="prefix">
 		<!-- links -->
@@ -9,7 +10,5 @@
 					<mesh filename="package://fanuc_m430ia_support/meshes/m430ia2f/visual/base_link.stl"/>
 				</geometry>
-				<material name="white">
-					<color rgba="0.9 0.9 0.9 1"/>
-				</material>
+				<xacro:material_fanuc_white />
 			</visual>
 			<collision>
@@ -26,7 +25,5 @@
 					<mesh filename="package://fanuc_m430ia_support/meshes/m430ia2f/visual/link_1.stl"/>
 				</geometry>
-				<material name="">
-					<color rgba="0.89804 0.89804 0.89804 1"/>
-				</material>
+				<xacro:material_fanuc_white />
 			</visual>
 			<collision>
@@ -43,7 +40,5 @@
 					<mesh filename="package://fanuc_m430ia_support/meshes/m430ia2f/visual/link_2.stl"/>
 				</geometry>
-				<material name="">
-					<color rgba="0.89804 0.89804 0.89804 1"/>
-				</material>
+				<xacro:material_fanuc_white />
 			</visual>
 			<collision>
@@ -64,7 +59,5 @@
 					<mesh filename="package://fanuc_m430ia_support/meshes/m430ia2f/visual/link_3.stl"/>
 				</geometry>
-				<material name="">
-					<color rgba="0.89804 0.89804 0.89804 1"/>
-				</material>
+				<xacro:material_fanuc_white />
 			</visual>
 			<collision>
@@ -83,7 +76,5 @@
 					<mesh filename="package://fanuc_m430ia_support/meshes/m430ia2f/visual/link_4.stl"/>
 				</geometry>
-				<material name="">
-					<color rgba="0.89804 0.89804 0.89804 1"/>
-				</material>
+				<xacro:material_fanuc_white />
 			</visual>
 			<collision>
@@ -100,7 +91,5 @@
 					<mesh filename="package://fanuc_m430ia_support/meshes/m430ia2f/visual/link_5.stl"/>
 				</geometry>
-				<material name="">
-					<color rgba="0.75294 0.75294 0.75294 1"/>
-				</material>
+				<xacro:material_fanuc_white />
 			</visual>
 			<collision>
