Commit message: Mesh STLs should be lower case, extension as well.
Also update XACRO & URDF.

File: branches/fanuc_pkg_rename/fanuc_m16ib_support/urdf/m16ib20.urdf (robot description, URDF)
Before this commit: robot fanuc_m16ib20, 8 links, 7 joints
Links:
- link link_1: geometry collision mesh filename=package://fanuc_m16ib_support/meshes/m16ib20/collision/link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; visual mesh filename=package://fanuc_m16ib_support/meshes/m16ib20/visual/link_1.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
- link link_2: geometry collision mesh filename=package://fanuc_m16ib_support/meshes/m16ib20/collision/link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; visual mesh filename=package://fanuc_m16ib_support/meshes/m16ib20/visual/link_2.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
- link link_3: geometry collision mesh filename=package://fanuc_m16ib_support/meshes/m16ib20/collision/link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; visual mesh filename=package://fanuc_m16ib_support/meshes/m16ib20/visual/link_3.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
- link link_4: geometry collision mesh filename=package://fanuc_m16ib_support/meshes/m16ib20/collision/link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; visual mesh filename=package://fanuc_m16ib_support/meshes/m16ib20/visual/link_4.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
- link link_5: geometry collision mesh filename=package://fanuc_m16ib_support/meshes/m16ib20/collision/link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; visual mesh filename=package://fanuc_m16ib_support/meshes/m16ib20/visual/link_5.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
- link link_6: geometry collision mesh filename=package://fanuc_m16ib_support/meshes/m16ib20/collision/link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; visual mesh filename=package://fanuc_m16ib_support/meshes/m16ib20/visual/link_6.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

File: branches/fanuc_pkg_rename/fanuc_m16ib_support/urdf/m16ib20_macro.xacro (robot description, xacro)
@@ -8,5 +8,5 @@
 				<origin xyz="0 0 0" rpy="0 0 0"/>
 				<geometry>
-					<mesh filename="package://fanuc_m16ib_support/meshes/m16ib20/visual/base_link.STL"/>
+					<mesh filename="package://fanuc_m16ib_support/meshes/m16ib20/visual/base_link.stl"/>
 				</geometry>
 				<xacro:material_fanuc_yellow />
@@ -15,5 +15,5 @@
 				<origin xyz="0 0 0" rpy="0 0 0"/>
 				<geometry>
-					<mesh filename="package://fanuc_m16ib_support/meshes/m16ib20/collision/base_link.STL"/>
+					<mesh filename="package://fanuc_m16ib_support/meshes/m16ib20/collision/base_link.stl"/>
 				</geometry>
 			</collision>
@@ -23,5 +23,5 @@
 				<origin xyz="0 0 0" rpy="0 0 0"/>
 				<geometry>
-					<mesh filename="package://fanuc_m16ib_support/meshes/m16ib20/visual/Link_1.STL"/>
+					<mesh filename="package://fanuc_m16ib_support/meshes/m16ib20/visual/link_1.stl"/>
 				</geometry>
 				<xacro:material_fanuc_yellow />
@@ -30,5 +30,5 @@
 				<origin xyz="0 0 0" rpy="0 0 0"/>
 				<geometry>
-					<mesh filename="package://fanuc_m16ib_support/meshes/m16ib20/collision/Link_1.STL"/>
+					<mesh filename="package://fanuc_m16ib_support/meshes/m16ib20/collision/link_1.stl"/>
 				</geometry>
 			</collision>
@@ -38,5 +38,5 @@
 				<origin xyz="0 0 0" rpy="0 0 0"/>
 				<geometry>
-					<mesh filename="package://fanuc_m16ib_support/meshes/m16ib20/visual/Link_2.STL"/>
+					<mesh filename="package://fanuc_m16ib_support/meshes/m16ib20/visual/link_2.stl"/>
 				</geometry>
 				<xacro:material_fanuc_yellow />
@@ -45,5 +45,5 @@
 				<origin xyz="0 0 0" rpy="0 0 0"/>
 				<geometry>
-					<mesh filename="package://fanuc_m16ib_support/meshes/m16ib20/collision/Link_2.STL"/>
+					<mesh filename="package://fanuc_m16ib_support/meshes/m16ib20/collision/link_2.stl"/>
 				</geometry>
 			</collision>
@@ -53,5 +53,5 @@
 				<origin xyz="0 0 0" rpy="0 0 0"/>
 				<geometry>
-					<mesh filename="package://fanuc_m16ib_support/meshes/m16ib20/visual/Link_3.STL"/>
+					<mesh filename="package://fanuc_m16ib_support/meshes/m16ib20/visual/link_3.stl"/>
 				</geometry>
 				<xacro:material_fanuc_yellow />
@@ -60,5 +60,5 @@
 				<origin xyz="0 0 0" rpy="0 0 0"/>
 				<geometry>
-					<mesh filename="package://fanuc_m16ib_support/meshes/m16ib20/collision/Link_3.STL"/>
+					<mesh filename="package://fanuc_m16ib_support/meshes/m16ib20/collision/link_3.stl"/>
 				</geometry>
 			</collision>
@@ -68,5 +68,5 @@
 				<origin xyz="0 0 0" rpy="0 0 0"/>
 				<geometry>
-					<mesh filename="package://fanuc_m16ib_support/meshes/m16ib20/visual/Link_4.STL"/>
+					<mesh filename="package://fanuc_m16ib_support/meshes/m16ib20/visual/link_4.stl"/>
 				</geometry>
 				<xacro:material_fanuc_yellow />
@@ -75,5 +75,5 @@
 				<origin xyz="0 0 0" rpy="0 0 0"/>
 				<geometry>
-					<mesh filename="package://fanuc_m16ib_support/meshes/m16ib20/collision/Link_4.STL"/>
+					<mesh filename="package://fanuc_m16ib_support/meshes/m16ib20/collision/link_4.stl"/>
 				</geometry>
 			</collision>
@@ -83,5 +83,5 @@
 				<origin xyz="0 0 0" rpy="0 0 0"/>
 				<geometry>
-					<mesh filename="package://fanuc_m16ib_support/meshes/m16ib20/visual/Link_5.STL"/>
+					<mesh filename="package://fanuc_m16ib_support/meshes/m16ib20/visual/link_5.stl"/>
 				</geometry>
 				<xacro:material_fanuc_yellow />
@@ -90,5 +90,5 @@
 				<origin xyz="0 0 0" rpy="0 0 0"/>
 				<geometry>
-					<mesh filename="package://fanuc_m16ib_support/meshes/m16ib20/collision/Link_5.STL"/>
+					<mesh filename="package://fanuc_m16ib_support/meshes/m16ib20/collision/link_5.stl"/>
 				</geometry>
 			</collision>
@@ -98,5 +98,5 @@
 				<origin xyz="0 0 0" rpy="0 0 0"/>
 				<geometry>
-					<mesh filename="package://fanuc_m16ib_support/meshes/m16ib20/visual/Link_6.STL"/>
+					<mesh filename="package://fanuc_m16ib_support/meshes/m16ib20/visual/link_6.stl"/>
 				</geometry>
 				<xacro:material_fanuc_black />
@@ -105,5 +105,5 @@
 				<origin xyz="0 0 0" rpy="0 0 0"/>
 				<geometry>
-					<mesh filename="package://fanuc_m16ib_support/meshes/m16ib20/collision/Link_6.STL"/>
+					<mesh filename="package://fanuc_m16ib_support/meshes/m16ib20/collision/link_6.stl"/>
 				</geometry>
 			</collision>
